File: PCB_CARRIER/cm4-high-speed.kicad_sch (KiCad schematic)
At the start: 1 part

Commit message: updating journal
Parts:
- renumbered Module1 to Module2
Connections:
- net GND: no longer Module2.107 (GND), Module2.108 (GND), Module2.113 (GND), Module2.114 (GND), Module2.119 (GND), Module2.120 (GND), Module2.125 (GND), Module2.126 (GND), Module2.131 (GND), Module2.132 (GND), Module2.137 (GND), Module2.138 (GND), Module2.144 (GND), Module2.150 (GND), Module2.155 (GND), Module2.156 (GND), Module2.161 (GND), Module2.162 (GND), Module2.167 (GND), Module2.168 (GND), Module2.173 (GND), Module2.174 (GND), Module2.179 (GND), Module2.180 (GND), Module2.185 (GND), Module2.186 (GND), Module2.191 (GND), Module2.192 (GND), Module2.197 (GND), Module2.198 (GND)
Other:
- title: Raspberry Pi Compute Module 4 Carrier Template -> CM4/CM5 Carrier Board
Changed lines of the file:
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@@
 	(paper "A4")
 	(title_block
-		(title "Raspberry Pi Compute Module 4 Carrier Template")
-		(date "2020-10-31")
-		(rev "v01")
-		(comment 2 "creativecommons.org/licenses/by-sa/4.0")
-		(comment 3 "License: CC BY 4.0")
-		(comment 4 "Author: Shawn Hymel")
+		(title "CM4/CM5 Carrier Board")
 	)
 	(junction
@@
 		(on_board yes)
 		(dnp no)
-		(property "Reference" "#PWR?"
+		(property "Reference" "#PWR01"
 			(at 40.64 181.61 0)
 			(effects
@@
 		)
 		(pin "1"
-		)
-		(instances
-			(project ""
-				(path "/f52509e6-8053-454c-b8e9-3e2670c5a5fe/caa71f4c-454d-4ac9-b287-456eafb34991"
-					(reference "#PWR?")
-					(unit 1)
-				)
-			)
 		)
 	)
@@
 		(on_board yes)
 		(dnp no)
-		(property "Reference" "#PWR?"
+		(property "Reference" "#PWR02"
 			(at 106.68 181.61 0)
 			(effects
@@
 		)
 		(pin "1"
-		)
-		(instances
-			(project ""
-				(path "/f52509e6-8053-454c-b8e9-3e2670c5a5fe/caa71f4c-454d-4ac9-b287-456eafb34991"
-					(reference "#PWR?")
-					(unit 1)
-				)
-			)
 		)
 	)
@@
 		(lib_id "CM4IO:ComputeModule4-CM4")
 		(at -66.04 106.68 0)
-		(unit 2)
+		(unit 1)
 		(exclude_from_sim no)
 		(in_bom yes)
 		(on_board yes)
 		(dnp no)
-		(property "Reference" "Module1"
+		(property "Reference" "Module2"
 			(at 73.66 33.02 0)
 			(effects
@@
 		(pin "153"
 		)
-		(instances
-			(project ""
-				(path "/f52509e6-8053-454c-b8e9-3e2670c5a5fe/caa71f4c-454d-4ac9-b287-456eafb34991"
-					(reference "Module1")
-					(unit 2)
-				)
-			)
-		)
-	)
+	)

Commit message: added in the SODIMM connectors to schematic
Parts:
- renumbered Module2 to Module?
Changed lines of the file:
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@@
 		(on_board yes)
 		(dnp no)
-		(property "Reference" "#PWR01"
+		(property "Reference" "#PWR?"
 			(at 40.64 181.61 0)
 			(effects
@@
 		)
 		(pin "1"
+		)
+		(instances
+			(project "carrier"
+				(path "/f52509e6-8053-454c-b8e9-3e2670c5a5fe/caa71f4c-454d-4ac9-b287-456eafb34991"
+					(reference "#PWR?")
+					(unit 1)
+				)
+			)
 		)
 	)
@@
 		(on_board yes)
 		(dnp no)
-		(property "Reference" "#PWR02"
+		(property "Reference" "#PWR?"
 			(at 106.68 181.61 0)
 			(effects
@@
 		)
 		(pin "1"
+		)
+		(instances
+			(project "carrier"
+				(path "/f52509e6-8053-454c-b8e9-3e2670c5a5fe/caa71f4c-454d-4ac9-b287-456eafb34991"
+					(reference "#PWR?")
+					(unit 1)
+				)
+			)
 		)
 	)
@@
 		(on_board yes)
 		(dnp no)
-		(property "Reference" "Module2"
+		(property "Reference" "Module?"
 			(at 73.66 33.02 0)
 			(effects
@@
 		(pin "153"
 		)
+		(instances
+			(project "carrier"
+				(path "/f52509e6-8053-454c-b8e9-3e2670c5a5fe/caa71f4c-454d-4ac9-b287-456eafb34991"
+					(reference "Module?")
+					(unit 1)
+				)
+			)
+		)
 	)

Commit message: updating every single symbol to be more accurate!
Changed lines of the file:
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@@
 			)
 		)
-		(property "Description" ""
+		(property "Description" "Power symbol creates a global label with name \"GND\" , ground"
 			(at 40.64 175.26 0)
 			(effects
@@
 			)
 		)
-		(property "Description" ""
+		(property "Description" "Power symbol creates a global label with name \"GND\" , ground"
 			(at 106.68 175.26 0)
 			(effects

Commit message: symbol got messed up for some reason
Connections:
- net GND: now also Module?.107 (GND), Module?.108 (GND), Module?.113 (GND), Module?.114 (GND), Module?.119 (GND), Module?.120 (GND), Module?.125 (GND), Module?.126 (GND), Module?.131 (GND), Module?.132 (GND), Module?.137 (GND), Module?.138 (GND), Module?.144 (GND), Module?.150 (GND), Module?.155 (GND), Module?.156 (GND), Module?.161 (GND), Module?.162 (GND), Module?.167 (GND), Module?.168 (GND), Module?.173 (GND), Module?.174 (GND), Module?.179 (GND), Module?.180 (GND), Module?.185 (GND), Module?.186 (GND), Module?.191 (GND), Module?.192 (GND), Module?.197 (GND), Module?.198 (GND)
Changed lines of the file:
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@@
 					(size 1.27 1.27)
 				)
+				(hide yes)
 			)
 		)
@@
 					(size 1.27 1.27)
 				)
+				(hide yes)
 			)
 		)
@@
 		(lib_id "CM4IO:ComputeModule4-CM4")
 		(at -66.04 106.68 0)
-		(unit 1)
+		(unit 2)
 		(exclude_from_sim no)
 		(in_bom yes)
@@
 		)
 		(property "Manufacturer" "Hirose"
-			(at -66.04 106.68 0)
+			(at 74.422 114.3 0)
 			(effects
 				(font
@@
 		)
 		(property "MPN" "2x DF40C-100DS-0.4V"
-			(at -66.04 109.22 0)
+			(at 74.422 116.84 0)
 			(effects
 				(font
@@
 		)
 		(property "MPN (Alt)" "2x DF40HC(3.0)-100DS-0.4V"
-			(at -66.04 106.68 0)
+			(at 74.422 114.3 0)
 			(effects
 				(font
@@
 				(path "/f52509e6-8053-454c-b8e9-3e2670c5a5fe/caa71f4c-454d-4ac9-b287-456eafb34991"
 					(reference "Module?")
-					(unit 1)
-				)
-			)
+					(unit 2)
+				)
+			)
