File: PCB_CARRIER/cm4-high-speed.kicad_sch (KiCad schematic)
At the start: 1 part

Commit message: time to switch the mezzanine connector, saving at this point if I mess up
Parts:
- Module1: footprint CM4IO:Raspberry-Pi-4-Compute-Module -> kai's library:Raspberry-Pi-4-Compute-Module
Changed lines of the file:
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@@
 			)
 		)
-		(property "Footprint" "CM4IO:Raspberry-Pi-4-Compute-Module"
+		(property "Footprint" "kai's library:Raspberry-Pi-4-Compute-Module"
 			(at 132.08 123.19 0)
 			(effects

Commit message: separating mezzanine connector symbol/footprint for easy pcba, a bit sketch
Parts:
- removed Module1: ComputeModule4-CM4, kai's library:Raspberry-Pi-4-Compute-Module, symbol CM4IO:ComputeModule4-CM4
- added Module1: Mezzanine_B, kai's library:Raspberry-Pi-4-Compute-Module-B, symbol kai-library:Mezzanine_B
Connections:
- net CSI-0_CLK_N: now also Module1.127 (CAM1_C_N)
- net CSI-0_CLK_P: now also Module1.129 (CAM1_C_P)
- net CSI-0_D0_N: now also Module1.115 (CAM1_D0_N)
- net CSI-0_D0_P: now also Module1.117 (CAM1_D0_P)
- net CSI-0_D1_N: now also Module1.121 (CAM1_D1_N)
- net CSI-0_D1_P: now also Module1.123 (CAM1_D1_P)
- net CSI-0_D2_N: now also Module1.133 (CAM1_D2_N)
- net CSI-0_D2_P: now also Module1.135 (CAM1_D2_P)
- net CSI-0_D3_N: now also Module1.139 (CAM1_D3_N)
- net CSI-0_D3_P: now also Module1.141 (CAM1_D3_P)
- net CSI-1_CLK_N: now also Module1.187 (DSI1_C_N)
- net CSI-1_CLK_P: now also Module1.189 (DSI1_C_P)
- net CSI-1_D0_N: now also Module1.175 (DSI1_D0_N)
- net CSI-1_D0_P: now also Module1.177 (DSI1_D0_P)
- net CSI-1_D1_N: now also Module1.181 (DSI1_D1_N)
- net CSI-1_D1_P: now also Module1.183 (DSI1_D1_P)
- net CSI-1_D2_N: now also Module1.193 (DSI1_D2_N)
- net CSI-1_D2_P: now also Module1.195 (DSI1_D2_P)
- net CSI-1_D3_N: now also Module1.194 (DSI1_D3_N)
- net CSI-1_D3_P: now also Module1.196 (DSI1_D3_P)
- net GND: now also Module1.107 (GND), Module1.108 (GND), Module1.113 (GND), Module1.114 (GND), Module1.119 (GND), Module1.120 (GND), Module1.125 (GND), Module1.126 (GND), Module1.131 (GND), Module1.132 (GND), Module1.137 (GND), Module1.138 (GND), Module1.144 (GND), Module1.150 (GND), Module1.155 (GND), Module1.156 (GND), Module1.161 (GND), Module1.162 (GND), Module1.167 (GND), Module1.168 (GND), Module1.173 (GND), Module1.174 (GND), Module1.179 (GND), Module1.180 (GND), Module1.185 (GND), Module1.186 (GND), Module1.191 (GND), Module1.192 (GND), Module1.197 (GND), Module1.198 (GND)
- net HDMI-0_CEC: now also Module1.151 (HDMI0_CEC)
- net HDMI-0_CLK_N: now also Module1.190 (HDMI0_CLK_N)
- net HDMI-0_CLK_P: now also Module1.188 (HDMI0_CLK_P)
- net HDMI-0_HPD: now also Module1.153 (HDMI0_HOTPLUG)
- net HDMI-0_SCL: now also Module1.200 (HDMI0_SCL)
- net HDMI-0_SDA: now also Module1.199 (HDMI0_SDA)
- net HDMI-0_TX0_N: now also Module1.184 (HDMI0_TX0_N)
- net HDMI-0_TX0_P: now also Module1.182 (HDMI0_TX0_P)
- net HDMI-0_TX1_N: now also Module1.178 (HDMI0_TX1_N)
- net HDMI-0_TX1_P: now also Module1.176 (HDMI0_TX1_P)
- net HDMI-0_TX2_N: now also Module1.172 (HDMI0_TX2_N)
- net HDMI-0_TX2_P: now also Module1.170 (HDMI0_TX2_P)
- net PCIe_CLKREQ: now also Module1.102 (PCIe_CLK_nREQ)
- net PCIe_CLK_N: now also Module1.112 (PCIe_CLK_N)
- net PCIe_CLK_P: now also Module1.110 (PCIe_CLK_P)
- net PCIe_RX_N: now also Module1.118 (PCIe_RX_N)
- net PCIe_RX_P: now also Module1.116 (PCIe_RX_P)
- net PCIe_TX_N: now also Module1.124 (PCIe_TX_N)
- net PCIe_TX_P: now also Module1.122 (PCIe_TX_P)
- net PCIe_nRST: now also Module1.109 (PCIe_nRST)
- net USB3-0-DN: now also Module1.136 (CAM0_D1_P)
- net USB3-0-DP: now also Module1.134 (CAM0_D1_N)
- net USB3-0-RX_N: now also Module1.128 (CAM0_D0_N)
- net USB3-0-RX_P: now also Module1.130 (CAM0_D0_P)
- net USB3-0-TX_N: now also Module1.140 (CAM0_C_N)
- net USB3-0-TX_P: now also Module1.142 (CAM0_C_P)
- net USB3-1-DN: now also Module1.165 (DSI0_D1_P)
- net USB3-1-DP: now also Module1.163 (DSI0_D1_N)
- net USB3-1-RX_N: now also Module1.157 (DSI0_D0_N)
- net USB3-1-RX_P: now also Module1.159 (DSI0_D0_P)
- net USB3-1-TX_N: now also Module1.169 (DSI0_C_N)
- net USB3-1-TX_P: now also Module1.171 (DSI0_C_P)
- net USB_N: now also Module1.103 (USB2_N)
- net USB_P: now also Module1.105 (USB2_P)

Commit message: making the schematic more clear!
Parts:
- Module1: value Mezzanine_B -> 10164227-1004A1RLF
Changed lines of the file:
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@@
 			)
 		)
-		(property "Value" "Mezzanine_B"
+		(property "Value" "10164227-1004A1RLF"
 			(at 130.302 21.082 0)
 			(effects
