File: PCB_CARRIER/SO-DIMM.kicad_sch (KiCad schematic)
At the start: 1 part, among them J1 SODIMM-260_Split

Commit message: symbol got messed up for some reason
Connections:
- net GNDA: now reaches J1.1 (1A)
- net TX1_P: now reaches J1.3 (3A)
Other:
- moved on the sheet: J1A, J1B, J1C, J1D, J1E, J1F, J1G
Changed lines of the file:
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@@
 	(generator_version "9.0")
 	(paper "A4")
+	(wire
+		(pts
+			(xy 35.56 35.56) (xy 38.1 35.56)
+		)
+		(stroke
+			(width 0)
+			(type default)
+		)
+	)
+	(wire
+		(pts
+			(xy 33.02 38.1) (xy 38.1 38.1)
+		)
+		(stroke
+			(width 0)
+			(type default)
+		)
+	)
+	(global_label "TX1_P"
+		(shape input)
+		(at 33.02 38.1 180)
+		(fields_autoplaced yes)
+		(effects
+			(font
+				(size 1.27 1.27)
+			)
+			(justify right)
+		)
+		(property "Intersheetrefs" "${INTERSHEET_REFS}"
+			(at 24.3155 38.1 0)
+			(effects
+				(font
+					(size 1.27 1.27)
+				)
+				(justify right)
+				(hide yes)
+			)
+		)
+	)
 	(symbol
 		(lib_id "SODIMM:SODIMM-260_Split")
-		(at 44.45 54.61 0)
+		(at 55.88 58.42 0)
 		(unit 1)
 		(exclude_from_sim no)
@@
 		(fields_autoplaced yes)
 		(property "Reference" "J1"
-			(at 44.45 24.13 0)
+			(at 55.88 27.94 0)
 			(effects
 				(font
@@
 		)
 		(property "Value" "SODIMM-260_Split"
-			(at 44.45 26.67 0)
+			(at 55.88 30.48 0)
 			(effects
 				(font
@@
 		)
 		(property "Footprint" ""
-			(at 80.01 33.02 0)
+			(at 91.44 36.83 0)
 			(effects
 				(font
@@
 		)
 		(property "Datasheet" "~"
-			(at 80.01 33.02 0)
+			(at 91.44 36.83 0)
 			(effects
 				(font
@@
 		)
 		(property "Description" "SODIMM 200 Pin socket"
-			(at 44.45 44.704 0)
+			(at 55.88 48.514 0)
 			(effects
 				(font
@@
 	)
 	(symbol
+		(lib_id "power:GNDA")
+		(at 35.56 35.56 0)
+		(unit 1)
+		(exclude_from_sim no)
+		(in_bom yes)
+		(on_board yes)
+		(dnp no)
+		(property "Reference" "#PWR01"
+			(at 35.56 41.91 0)
+			(effects
+				(font
+					(size 1.27 1.27)
+				)
+				(hide yes)
+			)
+		)
+		(property "Value" "GNDA"
+			(at 31.242 35.306 0)
+			(effects
+				(font
+					(size 1.27 1.27)
+				)
+			)
+		)
+		(property "Footprint" ""
+			(at 35.56 35.56 0)
+			(effects
+				(font
+					(size 1.27 1.27)
+				)
+				(hide yes)
+			)
+		)
+		(property "Datasheet" ""
+			(at 35.56 35.56 0)
+			(effects
+				(font
+					(size 1.27 1.27)
+				)
+				(hide yes)
+			)
+		)
+		(property "Description" "Power symbol creates a global label with name \"GNDA\" , analog ground"
+			(at 35.56 35.56 0)
+			(effects
+				(font
+					(size 1.27 1.27)
+				)
+				(hide yes)
+			)
+		)
+		(pin "1"
+		)
+		(instances
+			(project ""
+				(path "/f52509e6-8053-454c-b8e9-3e2670c5a5fe/9924afb8-28d2-4519-98a2-71323cd667d5"
+					(reference "#PWR01")
+					(unit 1)
+				)
+			)
+		)
+	)
+	(symbol
 		(lib_id "SODIMM:SODIMM-260_Split")
-		(at 160.02 132.08 0)
+		(at 171.45 135.89 0)
 		(unit 7)
 		(exclude_from_sim no)
@@
 		(fields_autoplaced yes)
 		(property "Reference" "J1"
-			(at 160.02 101.6 0)
+			(at 171.45 105.41 0)
 			(effects
 				(font
@@
 		)
 		(property "Value" "SODIMM-260_Split"
-			(at 160.02 104.14 0)
+			(at 171.45 107.95 0)
 			(effects
 				(font
@@
 		)
 		(property "Footprint" ""
-			(at 195.58 110.49 0)
+			(at 207.01 114.3 0)
 			(effects
 				(font
@@
 		)
 		(property "Datasheet" "~"
-			(at 195.58 110.49 0)
+			(at 207.01 114.3 0)
 			(effects
 				(font
@@
 		)
 		(property "Description" "SODIMM 200 Pin socket"
-			(at 160.02 122.174 0)
+			(at 171.45 125.984 0)
 			(effects
 				(font
@@
 	(symbol
 		(lib_id "SODIMM:SODIMM-260_Split")
-		(at 102.87 54.61 0)
+		(at 114.3 58.42 0)
 		(unit 2)
 		(exclude_from_sim no)
@@
 		(fields_autoplaced yes)
 		(property "Reference" "J1"
-			(at 102.87 25.4 0)
+			(at 114.3 29.21 0)
 			(effects
 				(font
@@
 		)
 		(property "Value" "SODIMM-260_Split"
-			(at 102.87 27.94 0)
+			(at 114.3 31.75 0)
 			(effects
 				(font
@@
 		)
 		(property "Footprint" ""
-			(at 138.43 33.02 0)
+			(at 149.86 36.83 0)
 			(effects
 				(font
@@
 		)
 		(property "Datasheet" "~"
-			(at 138.43 33.02 0)
+			(at 149.86 36.83 0)
 			(effects
 				(font
@@
 		)
 		(property "Description" "SODIMM 200 Pin socket"
-			(at 102.87 44.704 0)
+			(at 114.3 48.514 0)
 			(effects
 				(font
@@
 	(symbol
 		(lib_id "SODIMM:SODIMM-260_Split")
-		(at 102.87 132.08 0)
+		(at 114.3 135.89 0)
 		(unit 6)
 		(exclude_from_sim no)
@@
 		(fields_autoplaced yes)
 		(property "Reference" "J1"
-			(at 102.87 101.6 0)
+			(at 114.3 105.41 0)
 			(effects
 				(font
@@
 		)
 		(property "Value" "SODIMM-260_Split"
-			(at 102.87 104.14 0)
+			(at 114.3 107.95 0)
 			(effects
 				(font
@@
 		)
 		(property "Footprint" ""
-			(at 138.43 110.49 0)
+			(at 149.86 114.3 0)
 			(effects
 				(font
@@
 		)
 		(property "Datasheet" "~"
-			(at 138.43 110.49 0)
+			(at 149.86 114.3 0)
 			(effects
 				(font
@@
 		)
 		(property "Description" "SODIMM 200 Pin socket"
-			(at 102.87 122.174 0)
+			(at 114.3 125.984 0)
 			(effects
 				(font
@@
 	(symbol
 		(lib_id "SODIMM:SODIMM-260_Split")
-		(at 160.02 54.61 0)
+		(at 171.45 58.42 0)
 		(unit 3)
 		(exclude_from_sim no)
@@
 		(fields_autoplaced yes)
 		(property "Reference" "J1"
-			(at 160.02 25.4 0)
+			(at 171.45 29.21 0)
 			(effects
 				(font
@@
 		)
 		(property "Value" "SODIMM-260_Split"
-			(at 160.02 27.94 0)
+			(at 171.45 31.75 0)
 			(effects
 				(font
@@
 		)
 		(property "Footprint" ""
-			(at 195.58 33.02 0)
+			(at 207.01 36.83 0)
 			(effects
 				(font
@@
 		)
 		(property "Datasheet" "~"
-			(at 195.58 33.02 0)
+			(at 207.01 36.83 0)
 			(effects
 				(font
@@
 		)
 		(property "Description" "SODIMM 200 Pin socket"
-			(at 160.02 44.704 0)
+			(at 171.45 48.514 0)
 			(effects
 				(font
@@
 	(symbol
 		(lib_id "SODIMM:SODIMM-260_Split")
-		(at 218.44 54.61 0)
+		(at 229.87 58.42 0)
 		(unit 4)
 		(exclude_from_sim no)
@@
 		(fields_autoplaced yes)
 		(property "Reference" "J1"
-			(at 218.44 25.4 0)
+			(at 229.87 29.21 0)
 			(effects
 				(font
@@
 		)
 		(property "Value" "SODIMM-260_Split"
-			(at 218.44 27.94 0)
+			(at 229.87 31.75 0)
 			(effects
 				(font
@@
 		)
 		(property "Footprint" ""
-			(at 254 33.02 0)
+			(at 265.43 36.83 0)
 			(effects
 				(font
@@
 		)
 		(property "Datasheet" "~"
-			(at 254 33.02 0)
+			(at 265.43 36.83 0)
 			(effects
 				(font
@@
 		)
 		(property "Description" "SODIMM 200 Pin socket"
-			(at 218.44 44.704 0)
+			(at 229.87 48.514 0)
 			(effects
 				(font
@@
 	(symbol
 		(lib_id "SODIMM:SODIMM-260_Split")
-		(at 44.45 132.08 0)
+		(at 55.88 135.89 0)
 		(unit 5)
 		(exclude_from_sim no)
@@
 		(fields_autoplaced yes)
 		(property "Reference" "J1"
-			(at 44.45 102.87 0)
+			(at 55.88 106.68 0)
 			(effects
 				(font
@@
 		)
 		(property "Value" "SODIMM-260_Split"
-			(at 44.45 105.41 0)
+			(at 55.88 109.22 0)
 			(effects
 				(font
@@
 		)
 		(property "Footprint" ""
-			(at 80.01 110.49 0)
+			(at 91.44 114.3 0)
 			(effects
 				(font
@@
 		)
 		(property "Datasheet" "~"
-			(at 80.01 110.49 0)
+			(at 91.44 114.3 0)
 			(effects
 				(font
@@
 		)
 		(property "Description" "SODIMM 200 Pin socket"
-			(at 44.45 122.174 0)
+			(at 55.88 125.984 0)
 			(effects
 				(font

Commit message: updated every single symbol to put a/b at the start
Connections:
- net GNDA: now also J1.12 (A12)
- net GND: now reaches J1.131 (B1)
- net GND: now also J1.142 (B12)
- net TX1_P: no longer names the net of J1.3 (A3)
- no-connect marks 0 -> 2
Changed lines of the file:
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@@
 	(generator_version "9.0")
 	(paper "A4")
+	(no_connect
+		(at 247.65 55.88)
+	)
+	(no_connect
+		(at 73.66 43.18)
+	)
 	(wire
 		(pts
-			(xy 35.56 35.56) (xy 38.1 35.56)
+			(xy 34.29 35.56) (xy 38.1 35.56)
 		)
 		(stroke
@@
 	(wire
 		(pts
-			(xy 33.02 38.1) (xy 38.1 38.1)
+			(xy 208.28 48.26) (xy 212.09 48.26)
 		)
 		(stroke
@@
 		)
 	)
-	(global_label "TX1_P"
-		(shape input)
-		(at 33.02 38.1 180)
-		(fields_autoplaced yes)
-		(effects
-			(font
-				(size 1.27 1.27)
-			)
-			(justify right)
-		)
-		(property "Intersheetrefs" "${INTERSHEET_REFS}"
-			(at 24.3155 38.1 0)
-			(effects
-				(font
-					(size 1.27 1.27)
-				)
-				(justify right)
-				(hide yes)
-			)
+	(wire
+		(pts
+			(xy 77.47 48.26) (xy 73.66 48.26)
+		)
+		(stroke
+			(width 0)
+			(type default)
+		)
+	)
+	(wire
+		(pts
+			(xy 251.46 60.96) (xy 247.65 60.96)
+		)
+		(stroke
+			(width 0)
+			(type default)
 		)
 	)
@@
 	(symbol
 		(lib_id "power:GNDA")
-		(at 35.56 35.56 0)
+		(at 77.47 48.26 0)
 		(unit 1)
 		(exclude_from_sim no)
@@
 		(on_board yes)
 		(dnp no)
+		(fields_autoplaced yes)
+		(property "Reference" "#PWR02"
+			(at 77.47 54.61 0)
+			(effects
+				(font
+					(size 1.27 1.27)
+				)
+				(hide yes)
+			)
+		)
+		(property "Value" "GNDA"
+			(at 77.47 53.34 0)
+			(effects
+				(font
+					(size 1.27 1.27)
+				)
+			)
+		)
+		(property "Footprint" ""
+			(at 77.47 48.26 0)
+			(effects
+				(font
+					(size 1.27 1.27)
+				)
+				(hide yes)
+			)
+		)
+		(property "Datasheet" ""
+			(at 77.47 48.26 0)
+			(effects
+				(font
+					(size 1.27 1.27)
+				)
+				(hide yes)
+			)
+		)
+		(property "Description" "Power symbol creates a global label with name \"GNDA\" , analog ground"
+			(at 77.47 48.26 0)
+			(effects
+				(font
+					(size 1.27 1.27)
+				)
+				(hide yes)
+			)
+		)
+		(pin "1"
+		)
+		(instances
+			(project ""
+				(path "/f52509e6-8053-454c-b8e9-3e2670c5a5fe/9924afb8-28d2-4519-98a2-71323cd667d5"
+					(reference "#PWR02")
+					(unit 1)
+				)
+			)
+		)
+	)
+	(symbol
+		(lib_id "power:GND")
+		(at 208.28 48.26 0)
+		(unit 1)
+		(exclude_from_sim no)
+		(in_bom yes)
+		(on_board yes)
+		(dnp no)
+		(fields_autoplaced yes)
+		(property "Reference" "#PWR03"
+			(at 208.28 54.61 0)
+			(effects
+				(font
+					(size 1.27 1.27)
+				)
+				(hide yes)
+			)
+		)
+		(property "Value" "GND"
+			(at 208.28 53.34 0)
+			(effects
+				(font
+					(size 1.27 1.27)
+				)
+			)
+		)
+		(property "Footprint" ""
+			(at 208.28 48.26 0)
+			(effects
+				(font
+					(size 1.27 1.27)
+				)
+				(hide yes)
+			)
+		)
+		(property "Datasheet" ""
+			(at 208.28 48.26 0)
+			(effects
+				(font
+					(size 1.27 1.27)
+				)
+				(hide yes)
+			)
+		)
+		(property "Description" "Power symbol creates a global label with name \"GND\" , ground"
+			(at 208.28 48.26 0)
+			(effects
+				(font
+					(size 1.27 1.27)
+				)
+				(hide yes)
+			)
+		)
+		(pin "1"
+		)
+		(instances
+			(project ""
+				(path "/f52509e6-8053-454c-b8e9-3e2670c5a5fe/9924afb8-28d2-4519-98a2-71323cd667d5"
+					(reference "#PWR03")
+					(unit 1)
+				)
+			)
+		)
+	)
+	(symbol
+		(lib_id "power:GNDA")
+		(at 34.29 35.56 0)
+		(unit 1)
+		(exclude_from_sim no)
+		(in_bom yes)
+		(on_board yes)
+		(dnp no)
+		(fields_autoplaced yes)
 		(property "Reference" "#PWR01"
-			(at 35.56 41.91 0)
+			(at 34.29 41.91 0)
 			(effects
 				(font
@@
 		)
 		(property "Value" "GNDA"
-			(at 31.242 35.306 0)
+			(at 34.29 40.64 0)
 			(effects
 				(font
@@
 		)
 		(property "Footprint" ""
-			(at 35.56 35.56 0)
+			(at 34.29 35.56 0)
 			(effects
 				(font
@@
 		)
 		(property "Datasheet" ""
-			(at 35.56 35.56 0)
+			(at 34.29 35.56 0)
 			(effects
 				(font
@@
 		)
 		(property "Description" "Power symbol creates a global label with name \"GNDA\" , analog ground"
-			(at 35.56 35.56 0)
+			(at 34.29 35.56 0)
 			(effects
 				(font
@@
 				)
 			)
+		)
+	)
+	(symbol
+		(lib_id "power:GND")
+		(at 251.46 60.96 0)
+		(unit 1)
+		(exclude_from_sim no)
+		(in_bom yes)
+		(on_board yes)
+		(dnp no)
+		(fields_autoplaced yes)
+		(property "Reference" "#PWR04"
+			(at 251.46 67.31 0)
+			(effects
+				(font
+					(size 1.27 1.27)
+				)
+				(hide yes)
+			)
+		)
+		(property "Value" "GND"
+			(at 251.46 66.04 0)
+			(effects
+				(font
+					(size 1.27 1.27)
+				)
+			)
+		)
+		(property "Footprint" ""
+			(at 251.46 60.96 0)
+			(effects
+				(font
+					(size 1.27 1.27)
+				)
+				(hide yes)
+			)
+		)
+		(property "Datasheet" ""
+			(at 251.46 60.96 0)
+			(effects
+				(font
+					(size 1.27 1.27)
+				)
+				(hide yes)
+			)
+		)
+		(property "Description" "Power symbol creates a global label with name \"GND\" , ground"
+			(at 251.46 60.96 0)
+			(effects
+				(font
+					(size 1.27 1.27)
+				)
+				(hide yes)
+			)
+		)
+		(pin "1"
+		)
+		(instances
+			(project "carrier"
+				(path "/f52509e6-8053-454c-b8e9-3e2670c5a5fe/9924afb8-28d2-4519-98a2-71323cd667d5"
+					(reference "#PWR04")
+					(unit 1)
+				)
+			)

Commit message: working on getting all the grounds into SODIMM
Connections:
- net GND: now also J1.1 (A1), J1.102 (A102), J1.107 (A107), J1.113 (A113), J1.119 (A119), J1.13 (A13), J1.14 (A14), J1.19 (A19), J1.2 (A2), J1.20 (A20), J1.25 (A25), J1.26 (A26), J1.31 (A31), J1.32 (A32), J1.37 (A37), J1.38 (A38), J1.43 (A43), J1.44 (A44), J1.49 (A49), J1.50 (A50), J1.55 (A55), J1.56 (A56), J1.61 (A61), J1.62 (A62), J1.67 (A67), J1.68 (A68), J1.7 (A7), J1.73 (A73), J1.74 (A74), J1.79 (A79), J1.8 (A8), J1.80 (A80), J1.85 (A85), J1.86 (A86); no longer J1.131 (B1), J1.142 (B12)
- net GNDA: no longer names the net of J1.12 (A12)
- net GNDA: no longer J1.1 (A1)
- no-connect marks 2 -> 0

Commit message: all the ground SODIMM's have been wired up
Connections:
- net GND: now also J1.125 (A125), J1.129 (A129), J1.132 (B2), J1.135 (B5), J1.138 (B8), J1.141 (B11), J1.144 (B14), J1.146 (B16), J1.147 (B17), J1.152 (B22), J1.153 (B23), J1.158 (B28), J1.159 (B29), J1.164 (B34), J1.165 (B35), J1.170 (B40), J1.171 (B41), J1.176 (B46), J1.177 (B47), J1.200 (B70), J1.201 (B71), J1.231 (B101), J1.241 (B111), J1.242 (B112), J1.243 (B113), J1.244 (B114), J1.245 (B115), J1.246 (B116), J1.247 (B117), J1.248 (B118), J1.249 (B119), J1.250 (B120)
Other:
- moved on the sheet: J1F

Commit message: adding in the power pins, this is going to take a long time...
Connections:
- net +5V: now reaches J1.251 (B121)
- net +5V: now also J1.252 (B122), J1.253 (B123), J1.254 (B124), J1.255 (B125), J1.256 (B126), J1.257 (B127), J1.258 (B128), J1.259 (B129)
Changed lines of the file:
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@@
+	)
+	(junction
+		(at 152.4 130.81)
+		(diameter 0)
+		(color 0 0 0 0)
 	)
 	(junction
@@
 	)
 	(junction
+		(at 152.4 128.27)
+		(diameter 0)
+		(color 0 0 0 0)
+	)
+	(junction
 		(at 151.13 68.58)
 		(diameter 0)
@@
 	)
 	(junction
+		(at 190.5 128.27)
+		(diameter 0)
+		(color 0 0 0 0)
+	)
+	(junction
 		(at 76.2 58.42)
 		(diameter 0)
@@
 	)
 	(junction
+		(at 152.4 125.73)
+		(diameter 0)
+		(color 0 0 0 0)
+	)
+	(junction
 		(at 250.19 66.04)
 		(diameter 0)
@@
 	)
 	(junction
+		(at 152.4 133.35)
+		(diameter 0)
+		(color 0 0 0 0)
+	)
+	(junction
 		(at 76.2 130.81)
 		(diameter 0)
@@
 	)
 	(junction
+		(at 190.5 125.73)
+		(diameter 0)
+		(color 0 0 0 0)
+	)
+	(junction
 		(at 134.62 76.2)
 		(diameter 0)
@@
 	)
 	(junction
+		(at 190.5 130.81)
+		(diameter 0)
+		(color 0 0 0 0)
+	)
+	(junction
 		(at 35.56 125.73)
 		(diameter 0)
@@
 	(wire
 		(pts
+			(xy 152.4 133.35) (xy 152.4 135.89)
+		)
+		(stroke
+			(width 0)
+			(type default)
+		)
+	)
+	(wire
+		(pts
 			(xy 132.08 45.72) (xy 134.62 45.72)
 		)
@@
 	(wire
 		(pts
+			(xy 152.4 128.27) (xy 152.4 130.81)
+		)
+		(stroke
+			(width 0)
+			(type default)
+		)
+	)
+	(wire
+		(pts
 			(xy 132.08 76.2) (xy 134.62 76.2)
 		)
@@
 	(wire
 		(pts
+			(xy 189.23 128.27) (xy 190.5 128.27)
+		)
+		(stroke
+			(width 0)
+			(type default)
+		)
+	)
+	(wire
+		(pts
 			(xy 209.55 76.2) (xy 209.55 83.82)
 		)
@@
 	(wire
 		(pts
+			(xy 153.67 133.35) (xy 152.4 133.35)
+		)
+		(stroke
+			(width 0)
+			(type default)
+		)
+	)
+	(wire
+		(pts
 			(xy 76.2 161.29) (xy 76.2 166.37)
 		)
@@
 	(wire
 		(pts
+			(xy 189.23 125.73) (xy 190.5 125.73)
+		)
+		(stroke
+			(width 0)
+			(type default)
+		)
+	)
+	(wire
+		(pts
 			(xy 73.66 43.18) (xy 76.2 43.18)
 		)
@@
 	(wire
 		(pts
+			(xy 153.67 135.89) (xy 152.4 135.89)
+		)
+		(stroke
+			(width 0)
+			(type default)
+		)
+	)
+	(wire
+		(pts
 			(xy 153.67 40.64) (xy 151.13 40.64)
 		)
@@
 	(wire
 		(pts
+			(xy 153.67 125.73) (xy 152.4 125.73)
+		)
+		(stroke
+			(width 0)
+			(type default)
+		)
+	)
+	(wire
+		(pts
 			(xy 151.13 83.82) (xy 151.13 87.63)
 		)
@@
 	(wire
 		(pts
+			(xy 189.23 130.81) (xy 190.5 130.81)
+		)
+		(stroke
+			(width 0)
+			(type default)
+		)
+	)
+	(wire
+		(pts
 			(xy 93.98 53.34) (xy 96.52 53.34)
 		)
@@
 	(wire
 		(pts
+			(xy 153.67 130.81) (xy 152.4 130.81)
+		)
+		(stroke
+			(width 0)
+			(type default)
+		)
+	)
+	(wire
+		(pts
 			(xy 151.13 118.11) (xy 151.13 120.65)
 		)
@@
 	(wire
 		(pts
+			(xy 152.4 130.81) (xy 152.4 133.35)
+		)
+		(stroke
+			(width 0)
+			(type default)
+		)
+	)
+	(wire
+		(pts
 			(xy 247.65 55.88) (xy 250.19 55.88)
 		)
@@
 	(wire
 		(pts
+			(xy 190.5 107.95) (xy 190.5 125.73)
+		)
+		(stroke
+			(width 0)
+			(type default)
+		)
+	)
+	(wire
+		(pts
 			(xy 189.23 118.11) (xy 191.77 118.11)
 		)
@@
 	(wire
 		(pts
+			(xy 152.4 107.95) (xy 152.4 125.73)
+		)
+		(stroke
+			(width 0)
+			(type default)
+		)
+	)
+	(wire
+		(pts
 			(xy 250.19 81.28) (xy 250.19 87.63)
 		)
@@
 	(wire
 		(pts
+			(xy 190.5 125.73) (xy 190.5 128.27)
+		)
+		(stroke
+			(width 0)
+			(type default)
+		)
+	)
+	(wire
+		(pts
 			(xy 132.08 53.34) (xy 134.62 53.34)
 		)
@@
 	(wire
 		(pts
+			(xy 152.4 128.27) (xy 153.67 128.27)
+		)
+		(stroke
+			(width 0)
+			(type default)
+		)
+	)
+	(wire
+		(pts
 			(xy 191.77 120.65) (xy 191.77 123.19)
 		)
@@
 	(wire
 		(pts
+			(xy 189.23 133.35) (xy 190.5 133.35)
+		)
+		(stroke
+			(width 0)
+			(type default)
+		)
+	)
+	(wire
+		(pts
 			(xy 93.98 76.2) (xy 93.98 83.82)
 		)
@@
 	(wire
 		(pts
+			(xy 152.4 125.73) (xy 152.4 128.27)
+		)
+		(stroke
+			(width 0)
+			(type default)
+		)
+	)
+	(wire
+		(pts
 			(xy 209.55 40.64) (xy 209.55 45.72)
 		)
@@
 	(wire
 		(pts
+			(xy 190.5 130.81) (xy 190.5 133.35)
+		)
+		(stroke
+			(width 0)
+			(type default)
+		)
+	)
+	(wire
+		(pts
+			(xy 190.5 128.27) (xy 190.5 130.81)
+		)
+		(stroke
+			(width 0)
+			(type default)
+		)
+	)
+	(wire
+		(pts
 			(xy 35.56 50.8) (xy 38.1 50.8)
 		)
@@
 		)
 	)
+	(global_label "+5V"
+		(shape output)
+		(at 152.4 107.95 90)
+		(fields_autoplaced yes)
+		(effects
+			(font
+				(size 1.27 1.27)
+			)
+			(justify left)
+		)
+		(property "Intersheetrefs" "${INTERSHEET_REFS}"
+			(at 152.4 100.9992 90)
+			(effects
+				(font
+					(size 1.27 1.27)
+				)
+				(justify left)
+				(hide yes)
+			)
+		)
+	)
+	(global_label "+5V"
+		(shape output)
+		(at 190.5 107.95 90)
+		(fields_autoplaced yes)
+		(effects
+			(font
+				(size 1.27 1.27)
+			)
+			(justify left)
+		)
+		(property "Intersheetrefs" "${INTERSHEET_REFS}"
+			(at 190.5 100.9992 90)
+			(effects
+				(font
+					(size 1.27 1.27)
+				)
+				(justify left)
+				(hide yes)
+			)
+		)
+	)

Commit message: added decoupling for power on the daughter card
Connections:
- no-connect marks 0 -> 1
Other:
- note added: "<- Mechanical Pin"
Changed lines of the file:
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@@
 	(generator_version "9.0")
 	(paper "A4")
+	(text "<- Mechanical Pin"
+		(exclude_from_sim no)
+		(at 202.692 135.89 0)
+		(effects
+			(font
+				(size 1.27 1.27)
+			)
+		)
+	)
 	(junction
 		(at 76.2 161.29)
@@
 		(color 0 0 0 0)
 	)
+	(no_connect
+		(at 189.23 135.89)
+	)
 	(wire
