File: PCB_CARRIER/SO-DIMM.kicad_sch (KiCad schematic)
At the start: 1 part, among them J1 SODIMM-260_Split

Commit message: added sleep/wake and sys_reset
Connections:
- net SYS_RESET: now reaches J1.239
- net SLEEP/WAKE: now reaches J1.240
Other:
- note added: "< Research cluster board implement"
Changed lines of the file:
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@@
 		)
 	)
+	(text "< Research cluster board implement"
+		(exclude_from_sim no)
+		(at 232.664 203.454 0)
+		(effects
+			(font
+				(size 1.27 1.27)
+			)
+		)
+	)
 	(text "< Second camera?"
 		(exclude_from_sim no)
@@
 	(wire
 		(pts
+			(xy 152.4 203.2) (xy 157.48 203.2)
+		)
+		(stroke
+			(width 0)
+			(type default)
+		)
+	)
+	(wire
+		(pts
 			(xy 120.65 96.52) (xy 115.57 96.52)
 		)
@@
 	(wire
 		(pts
+			(xy 198.12 203.2) (xy 193.04 203.2)
+		)
+		(stroke
+			(width 0)
+			(type default)
+		)
+	)
+	(wire
+		(pts
 			(xy 152.4 160.02) (xy 157.48 160.02)
 		)
@@
 			(effects
 				(font
+					(size 1.27 1.27)
+				)
+				(justify left)
+				(hide yes)
+			)
+		)
+	)
+	(global_label "SYS_RESET"
+		(shape output)
+		(at 152.4 203.2 180)
+		(fields_autoplaced yes)
+		(effects
+			(font
+				(size 1.27 1.27)
+			)
+			(justify right)
+		)
+		(property "Intersheetrefs" "${INTERSHEET_REFS}"
+			(at 139.0994 203.2 0)
+			(effects
+				(font
+					(size 1.27 1.27)
+				)
+				(justify right)
+				(hide yes)
+			)
+		)
+	)
+	(global_label "SLEEP{slash}WAKE"
+		(shape bidirectional)
+		(at 198.12 203.2 0)
+		(fields_autoplaced yes)
+		(effects
+			(font
+				(size 1.27 1.27)
+			)
+			(justify left)
+		)
+		(property "Intersheetrefs" "${INTERSHEET_REFS}"
+			(at 214.3114 203.2 0)
+			(effects
+				(font

Commit message: added the NMOS for the PWR state
Connections:
- net SYS_RESET renamed RUN_PG
Changed lines of the file:
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@@
+		)
+	)
+	(global_label "RUN_PG"
+		(shape output)
+		(at 152.4 203.2 180)
+		(fields_autoplaced yes)
+		(effects
+			(font
+				(size 1.27 1.27)
+			)
+			(justify right)
+		)
+		(property "Intersheetrefs" "${INTERSHEET_REFS}"
+			(at 141.8811 203.2 0)
+			(effects
+				(font
+					(size 1.27 1.27)
+				)
+				(justify right)
+				(hide yes)
+			)
 		)
 	)
@@
 				(hide yes)
 			)
-		)
-	)
-	(global_label "SYS_RESET"
-		(shape output)
-		(at 152.4 203.2 180)
-		(fields_autoplaced yes)
-		(effects
-			(font
-				(size 1.27 1.27)
-			)
-			(justify right)
-		)
-		(property "Intersheetrefs" "${INTERSHEET_REFS}"
-			(at 139.0994 203.2 0)
-			(effects
-				(font
-					(size 1.27 1.27)
-				)
-				(justify right)
-				(hide yes)
-			)

Commit message: adding NMOS for the POWER
Connections:
- net POWER_EN renamed POWER_BMC
- net RUN_PG renamed RESET_BMC
Changed lines of the file:
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@@
 		)
 	)
-	(global_label "POWER_EN"
+	(global_label "POWER_BMC"
 		(shape output)
 		(at 152.4 200.66 180)
@@
 		)
 		(property "Intersheetrefs" "${INTERSHEET_REFS}"
-			(at 139.4017 200.66 0)
+			(at 137.8898 200.66 0)
 			(effects
 				(font
@@
 		)
 	)
-	(global_label "RUN_PG"
+	(global_label "RESET_BMC"
 		(shape output)
 		(at 152.4 203.2 180)
@@
 		)
 		(property "Intersheetrefs" "${INTERSHEET_REFS}"
-			(at 141.8811 203.2 0)
-			(effects
-				(font
+			(at 138.6156 203.2 0)
+			(effects
+				(font

Commit message: added system reset
Changed lines of the file:
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@@
 	)
 	(global_label "RESET_BMC"
-		(shape output)
+		(shape bidirectional)
 		(at 152.4 203.2 180)
 		(fields_autoplaced yes)
@@
 		)
 		(property "Intersheetrefs" "${INTERSHEET_REFS}"
-			(at 138.6156 203.2 0)
+			(at 137.5996 203.2 0)
 			(effects
 				(font

Commit message: adding shutdown req
Connections:
- net SHUT_REQ_BMC: now reaches J1.233
- no-connect marks 78 -> 77
Other:
- moved on the sheet: J1A, J1B, J1C, J1D, J1E, J1F, J1G

Commit message: fix pin 260 and some other stuff
Connections:
- net +5V: now also J1.260
- no-connect marks 77 -> 76
Other:
- note removed: "<- Mechanical Pin"
Changed lines of the file:
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@@
 	(generator_version "9.0")
 	(paper "A3")
-	(text "<- Mechanical Pin"
-		(exclude_from_sim no)
-		(at 284.988 176.784 0)
-		(effects
-			(font
-				(size 1.27 1.27)
-			)
-		)
-	)
 	(text "< Research cluster board implement"
 		(exclude_from_sim no)
@@
 	)
 	(junction
+		(at 273.05 173.99)
+		(diameter 0)
+		(color 0 0 0 0)
+	)
+	(junction
 		(at 274.32 101.6)
 		(diameter 0)
@@
 	)
 	(no_connect
-		(at 271.78 176.53)
-	)
-	(no_connect
 		(at 316.23 114.3)
 	)
@@
 	(wire
 		(pts
+			(xy 271.78 176.53) (xy 273.05 176.53)
+		)
+		(stroke
+			(width 0)
+			(type default)
+		)
+	)
+	(wire
+		(pts
 			(xy 274.32 158.75) (xy 274.32 161.29)
 		)
@@
 		)
 		(stroke
+			(width 0)
+			(type default)
+		)
+	)
+	(wire
+		(pts
+			(xy 273.05 176.53) (xy 273.05 173.99)
+		)
+		(stroke

Commit message: adding mod_sleep and removing one of the free GPIO's
Connections:
- net MOD_SLEEP: now reaches J1.178
- net GPIO_CLK: no longer names the net of J1.118
Changed lines of the file:
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@@
 	)
 	(no_connect
+		(at 271.78 121.92)
+	)
+	(no_connect
 		(at 191.77 76.2)
 	)
@@
 	)
 	(no_connect
-		(at 111.76 173.99)
-	)
-	(no_connect
 		(at 271.78 88.9)
 	)
@@
 	(wire
 		(pts
+			(xy 116.84 173.99) (xy 111.76 173.99)
+		)
+		(stroke
+			(width 0)
+			(type default)
+		)
+	)
+	(wire
+		(pts
 			(xy 71.12 184.15) (xy 76.2 184.15)
 		)
@@
 	(wire
 		(pts
-			(xy 276.86 121.92) (xy 271.78 121.92)
-		)
-		(stroke
-			(width 0)
-			(type default)
-		)
-	)
-	(wire
-		(pts
 			(xy 196.85 198.12) (xy 191.77 198.12)
 		)
@@
 		)
 	)
+	(global_label "MOD_SLEEP"
+		(shape input)
+		(at 116.84 173.99 0)
+		(fields_autoplaced yes)
+		(effects
+			(font
+				(size 1.27 1.27)
+			)
+			(justify left)
+		)
+		(property "Intersheetrefs" "${INTERSHEET_REFS}"
+			(at 130.7454 173.99 0)
+			(effects
+				(font
+					(size 1.27 1.27)
+				)
+				(justify left)
+				(hide yes)
+			)
+		)
+	)
 	(global_label "UART-0_TX"
 		(shape input)
@@
 				(hide yes)
 			)
-		)
-	)
-	(global_label "GPIO_CLK"
-		(shape input)
-		(at 276.86 121.92 0)
-		(fields_autoplaced yes)
-		(effects
-			(font
-				(size 1.27 1.27)
-			)
-			(justify left)
-		)
-		(property "Intersheetrefs" "${INTERSHEET_REFS}"
-			(at 288.9513 121.92 0)
-			(effects
-				(font
-					(size 1.27 1.27)
-				)
-				(justify left)
-				(hide yes)
-			)

Commit message: all pins used on the GPIO mezzanine finallygit add .!
Connections:
- net GPIO0: now reaches J1.118
- no-connect marks 76 -> 75
Changed lines of the file:
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@@
-	)
-	(no_connect
-		(at 271.78 121.92)
 	)
 	(no_connect
@@
 		(pts
 			(xy 273.05 176.53) (xy 273.05 173.99)
+		)
+		(stroke
+			(width 0)
+			(type default)
+		)
+	)
+	(wire
+		(pts
+			(xy 276.86 121.92) (xy 271.78 121.92)
 		)
 		(stroke
@@
 				(hide yes)
 			)
+		)
+	)
+	(global_label "GPIO0"
+		(shape bidirectional)
+		(at 276.86 121.92 0)
+		(fields_autoplaced yes)
+		(effects
+			(font
+				(size 1.27 1.27)
+			)
+			(justify left)
+		)
+		(property "Intersheetrefs" "${INTERSHEET_REFS}"
+			(at 286.6411 121.92 0)
+			(effects
+				(font
+					(size 1.27 1.27)
+				)
+				(justify left)
+				(hide yes)
+			)
