File: PCB_CARRIER/SO-DIMM.kicad_sch (KiCad schematic)
At the start: 1 part, among them J1 SODIMM-260_Split

Commit message: fully populated all the SODIMM pins FINALLY RAHHH
Connections:
- no-connect marks 75 -> 85
Other:
- note removed: "< Second camera?"
Changed lines of the file:
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@@
-		)
-	)
-	(text "< Second camera?"
-		(exclude_from_sim no)
-		(at 362.712 76.454 0)
-		(effects
-			(font
-				(size 1.27 1.27)
-			)
 		)
 	)
 	(text "Implement on BMC >\n"
 		(exclude_from_sim no)
-		(at 206.248 84.074 0)
+		(at 207.518 83.82 0)
 		(effects
 			(font
@@
 	)
 	(no_connect
+		(at 191.77 167.64)
+	)
+	(no_connect
 		(at 191.77 119.38)
 	)
@@
 	)
 	(no_connect
+		(at 316.23 83.82)
+	)
+	(no_connect
 		(at 191.77 177.8)
 	)
@@
 	)
 	(no_connect
+		(at 191.77 175.26)
+	)
+	(no_connect
 		(at 316.23 111.76)
 	)
 	(no_connect
+		(at 351.79 78.74)
+	)
+	(no_connect
 		(at 316.23 104.14)
 	)
@@
 	)
 	(no_connect
+		(at 351.79 83.82)
+	)
+	(no_connect
 		(at 191.77 182.88)
 	)
@@
 	)
 	(no_connect
+		(at 191.77 187.96)
+	)
+	(no_connect
 		(at 191.77 193.04)
 	)
@@
 	)
 	(no_connect
+		(at 191.77 172.72)
+	)
+	(no_connect
 		(at 351.79 109.22)
 	)
@@
 	)
 	(no_connect
+		(at 351.79 81.28)
+	)
+	(no_connect
 		(at 76.2 88.9)
 	)
@@
 	)
 	(no_connect
+		(at 191.77 160.02)
+	)
+	(no_connect
 		(at 76.2 176.53)
 	)
 	(no_connect
+		(at 351.79 86.36)
+	)
+	(no_connect

Commit message: removing GPIO with camera powerdown, I might want to actually break out some of these used GPIO's to be free io's though
Connections:
- net CSI-0_PWDN: now also J1.120
- net GPIO0: no longer names the net of J1.118
Changed lines of the file:
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@@
 	)
 	(no_connect
+		(at 271.78 121.92)
+	)
+	(no_connect
 		(at 76.2 168.91)
 	)
@@
 	)
 	(no_connect
-		(at 271.78 124.46)
-	)
-	(no_connect
 		(at 271.78 119.38)
 	)
@@
 	(wire
 		(pts
+			(xy 276.86 124.46) (xy 271.78 124.46)
+		)
+		(stroke
+			(width 0)
+			(type default)
+		)
+	)
+	(wire
+		(pts
 			(xy 71.12 116.84) (xy 76.2 116.84)
 		)
@@
 	(wire
 		(pts
-			(xy 276.86 121.92) (xy 271.78 121.92)
-		)
-		(stroke
-			(width 0)
-			(type default)
-		)
-	)
-	(wire
-		(pts
 			(xy 116.84 186.69) (xy 111.76 186.69)
 		)
@@
 		)
 	)
-	(global_label "GPIO0"
-		(shape bidirectional)
-		(at 276.86 121.92 0)
-		(fields_autoplaced yes)
-		(effects
-			(font
-				(size 1.27 1.27)
-			)
-			(justify left)
-		)
-		(property "Intersheetrefs" "${INTERSHEET_REFS}"
-			(at 286.6411 121.92 0)
-			(effects
-				(font
-					(size 1.27 1.27)
-				)
-				(justify left)
-				(hide yes)
-			)
-		)
-	)
 	(global_label "GBE_MDI3_N"
 		(shape bidirectional)
@@
 	)
 	(global_label "CSI-0_PWDN"
-		(shape input)
+		(shape output)
 		(at 276.86 116.84 0)
 		(fields_autoplaced yes)
@@
 			(effects
 				(font
+					(size 1.27 1.27)
+				)
+				(justify left)
+				(hide yes)
+			)
+		)
+	)
+	(global_label "CSI-0_PWDN"
+		(shape output)
+		(at 276.86 124.46 0)
+		(fields_autoplaced yes)
+		(effects
+			(font
+				(size 1.27 1.27)
+			)
+			(justify left)
+		)
+		(property "Intersheetrefs" "${INTERSHEET_REFS}"
+			(at 292.096 124.46 0)
+			(effects
+				(font

Commit message: removed USB VBUS because I'm doing it via BMC and added a general GPIO
Connections:
- net USB_VBUS renamed GPIO0
Other:
- note removed: "Implement on BMC >"
Changed lines of the file:
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@@
 		)
 	)
-	(text "Implement on BMC >\n"
-		(exclude_from_sim no)
-		(at 207.518 83.82 0)
-		(effects
-			(font
-				(size 1.27 1.27)
-			)
-		)
-	)
 	(text "SPI AND OTHERS MIGHT NEED 1.8V INSTEAD OF 3.3V!!!"
 		(exclude_from_sim no)
-		(at 142.748 40.132 0)
+		(at 142.24 56.642 0)
 		(effects
 			(font
@@
 	(wire
 		(pts
+			(xy 231.14 83.82) (xy 236.22 83.82)
+		)
+		(stroke
+			(width 0)
+			(type default)
+		)
+	)
+	(wire
+		(pts
 			(xy 114.3 76.2) (xy 114.3 83.82)
 		)
@@
 	(wire
 		(pts
-			(xy 231.14 83.82) (xy 236.22 83.82)
-		)
-		(stroke
-			(width 0)
-			(type default)
-		)
-	)
-	(wire
-		(pts
 			(xy 276.86 109.22) (xy 271.78 109.22)
 		)
@@
 		)
 	)
-	(global_label "USB_VBUS"
-		(shape input)
-		(at 231.14 83.82 180)
-		(fields_autoplaced yes)
-		(effects
-			(font
-				(size 1.27 1.27)
-			)
-			(justify right)
-		)
-		(property "Intersheetrefs" "${INTERSHEET_REFS}"
-			(at 218.3835 83.82 0)
-			(effects
-				(font
-					(size 1.27 1.27)
-				)
-				(justify right)
-				(hide yes)
-			)
-		)
-	)
 	(global_label "CSI-0_SDA"
 		(shape bidirectional)
@@
 				(hide yes)
 			)
+		)
+	)
+	(global_label "GPIO0"
+		(shape bidirectional)
+		(at 231.14 83.82 180)
+		(fields_autoplaced yes)
+		(effects
+			(font
+				(size 1.27 1.27)
+			)
+			(justify right)
+		)
+		(property "Intersheetrefs" "${INTERSHEET_REFS}"
+			(at 221.3589 83.82 0)
+			(effects
+				(font
+					(size 1.27 1.27)
+				)
+				(justify right)
+				(hide yes)
+			)

Commit message: fixed camera power pins, oops, researching a lot about level shifting
Connections:
- net CSI-0_PWDN: no longer J1.120
- new net CSI-1_PWDN: J1.120
Changed lines of the file:
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@@
 		)
 	)
-	(global_label "CSI-0_PWDN"
+	(global_label "CSI-1_PWDN"
 		(shape output)
 		(at 276.86 124.46 0)

Commit message: labelling SPI bidirectional, this is really cooking my head
Other:
- note added: "SPI multiplexed Master/Slave"
- note removed: "SPI AND OTHERS MIGHT NEED 1.8V INSTEAD OF 3.3V!!!"
Changed lines of the file:
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@@
 		)
 	)
-	(text "SPI AND OTHERS MIGHT NEED 1.8V INSTEAD OF 3.3V!!!"
+	(text "SPI multiplexed\nMaster/Slave"
 		(exclude_from_sim no)
-		(at 142.24 56.642 0)
+		(at 208.026 92.456 0)
 		(effects
 			(font
@@
 	)
 	(global_label "SPI-0_CS0"
-		(shape input)
+		(shape bidirectional)
 		(at 231.14 93.98 180)
 		(fields_autoplaced yes)
@@
 		)
 		(property "Intersheetrefs" "${INTERSHEET_REFS}"
-			(at 217.5369 93.98 0)
+			(at 216.5209 93.98 0)
 			(effects
 				(font
@@
 	)
 	(global_label "SPI-1_CLK"
-		(shape input)
+		(shape bidirectional)
 		(at 276.86 106.68 0)
 		(fields_autoplaced yes)
@@
 		)
 		(property "Intersheetrefs" "${INTERSHEET_REFS}"
-			(at 290.3422 106.68 0)
+			(at 291.3582 106.68 0)
 			(effects
 				(font
@@
 	)
 	(global_label "SPI-0_CS1"
-		(shape input)
+		(shape bidirectional)
 		(at 231.14 96.52 180)
 		(fields_autoplaced yes)
@@
 		)
 		(property "Intersheetrefs" "${INTERSHEET_REFS}"
-			(at 217.5369 96.52 0)
+			(at 216.5209 96.52 0)
 			(effects
 				(font
@@
 	)
 	(global_label "SPI-1_CS0"
-		(shape input)
+		(shape bidirectional)
 		(at 276.86 111.76 0)
 		(fields_autoplaced yes)
@@
 		)
 		(property "Intersheetrefs" "${INTERSHEET_REFS}"
-			(at 290.4631 111.76 0)
+			(at 291.4791 111.76 0)
 			(effects
 				(font
@@
 	)
 	(global_label "SPI-0_MOSI"
-		(shape input)
+		(shape bidirectional)
 		(at 231.14 86.36 180)
 		(fields_autoplaced yes)
@@
 		)
 		(property "Intersheetrefs" "${INTERSHEET_REFS}"
-			(at 216.6297 86.36 0)
+			(at 215.6137 86.36 0)
 			(effects
 				(font
@@
 	)
 	(global_label "SPI-1_MISO"
-		(shape output)
+		(shape bidirectional)
 		(at 276.86 109.22 0)
 		(fields_autoplaced yes)
@@
 		)
 		(property "Intersheetrefs" "${INTERSHEET_REFS}"
-			(at 291.3703 109.22 0)
+			(at 292.3863 109.22 0)
 			(effects
 				(font
@@
 	)
 	(global_label "SPI-1_MOSI"
-		(shape input)
+		(shape bidirectional)
 		(at 276.86 104.14 0)
 		(fields_autoplaced yes)
@@
 		)
 		(property "Intersheetrefs" "${INTERSHEET_REFS}"
-			(at 291.3703 104.14 0)
+			(at 292.3863 104.14 0)
 			(effects
 				(font
@@
 	)
 	(global_label "SPI-0_CLK"
-		(shape input)
+		(shape bidirectional)
 		(at 231.14 88.9 180)
 		(fields_autoplaced yes)
@@
 		)
 		(property "Intersheetrefs" "${INTERSHEET_REFS}"
-			(at 217.6578 88.9 0)
+			(at 216.6418 88.9 0)
 			(effects
 				(font
@@
 	)
 	(global_label "SPI-0_MISO"
-		(shape output)
+		(shape bidirectional)
 		(at 231.14 91.44 180)
 		(fields_autoplaced yes)
@@
 		)
 		(property "Intersheetrefs" "${INTERSHEET_REFS}"
-			(at 216.6297 91.44 0)
+			(at 215.6137 91.44 0)
 			(effects
 				(font
@@
 	)
 	(global_label "SPI-1_CS1"
-		(shape input)
+		(shape bidirectional)
 		(at 276.86 114.3 0)
 		(fields_autoplaced yes)
@@
 		)
 		(property "Intersheetrefs" "${INTERSHEET_REFS}"
-			(at 290.4631 114.3 0)
+			(at 291.4791 114.3 0)
 			(effects
 				(font

Commit message: fixing SPI label direction, and changing level shifting
Changed lines of the file:
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@@
 	)
 	(global_label "SPI-0_CS0"
-		(shape bidirectional)
+		(shape input)
 		(at 231.14 93.98 180)
 		(fields_autoplaced yes)
@@
 		)
 		(property "Intersheetrefs" "${INTERSHEET_REFS}"
-			(at 216.5209 93.98 0)
+			(at 217.5369 93.98 0)
 			(effects
 				(font
@@
 	)
 	(global_label "SPI-1_CLK"
-		(shape bidirectional)
+		(shape input)
 		(at 276.86 106.68 0)
 		(fields_autoplaced yes)
@@
 		)
 		(property "Intersheetrefs" "${INTERSHEET_REFS}"
-			(at 291.3582 106.68 0)
+			(at 290.3422 106.68 0)
 			(effects
 				(font
@@
 	)
 	(global_label "SPI-0_CS1"
-		(shape bidirectional)
+		(shape input)
 		(at 231.14 96.52 180)
 		(fields_autoplaced yes)
@@
 		)
 		(property "Intersheetrefs" "${INTERSHEET_REFS}"
-			(at 216.5209 96.52 0)
+			(at 217.5369 96.52 0)
 			(effects
 				(font
@@
 	)
 	(global_label "SPI-1_CS0"
-		(shape bidirectional)
+		(shape input)
 		(at 276.86 111.76 0)
 		(fields_autoplaced yes)
@@
 		)
 		(property "Intersheetrefs" "${INTERSHEET_REFS}"
-			(at 291.4791 111.76 0)
+			(at 290.4631 111.76 0)
 			(effects
 				(font
@@
 	)
 	(global_label "SPI-0_MOSI"
-		(shape bidirectional)
+		(shape input)
 		(at 231.14 86.36 180)
 		(fields_autoplaced yes)
@@
 		)
 		(property "Intersheetrefs" "${INTERSHEET_REFS}"
-			(at 215.6137 86.36 0)
+			(at 216.6297 86.36 0)
 			(effects
 				(font
@@
 	)
 	(global_label "SPI-1_MISO"
-		(shape bidirectional)
+		(shape output)
 		(at 276.86 109.22 0)
 		(fields_autoplaced yes)
@@
 		)
 		(property "Intersheetrefs" "${INTERSHEET_REFS}"
-			(at 292.3863 109.22 0)
+			(at 291.3703 109.22 0)
 			(effects
 				(font
@@
 	)
 	(global_label "SPI-1_MOSI"
-		(shape bidirectional)
+		(shape input)
 		(at 276.86 104.14 0)
 		(fields_autoplaced yes)
@@
 		)
 		(property "Intersheetrefs" "${INTERSHEET_REFS}"
-			(at 292.3863 104.14 0)
+			(at 291.3703 104.14 0)
 			(effects
 				(font
@@
 	)
 	(global_label "SPI-0_CLK"
-		(shape bidirectional)
+		(shape input)
 		(at 231.14 88.9 180)
 		(fields_autoplaced yes)
@@
 		)
 		(property "Intersheetrefs" "${INTERSHEET_REFS}"
-			(at 216.6418 88.9 0)
+			(at 217.6578 88.9 0)
 			(effects
 				(font
@@
 	)
 	(global_label "SPI-0_MISO"
-		(shape bidirectional)
+		(shape output)
 		(at 231.14 91.44 180)
 		(fields_autoplaced yes)
@@
 		)
 		(property "Intersheetrefs" "${INTERSHEET_REFS}"
-			(at 215.6137 91.44 0)
+			(at 216.6297 91.44 0)
 			(effects
 				(font
@@
 	)
 	(global_label "SPI-1_CS1"
-		(shape bidirectional)
+		(shape input)
 		(at 276.86 114.3 0)
 		(fields_autoplaced yes)
@@
 		)
 		(property "Intersheetrefs" "${INTERSHEET_REFS}"
-			(at 291.4791 114.3 0)
-			(effects
-				(font
+			(at 290.4631 114.3 0)
+			(effects
+				(font

Commit message: fixed SPI, mislabelled some stuff
Connections:
- net SPI-0_CLK renamed SPI-0_CLK_1V8
- net SPI-0_CS0 renamed SPI-0_CS0_1V8
- net SPI-0_CS1 renamed SPI-0_CS1_1V8
- net SPI-0_MISO renamed SPI-0_MISO_1V8
- net SPI-0_MOSI renamed SPI-0_MOSI_1V8
- net SPI-1_CLK renamed SPI-1_CLK_1V8
- net SPI-1_CS0 renamed SPI-1_CS0_1V8
- net SPI-1_CS1 renamed SPI-1_CS1_1V8
- net SPI-1_MISO renamed SPI-1_MISO_1V8
- net SPI-1_MOSI renamed SPI-1_MOSI_1V8
Changed lines of the file:
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@@
 	(text "SPI multiplexed\nMaster/Slave"
 		(exclude_from_sim no)
-		(at 208.026 92.456 0)
+		(at 204.978 92.71 0)
 		(effects
 			(font
@@
 		)
 	)
-	(global_label "SPI-0_CS0"
+	(global_label "SPI-0_CS0_1V8"
 		(shape input)
 		(at 231.14 93.98 180)
@@
 		)
 		(property "Intersheetrefs" "${INTERSHEET_REFS}"
-			(at 217.5369 93.98 0)
+			(at 213.0617 93.98 0)
 			(effects
 				(font
@@
 		)
 	)
-	(global_label "SPI-1_CLK"
+	(global_label "SPI-1_CLK_1V8"
 		(shape input)
 		(at 276.86 106.68 0)
@@
 		)
 		(property "Intersheetrefs" "${INTERSHEET_REFS}"
-			(at 290.3422 106.68 0)
+			(at 294.8174 106.68 0)
 			(effects
 				(font
@@
 		)
 	)
-	(global_label "SPI-0_CS1"
+	(global_label "SPI-0_CS1_1V8"
 		(shape input)
 		(at 231.14 96.52 180)
@@
 		)
 		(property "Intersheetrefs" "${INTERSHEET_REFS}"
-			(at 217.5369 96.52 0)
+			(at 213.0617 96.52 0)
 			(effects
 				(font
@@
 		)
 	)
-	(global_label "SPI-1_CS0"
+	(global_label "SPI-1_CS0_1V8"
 		(shape input)
 		(at 276.86 111.76 0)
@@
 		)
 		(property "Intersheetrefs" "${INTERSHEET_REFS}"
-			(at 290.4631 111.76 0)
+			(at 294.9383 111.76 0)
 			(effects
 				(font
@@
 		)
 	)
-	(global_label "SPI-0_MOSI"
+	(global_label "SPI-0_MOSI_1V8"
 		(shape input)
 		(at 231.14 86.36 180)
@@
 		)
 		(property "Intersheetrefs" "${INTERSHEET_REFS}"
-			(at 216.6297 86.36 0)
+			(at 212.1545 86.36 0)
 			(effects
 				(font
@@
 		)
 	)
-	(global_label "SPI-1_MISO"
+	(global_label "SPI-1_MISO_1V8"
 		(shape output)
 		(at 276.86 109.22 0)
@@
 		)
 		(property "Intersheetrefs" "${INTERSHEET_REFS}"
-			(at 291.3703 109.22 0)
+			(at 295.8455 109.22 0)
 			(effects
 				(font
@@
 		)
 	)
-	(global_label "SPI-1_MOSI"
+	(global_label "SPI-1_MOSI_1V8"
 		(shape input)
 		(at 276.86 104.14 0)
@@
 		)
 		(property "Intersheetrefs" "${INTERSHEET_REFS}"
-			(at 291.3703 104.14 0)
+			(at 295.8455 104.14 0)
 			(effects
 				(font
@@
 		)
 	)
-	(global_label "SPI-0_CLK"
+	(global_label "SPI-0_CLK_1V8"
 		(shape input)
 		(at 231.14 88.9 180)
@@
 		)
 		(property "Intersheetrefs" "${INTERSHEET_REFS}"
-			(at 217.6578 88.9 0)
+			(at 213.1826 88.9 0)
 			(effects
 				(font
@@
 		)
 	)
-	(global_label "SPI-0_MISO"
+	(global_label "SPI-0_MISO_1V8"
 		(shape output)
 		(at 231.14 91.44 180)
@@
 		)
 		(property "Intersheetrefs" "${INTERSHEET_REFS}"
-			(at 216.6297 91.44 0)
+			(at 212.1545 91.44 0)
 			(effects
 				(font
@@
 		)
 	)
-	(global_label "SPI-1_CS1"
+	(global_label "SPI-1_CS1_1V8"
 		(shape input)
 		(at 276.86 114.3 0)
@@
 		)
 		(property "Intersheetrefs" "${INTERSHEET_REFS}"
-			(at 290.4631 114.3 0)
+			(at 294.9383 114.3 0)
 			(effects
 				(font

Commit message: re-naming all UART signals for shifting preparation
Connections:
- net UART-0_CTS renamed UART-0_CTS_1V8
- net UART-0_RTS renamed UART-0_RTS_1V8
- net UART-0_RX renamed UART-0_RX_1V8
- net UART-0_TX renamed UART-0_TX_1V8
- net UART-1_CTS renamed UART-1_CTS_1V8
- net UART-1_RTS renamed UART-1_RTS_1V8
- net UART-1_RX renamed UART-1_RX_1V8
- net UART-1_TX renamed UART-1_TX_1V8
- net UART-2_RX renamed UART-2_RX_1V8
- net UART-2_TX renamed UART-2_TX_1V8
Other:
- moved on the sheet: J1A, J1B, J1C, J1D, J1E, J1F, J1G
