File: PCB_CARRIER/cm4-gpio.kicad_sch (KiCad schematic)
At the start: 17 parts, among them J2 Micro_SD_Card_Det2, Q1 NMOS, SW1 SW_Push, U1 RT9742GGJ5

Commit message: adding NMOS for the POWER
Parts:
- added Q2: BSS138, symbol Simulation_SPICE:NMOS
- added R4: 110, symbol Device:R
- added SW2: TS-1088, https://jlcpcb.com/api/file/downloadByFileSystemAccessId/8588886944068096000, symbol Switch:SW_Push
- Q1: value NMOS -> BSS138
- SW1: value SW_Push -> TS-1088; footprint (none) -> https://jlcpcb.com/api/file/downloadByFileSystemAccessId/8588886944068096000
Connections:
- net GND: now also Q2.3 (S), SW2.2
- net POWER_EN: no longer names the net of Module1.99 (Global_EN)
- net POWER_EN: now also Q2.1 (D), SW2.1
- net PWR_GPIO renamed RESET_BMC
- new net: Q2.2 (G), R4.1
- new net POWER_BMC: R4.2
Other:
- moved on the sheet: SW1

Commit message: added hiearchial sheet for NMOS
Parts:
- removed Q1, Q2: BSS138, symbol Simulation_SPICE:NMOS
- removed R3, R4: 110, symbol Device:R
- removed SW1, SW2: TS-1088, https://jlcpcb.com/api/file/downloadByFileSystemAccessId/8588886944068096000, symbol Switch:SW_Push
Connections:
- net NMOS BMC Switch/OUTPUT: now reaches Module1.92 (RUN_PG)
- net NMOS BMC Switch1/OUTPUT: now reaches Module1.99 (Global_EN)
Other:
- added sheet NMOS BMC Switch (nmos.kicad_sch)
- added sheet NMOS BMC Switch1 (nmos.kicad_sch)

Commit message: nRPI boot wiring
Parts:
- added SW2: TS-1088, https://jlcpcb.com/api/file/downloadByFileSystemAccessId/8588886944068096000, symbol Switch:SW_Push
Connections:
- net GND: now also SW2.2
- net at Module1.93 (nRPIBOOT): now also SW2.1
Other:
- note added: "< As many 0.1uF as can fit, a 10uF/1uF for bulk"
- note removed: "As many 0.1uF as can fit, a 10uF/1uF for bulk"
Changed lines of the file:
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@@
 		)
 	)
-	(text "As many 0.1uF as can fit, a 10uF/1uF for bulk"
+	(text "< As many 0.1uF as can fit, a 10uF/1uF for bulk"
 		(exclude_from_sim no)
-		(at 166.116 147.574 0)
+		(at 211.328 138.684 0)
 		(effects
 			(font
@@
 	(wire
 		(pts
+			(xy 135.89 162.56) (xy 144.78 162.56)
+		)
+		(stroke
+			(width 0)
+			(type default)
+		)
+	)
+	(wire
+		(pts
 			(xy 140.97 101.6) (xy 135.89 101.6)
 		)
@@
 	(wire
 		(pts
+			(xy 156.21 154.94) (xy 154.94 154.94)
+		)
+		(stroke
+			(width 0)
+			(type default)
+		)
+	)
+	(wire
+		(pts
 			(xy 140.97 93.98) (xy 135.89 93.98)
 		)
@@
 	(wire
 		(pts
+			(xy 40.64 152.4) (xy 41.91 152.4)
+		)
+		(stroke
+			(width 0)
+			(type default)
+		)
+	)
+	(wire
+		(pts
 			(xy 142.24 142.24) (xy 148.59 142.24)
 		)
@@
 	(wire
 		(pts
-			(xy 135.89 162.56) (xy 144.78 162.56)
-		)
-		(stroke
-			(width 0)
-			(type default)
-		)
-	)
-	(wire
-		(pts
 			(xy 137.16 134.62) (xy 142.24 134.62)
 		)
@@
 	(wire
 		(pts
-			(xy 165.1 162.56) (xy 163.83 162.56)
-		)
-		(stroke
-			(width 0)
-			(type default)
-		)
-	)
-	(wire
-		(pts
 			(xy 217.17 95.25) (xy 218.44 95.25)
 		)
@@
 	(wire
 		(pts
-			(xy 40.64 152.4) (xy 41.91 152.4)
-		)
-		(stroke
-			(width 0)
-			(type default)
-		)
-	)
-	(wire
-		(pts
 			(xy 72.39 45.72) (xy 74.93 45.72)
 		)
@@
 	(wire
 		(pts
+			(xy 165.1 162.56) (xy 163.83 162.56)
+		)
+		(stroke
+			(width 0)
+			(type default)
+		)
+	)
+	(wire
+		(pts
 			(xy 73.66 142.24) (xy 74.93 142.24)
 		)
@@
 	(wire
 		(pts
+			(xy 135.89 154.94) (xy 144.78 154.94)
+		)
+		(stroke
+			(width 0)
+			(type default)
+		)
+	)
+	(wire
+		(pts
 			(xy 72.39 38.1) (xy 72.39 45.72)
 		)
@@
 	)
 	(symbol
+		(lib_id "Switch:SW_Push")
+		(at 149.86 154.94 0)
+		(unit 1)
+		(exclude_from_sim no)
+		(in_bom yes)
+		(on_board yes)
+		(dnp no)
+		(property "Reference" "SW2"
+			(at 149.86 156.718 0)
+			(effects
+				(font
+					(size 1.27 1.27)
+				)
+			)
+		)
+		(property "Value" "TS-1088"
+			(at 149.86 150.622 0)
+			(effects
+				(font
+					(size 1.143 1.143)
+				)
+			)
+		)
+		(property "Footprint" "https://jlcpcb.com/api/file/downloadByFileSystemAccessId/8588886944068096000"
+			(at 149.86 149.86 0)
+			(effects
+				(font
+					(size 1.27 1.27)
+				)
+				(hide yes)
+			)
+		)
+		(property "Datasheet" "~"
+			(at 149.86 149.86 0)
+			(effects
+				(font
+					(size 1.27 1.27)
+				)
+				(hide yes)
+			)
+		)
+		(property "Description" "Push button switch, generic, two pins"
+			(at 149.86 154.94 0)
+			(effects
+				(font
+					(size 1.27 1.27)
+				)
+				(hide yes)
+			)
+		)
+		(pin "2"
+		)
+		(pin "1"
+		)
+		(instances
+			(project "carrier"
+				(path "/f52509e6-8053-454c-b8e9-3e2670c5a5fe/fc4c71a5-1008-4ac4-98db-57c838c57d91"
+					(reference "SW2")
+					(unit 1)
+				)
+			)
+		)
+	)
+	(symbol
 		(lib_id "power:GND")
 		(at 72.39 167.64 0)
@@
 	)
 	(symbol
+		(lib_id "power:GND")
+		(at 156.21 154.94 0)
+		(unit 1)
+		(exclude_from_sim no)
+		(in_bom yes)
+		(on_board yes)
+		(dnp no)
+		(property "Reference" "#PWR026"
+			(at 156.21 161.29 0)
+			(effects
+				(font
+					(size 1.27 1.27)
+				)
+				(hide yes)
+			)
+		)
+		(property "Value" "GND"
+			(at 160.02 156.718 0)
+			(effects
+				(font
+					(size 1.27 1.27)
+				)
+			)
+		)
+		(property "Footprint" ""
+			(at 156.21 154.94 0)
+			(effects
+				(font
+					(size 1.27 1.27)
+				)
+				(hide yes)
+			)
+		)
+		(property "Datasheet" ""
+			(at 156.21 154.94 0)
+			(effects
+				(font
+					(size 1.27 1.27)
+				)
+				(hide yes)
+			)
+		)
+		(property "Description" "Power symbol creates a global label with name \"GND\" , ground"
+			(at 156.21 154.94 0)
+			(effects
+				(font
+					(size 1.27 1.27)
+				)
+				(hide yes)
+			)
+		)
+		(pin "1"
+		)
+		(instances
+			(project ""
+				(path "/f52509e6-8053-454c-b8e9-3e2670c5a5fe/fc4c71a5-1008-4ac4-98db-57c838c57d91"
+					(reference "#PWR026")
+					(unit 1)
+				)
+			)
+		)
+	)
+	(symbol
 		(lib_id "Device:C")
 		(at 142.24 138.43 0)
@@
 	)
 	(sheet
-		(at 144.78 158.75)
-		(size 19.05 7.62)
+		(at 144.78 160.02)
+		(size 19.05 5.08)
 		(exclude_from_sim no)
 		(in_bom yes)
 		(on_board yes)
 		(dnp no)
-		(fields_autoplaced yes)
 		(stroke
 			(width 0.1524)
@@
 		)
 		(property "Sheetname" "NMOS BMC Switch1"
-			(at 144.78 158.0384 0)
+			(at 144.78 169.418 0)
 			(effects
 				(font
@@
 		)
 		(property "Sheetfile" "nmos.kicad_sch"
-			(at 144.78 166.9546 0)
+			(at 144.78 165.6846 0)
 			(effects
 				(font
@@
 	)
 	(sheet
-		(at 41.91 148.59)
-		(size 19.05 7.62)
+		(at 41.91 149.86)
+		(size 19.05 5.08)
 		(exclude_from_sim no)
 		(in_bom yes)
@@
 		)
 		(property "Sheetname" "NMOS BMC Switch"
-			(at 41.91 147.8784 0)
+			(at 41.91 149.1484 0)
 			(effects
 				(font
@@
 		)
 		(property "Sheetfile" "nmos.kicad_sch"
-			(at 41.91 156.7946 0)
+			(at 41.91 155.5246 0)
 			(effects
 				(font

Commit message: adding global button for all 4 NMOS's
Parts:
- removed SW2: TS-1088, https://jlcpcb.com/api/file/downloadByFileSystemAccessId/8588886944068096000, symbol Switch:SW_Push
- added SW4: SW_DIP_x04, symbol Switch:SW_DIP_x04
Connections:
- net GND: now also SW4.1, SW4.2, SW4.3, SW4.4
- net nRPIBOOT: now reaches Module1.93 (nRPIBOOT)
- net nRPIBOOT: now also SW4.6
- net NMOS BMC Switch/OUTPUT renamed RUN_PG
- net RUN_PG: now also SW4.8
- net NMOS BMC Switch1/OUTPUT renamed PMIC_EN
- net PMIC_EN: now also SW4.7
Other:
- moved on the sheet: C1, C11, C12, C2, C4, C5, C6, C7, D1, J2, Module1A, R1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

Commit message: adding EEPROM_nWP
Connections:
- net EEPROM_nWP: now reaches Module1.20 (EEPROM_nWP)
- net EEPROM_nWP: now also SW4.5
- no-connect marks 5 -> 4
Other:
- moved on the sheet: C1, C11, C12, C2, C4, C5, C6, C7, D1, J2, Module1A, R1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

Commit message: remapping reset, not done yet
Connections:
- net RUN_PG renamed PWR_Button
Other:
- removed sheet NMOS BMC Switch
Changed lines of the file:
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@@
 	)
 	(junction
-		(at 55.88 147.32)
-		(diameter 0)
-		(color 0 0 0 0)
-	)
-	(junction
 		(at 165.1 137.16)
 		(diameter 0)
@@
 	(wire
 		(pts
-			(xy 55.88 147.32) (xy 66.04 147.32)
+			(xy 60.96 147.32) (xy 66.04 147.32)
 		)
 		(stroke
@@
 	(wire
 		(pts
-			(xy 31.75 147.32) (xy 33.02 147.32)
-		)
-		(stroke
-			(width 0)
-			(type default)
-		)
-	)
-	(wire
-		(pts
 			(xy 133.35 137.16) (xy 139.7 137.16)
 		)
@@
 	(wire
 		(pts
-			(xy 52.07 147.32) (xy 55.88 147.32)
-		)
-		(stroke
-			(width 0)
-			(type default)
-		)
-	)
-	(wire
-		(pts
 			(xy 63.5 71.12) (xy 63.5 83.82)
 		)
@@
 	(wire
 		(pts
-			(xy 55.88 149.86) (xy 55.88 147.32)
-		)
-		(stroke
-			(width 0)
-			(type default)
-		)
-	)
-	(wire
-		(pts
 			(xy 127 58.42) (xy 144.78 58.42)
 		)
@@
 		)
 	)
-	(global_label "RUN_PG"
-		(shape output)
-		(at 104.14 173.99 0)
+	(global_label "PMIC_EN"
+		(shape input)
+		(at 135.89 160.02 270)
 		(fields_autoplaced yes)
 		(effects
@@
 				(size 1.27 1.27)
 			)
-			(justify left)
+			(justify right)
 		)
 		(property "Intersheetrefs" "${INTERSHEET_REFS}"
-			(at 114.6589 173.99 0)
+			(at 135.89 171.1436 90)
 			(effects
 				(font
 					(size 1.27 1.27)
 				)
-				(justify left)
+				(justify right)
 				(hide yes)
 			)
 		)
 	)
-	(global_label "PMIC_EN"
-		(shape input)
-		(at 135.89 160.02 270)
+	(global_label "SD_DAT3"
+		(shape bidirectional)
+		(at 132.08 109.22 0)
 		(fields_autoplaced yes)
 		(effects
@@
 				(size 1.27 1.27)
 			)
-			(justify right)
+			(justify left)
 		)
 		(property "Intersheetrefs" "${INTERSHEET_REFS}"
-			(at 135.89 171.1436 90)
+			(at 144.1591 109.22 0)
 			(effects
 				(font
 					(size 1.27 1.27)
 				)
-				(justify right)
+				(justify left)
 				(hide yes)
 			)
 		)
 	)
-	(global_label "SD_DAT3"
+	(global_label "GBE_MDI3_P"
 		(shape bidirectional)
-		(at 132.08 109.22 0)
+		(at 132.08 35.56 0)
 		(fields_autoplaced yes)
 		(effects
@@
 		)
 		(property "Intersheetrefs" "${INTERSHEET_REFS}"
-			(at 144.1591 109.22 0)
+			(at 147.6062 35.56 0)
 			(effects
 				(font
@@
 		)
 	)
-	(global_label "GBE_MDI3_P"
-		(shape bidirectional)
-		(at 132.08 35.56 0)
+	(global_label "PWR_Button"
+		(shape output)
+		(at 104.14 173.99 0)
 		(fields_autoplaced yes)
 		(effects
@@
 		)
 		(property "Intersheetrefs" "${INTERSHEET_REFS}"
-			(at 147.6062 35.56 0)
+			(at 118.3477 173.99 0)
 			(effects
 				(font
@@
 		)
 	)
-	(global_label "RESET_BMC"
-		(shape input)
-		(at 31.75 147.32 180)
-		(fields_autoplaced yes)
-		(effects
-			(font
-				(size 1.27 1.27)
-			)
-			(justify right)
-		)
-		(property "Intersheetrefs" "${INTERSHEET_REFS}"
-			(at 17.9656 147.32 0)
-			(effects
-				(font
-					(size 1.27 1.27)
-				)
-				(justify right)
-				(hide yes)
-			)
-		)
-	)
 	(global_label "GBE_MDI0_N"
 		(shape bidirectional)
@@
 		)
 	)
-	(global_label "RUN_PG"
+	(global_label "PWR_Button"
 		(shape input)
-		(at 55.88 149.86 270)
+		(at 60.96 147.32 180)
 		(fields_autoplaced yes)
 		(effects
@@
 		)
 		(property "Intersheetrefs" "${INTERSHEET_REFS}"
-			(at 55.88 160.3789 90)
+			(at 46.7523 147.32 0)
 			(effects
 				(font
@@
 		)
 		(property "Sheetname" "NMOS BMC Switch1"
-			(at 138.43 164.338 0)
+			(at 138.43 154.432 0)
 			(effects
 				(font
@@
 				)
 			)
-		)
-	)
-	(sheet
-		(at 33.02 144.78)
-		(size 19.05 5.08)
-		(exclude_from_sim no)
-		(in_bom yes)
-		(on_board yes)
-		(dnp no)
-		(fields_autoplaced yes)
-		(stroke
-			(width 0.1524)
-			(type solid)
-		)
-		(fill
-			(color 0 0 0 0.0000)
-		)
-		(property "Sheetname" "NMOS BMC Switch"
-			(at 33.02 144.0684 0)
-			(effects
-				(font
-					(size 1.27 1.27)
-				)
-				(justify left bottom)
-			)
-		)
-		(property "Sheetfile" "nmos.kicad_sch"
-			(at 33.02 150.4446 0)
-			(effects
-				(font
-					(size 1.27 1.27)
-				)
-				(justify left top)
-			)
-		)
-		(pin "INPUT" input
-			(at 33.02 147.32 180)
-			(effects
-				(font
-					(size 1.27 1.27)
-				)
-				(justify left)
-			)
-		)
-		(pin "OUTPUT" output
-			(at 52.07 147.32 0)
-			(effects
-				(font
-					(size 1.27 1.27)
-				)
-				(justify right)
-			)
-		)
-		(instances
-			(project "carrier"
-				(path "/f52509e6-8053-454c-b8e9-3e2670c5a5fe/fc4c71a5-1008-4ac4-98db-57c838c57d91"
-					(page "5")
-				)
-			)

Commit message: removing the NMOS component, this is going to be a large revamp..
Parts:
- added Q1: BSS138, symbol Simulation_SPICE:NMOS
- added R3: 100, symbol Device:R
- added R4: 100K, symbol Device:R
Connections:
- net GND: now also Q1.3 (S), R4.2
- net PMIC_EN: now also Q1.1 (D)
- net POWER_BMC: now also R3.2
- new net: Q1.2 (G), R3.1, R4.1
Other:
- removed sheet NMOS BMC Switch1
- moved on the sheet: C12, J2, R2, U1

Commit message: added system reset
Parts:
- added Q2: BSS138, symbol Simulation_SPICE:NMOS
- added R5: 10K, symbol Device:R
- added R6: 100, symbol Device:R
Connections:
- net +1V8: now also R5.1
- net GND: now also Q2.3 (S)
- net ACTIVITY_LED: now reaches D1.1 (K), Module1.21 (PI_nLED_Activity)
- net SYS_RESET: now reaches Module1.41 (GPIO25)
- net SYS_RESET: now also R6.1
- new net: Q2.2 (G), R6.2
- new net RESET_BMC: Q2.1 (D), R5.2
Other:
- note added: "BMC Power Switch"
- moved on the sheet: C1, C11, C12, C2, C4, C5, C6, C7, D1, J2, Module1A, Q1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
