File: PCB_CARRIER/cm4-gpio.kicad_sch (KiCad schematic)
At the start: 35 parts, among them J2 Micro_SD_Card_Det2, Q1 BSS138, Q2 BSS138, Q3 BSS138, Q4 BC817-40, SW1 SW_DIP_x04, U4 RT9742GGJ5

Commit message: fixing the mosfet logic on PMIC_EN
Parts:
- R12: value 5K -> 10K
- R13: value 100 -> 10K
Connections:
- net +3V3: now also Q3.2 (G), R13.1
- net GND: no longer Q3.3 (S)
- net PMIC_EN: now also Q3.3 (S), R13.2
- net SHUTDOWN_REQ: no longer R13.2
Other:
- note added: "Shift 5V Shutdown Req to 3V3 Shutdown!"
- moved on the sheet: Q3, R12

Commit message: fixed logic on both PCB and schematic :D
Parts:
- R12, R13: value 10K -> 5K
Connections:
- net SHUTDOWN_REQ: no longer names the net of Module1.29 (GPIO16)
Changed lines of the file:
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@@
 	(text "Shift 5V Shutdown Req to 3V3 Shutdown!"
 		(exclude_from_sim no)
-		(at 57.15 165.862 0)
+		(at 57.15 166.37 0)
 		(effects
 			(font
@@
 	(wire
 		(pts
-			(xy 209.55 120.65) (xy 204.47 120.65)
-		)
-		(stroke
-			(width 0)
-			(type default)
-		)
-	)
-	(wire
-		(pts
 			(xy 143.51 196.85) (xy 142.24 196.85)
 		)
@@
 		)
 	)
-	(global_label "SHUTDOWN_REQ"
-		(shape output)
-		(at 209.55 120.65 0)
-		(fields_autoplaced yes)
-		(effects
-			(font
-				(size 1.27 1.27)
-			)
-			(justify left)
-		)
-		(property "Intersheetrefs" "${INTERSHEET_REFS}"
-			(at 227.5679 120.65 0)
-			(effects
-				(font
-					(size 1.27 1.27)
-				)
-				(justify left)
-				(hide yes)
-			)
-		)
-	)
 	(global_label "CSI-0_SCL"
 		(shape bidirectional)
@@
 			)
 		)
-		(property "Value" "10K"
+		(property "Value" "5K"
 			(at 46.99 182.8799 0)
 			(effects
@@
 			)
 		)
-		(property "Value" "10K"
+		(property "Value" "5K"
 			(at 70.866 182.88 0)
 			(effects

Commit message: fixing another mosfet
Parts:
- removed Q2: BSS138, Package_TO_SOT_SMD:SOT-23-3, symbol Simulation_SPICE:NMOS
- removed R10: 10K, Resistor_SMD:R_0402_1005Metric, symbol Device:R
- removed R11: 100, Resistor_SMD:R_0402_1005Metric, symbol Device:R
- added Q5: BSS138, Package_TO_SOT_SMD:SOT-23-3, symbol Simulation_SPICE:NMOS
- added R24: 10K, Resistor_SMD:R_0402_1005Metric, symbol Device:R
- added R25: 5K, Resistor_SMD:R_0402_1005Metric, symbol Device:R
Connections:
- net RESET_Button is gone; now on net SYS_RESET: SW1.5
- net +1V8: now also R24.1
- net +3V3: now also Q5.2 (G), R25.1
- net RESET_BMC: now also Q5.1 (D), R24.2
- net SYS_RESET: now also Q5.3 (S), R25.2
Other:
- note added: "No Reset Button on CM5, but programmable through GPIO!"

Commit message: hopping off, mosfet logic is still wrong I think
Other:
- note added: "Carrier drives module"
- note added: "Module drives carrier"
Changed lines of the file:
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@@
+		)
+	)
+	(text "Carrier drives module"
+		(exclude_from_sim no)
+		(at -11.684 94.742 0)
+		(effects
+			(font
+				(size 1.27 1.27)
+			)
 		)
 	)
@@
 		(effects
 			(font
+				(size 1.27 1.27)
+			)
+		)
+	)
+	(text "Module drives carrier"
+		(exclude_from_sim no)
+		(at -11.684 179.324 0)
+		(effects
+			(font

Commit message: fixed shutdown logic
Parts:
- R13: value 5K -> 10K
Connections:
- net PMIC_EN: no longer Q3.3 (S), R13.2
- net MOD_PWR_REQ: now reaches Module1.29 (GPIO16)
- net MOD_PWR_REQ: now also Q3.3 (S), R13.2
Other:
- note added: "Shift 5V Shutdown Req to 3V3 Shutdown! Mod -> Carrier"
- note removed: "Module drives carrier"
- note removed: "Shift 5V Shutdown Req to 3V3 Shutdown!"
Changed lines of the file:
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@@
 		)
 	)
-	(text "Shift 5V Shutdown Req to 3V3 Shutdown!"
+	(text "Shift 5V Shutdown Req to 3V3 Shutdown! Mod -> Carrier"
 		(exclude_from_sim no)
 		(at 57.15 166.37 0)
@@
 		)
 	)
-	(text "Module drives carrier"
-		(exclude_from_sim no)
-		(at -11.684 179.324 0)
-		(effects
-			(font
-				(size 1.27 1.27)
-			)
-		)
-	)
 	(text "Sleep Status Output >"
 		(exclude_from_sim no)
@@
 	(wire
 		(pts
+			(xy 209.55 120.65) (xy 204.47 120.65)
+		)
+		(stroke
+			(width 0)
+			(type default)
+		)
+	)
+	(wire
+		(pts
 			(xy 330.2 148.59) (xy 336.55 148.59)
 		)
@@
 		)
 	)
+	(global_label "MOD_PWR_REQ"
+		(shape input)
+		(at 67.31 186.69 0)
+		(fields_autoplaced yes)
+		(effects
+			(font
+				(size 1.27 1.27)
+			)
+			(justify left)
+		)
+		(property "Intersheetrefs" "${INTERSHEET_REFS}"
+			(at 84.1183 186.69 0)
+			(effects
+				(font
+					(size 1.27 1.27)
+				)
+				(justify left)
+				(hide yes)
+			)
+		)
+	)
 	(global_label "SPI-1_CLK_3V3"
 		(shape output)
@@
 		)
 	)
+	(global_label "MOD_PWR_REQ"
+		(shape input)
+		(at 209.55 120.65 0)
+		(fields_autoplaced yes)
+		(effects
+			(font
+				(size 1.27 1.27)
+			)
+			(justify left)
+		)
+		(property "Intersheetrefs" "${INTERSHEET_REFS}"
+			(at 226.3583 120.65 0)
+			(effects
+				(font
+					(size 1.27 1.27)
+				)
+				(justify left)
+				(hide yes)
+			)
+		)
+	)
 	(global_label "UART-0_TX_3V3"
 		(shape output)
@@
 	)
 	(global_label "SHUT_REQ_BMC"
-		(shape input)
+		(shape output)
 		(at 46.99 186.69 180)
 		(fields_autoplaced yes)
@@
 		)
 	)
-	(global_label "PMIC_EN"
-		(shape output)
-		(at 67.31 186.69 0)
-		(fields_autoplaced yes)
-		(effects
-			(font
-				(size 1.27 1.27)
-			)
-			(justify left)
-		)
-		(property "Intersheetrefs" "${INTERSHEET_REFS}"
-			(at 78.4336 186.69 0)
-			(effects
-				(font
-					(size 1.27 1.27)
-				)
-				(justify left)
-				(hide yes)
-			)
-		)
-	)
 	(global_label "VBAT"
 		(shape output)
@@
 			)
 		)
-		(property "Value" "5K"
+		(property "Value" "10K"
 			(at 70.866 182.88 0)
 			(effects

Commit message: fixing the PMIC mosfet
Parts:
- added Q2: BSS138, Package_TO_SOT_SMD:SOT-23-3, symbol Simulation_SPICE:NMOS
- added R10: 5K, Resistor_SMD:R_0402_1005Metric, symbol Device:R
- added R11: 10K, Resistor_SMD:R_0402_1005Metric, symbol Device:R
Connections:
- net +3V3: now also Q2.2 (G), R11.1
- net +5V: now also R10.1
- net PMIC_EN: now also Q2.3 (S), R11.2
- net POWER_BMC: now also Q2.1 (D), R10.2
Other:
- note added: "Carrier 5V Analog triggering PMIC"
- moved on the sheet: Q1, Q3, R12, R13, R3, R4

Commit message: saving everything from school
Parts:
- removed Q1: BSS138, Package_TO_SOT_SMD:SOT-23-3, symbol Simulation_SPICE:NMOS
- removed R3: 100, Resistor_SMD:R_0402_1005Metric, symbol Device:R
- removed R4: 100K, Resistor_SMD:R_0402_1005Metric, symbol Device:R
Other:
- note added: "Carrier 5V analog triggering PMIC on mod"
- note removed: "Carrier 5V Analog triggering PMIC"
- note removed: "Carrier drives module"

Commit message: some journaling, wondering if I need a schmitt trigger for PMIC_EN
Parts:
- R10: value 5K -> 10K
Changed lines of the file:
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@@
 			)
 		)
-		(property "Value" "5K"
+		(property "Value" "10K"
 			(at 46.99 107.9499 0)
 			(effects
