File: PCB_CARRIER/level-shifting.kicad_sch (KiCad schematic)
At the start: 2 parts, among them U1 TXB0108DQSR, U3 TXB0108DQSR

Commit message: hopping off for the night, but I'm sincerely almost done the wiring
Other:
- note added: "LIKELY SHIFTED PINS: MOD SLEEP and PWM"
- note added: "SPI isn't good for these"
- moved on the sheet: U1, U3
Changed lines of the file:
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@@
 	(generator_version "9.0")
 	(paper "A4")
+	(text "LIKELY SHIFTED PINS: MOD SLEEP and PWM"
+		(exclude_from_sim no)
+		(at 61.722 82.55 0)
+		(effects
+			(font
+				(size 1.27 1.27)
+			)
+		)
+	)
+	(text "SPI isn't good for these"
+		(exclude_from_sim no)
+		(at 51.054 99.568 0)
+		(effects
+			(font
+				(size 1.27 1.27)
+			)
+		)
+	)
 	(symbol
 		(lib_id "Logic_LevelTranslator:TXB0108DQSR")
-		(at 153.67 100.33 0)
+		(at 175.26 100.33 0)
 		(unit 1)
 		(exclude_from_sim no)
@@
 		(fields_autoplaced yes)
 		(property "Reference" "U3"
-			(at 155.8133 118.11 0)
+			(at 177.4033 118.11 0)
 			(effects
 				(font
@@
 		)
 		(property "Value" "TXB0108DQSR"
-			(at 155.8133 120.65 0)
+			(at 177.4033 120.65 0)
 			(effects
 				(font
@@
 		)
 		(property "Footprint" "Package_SON:USON-20_2x4mm_P0.4mm"
-			(at 153.67 119.38 0)
+			(at 175.26 119.38 0)
 			(effects
 				(font
@@
 		)
 		(property "Datasheet" "http://www.ti.com/lit/ds/symlink/txb0108.pdf"
-			(at 153.67 102.87 0)
+			(at 175.26 102.87 0)
 			(effects
 				(font
@@
 		)
 		(property "Description" "8-Bit Bidirectional Voltage-Level Translator, Auto Direction Sensing and ±15-kV ESD Protection, 1.2 - 3.6V APort, 1.65 - 5.5V BPort, USON-20"
-			(at 153.67 100.33 0)
+			(at 175.26 100.33 0)
 			(effects
 				(font
@@
 	(symbol
 		(lib_id "Logic_LevelTranslator:TXB0108DQSR")
-		(at 114.3 99.06 0)
+		(at 135.89 100.33 0)
 		(unit 1)
 		(exclude_from_sim no)
@@
 		(fields_autoplaced yes)
 		(property "Reference" "U1"
-			(at 116.4433 116.84 0)
+			(at 138.0333 118.11 0)
 			(effects
 				(font
@@
 		)
 		(property "Value" "TXB0108DQSR"
-			(at 116.4433 119.38 0)
+			(at 138.0333 120.65 0)
 			(effects
 				(font
@@
 		)
 		(property "Footprint" "Package_SON:USON-20_2x4mm_P0.4mm"
-			(at 114.3 118.11 0)
+			(at 135.89 119.38 0)
 			(effects
 				(font
@@
 		)
 		(property "Datasheet" "http://www.ti.com/lit/ds/symlink/txb0108.pdf"
-			(at 114.3 101.6 0)
+			(at 135.89 102.87 0)
 			(effects
 				(font
@@
 		)
 		(property "Description" "8-Bit Bidirectional Voltage-Level Translator, Auto Direction Sensing and ±15-kV ESD Protection, 1.2 - 3.6V APort, 1.65 - 5.5V BPort, USON-20"
-			(at 114.3 99.06 0)
+			(at 135.89 100.33 0)
 			(effects
 				(font

Commit message: SPI level shift components, I think I finally got this down
Parts:
- removed U1, U3: TXB0108DQSR, Package_SON:USON-20_2x4mm_P0.4mm, symbol Logic_LevelTranslator:TXB0108DQSR
- added U1, U2: SN74LVC8T245, symbol Logic_LevelTranslator:SN74LVC8T245
Connections:
- new net: U1.11 (GND), U1.12 (GND), U1.13 (GND)
- new net: U1.23 (V_{CCB}), U1.24 (V_{CCB})
- new net: U2.11 (GND), U2.12 (GND), U2.13 (GND)
- new net: U2.23 (V_{CCB}), U2.24 (V_{CCB})
Other:
- note added: "SPI 8-Bit Unidirectional Transceiver"
- note removed: "LIKELY SHIFTED PINS: MOD SLEEP and PWM"
- note removed: "SPI isn't good for these"
Changed lines of the file:
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@@
 	(generator_version "9.0")
 	(paper "A4")
-	(text "LIKELY SHIFTED PINS: MOD SLEEP and PWM"
+	(text "SPI 8-Bit Unidirectional Transceiver\n"
 		(exclude_from_sim no)
-		(at 61.722 82.55 0)
+		(at 54.61 69.85 0)
 		(effects
 			(font
@@
 		)
 	)
-	(text "SPI isn't good for these"
-		(exclude_from_sim no)
-		(at 51.054 99.568 0)
-		(effects
-			(font
-				(size 1.27 1.27)
-			)
-		)
-	)
 	(symbol
-		(lib_id "Logic_LevelTranslator:TXB0108DQSR")
-		(at 175.26 100.33 0)
-		(unit 1)
-		(exclude_from_sim no)
-		(in_bom yes)
-		(on_board yes)
-		(dnp no)
-		(fields_autoplaced yes)
-		(property "Reference" "U3"
-			(at 177.4033 118.11 0)
-			(effects
-				(font
-					(size 1.27 1.27)
-				)
-				(justify left)
-			)
-		)
-		(property "Value" "TXB0108DQSR"
-			(at 177.4033 120.65 0)
-			(effects
-				(font
-					(size 1.27 1.27)
-				)
-				(justify left)
-			)
-		)
-		(property "Footprint" "Package_SON:USON-20_2x4mm_P0.4mm"
-			(at 175.26 119.38 0)
-			(effects
-				(font
-					(size 1.27 1.27)
-				)
-				(hide yes)
-			)
-		)
-		(property "Datasheet" "http://www.ti.com/lit/ds/symlink/txb0108.pdf"
-			(at 175.26 102.87 0)
-			(effects
-				(font
-					(size 1.27 1.27)
-				)
-				(hide yes)
-			)
-		)
-		(property "Description" "8-Bit Bidirectional Voltage-Level Translator, Auto Direction Sensing and ±15-kV ESD Protection, 1.2 - 3.6V APort, 1.65 - 5.5V BPort, USON-20"
-			(at 175.26 100.33 0)
-			(effects
-				(font
-					(size 1.27 1.27)
-				)
-				(hide yes)
-			)
-		)
-		(pin "9"
-		)
-		(pin "8"
-		)
-		(pin "20"
-		)
-		(pin "17"
-		)
-		(pin "16"
-		)
-		(pin "19"
-		)
-		(pin "3"
-		)
-		(pin "4"
-		)
-		(pin "13"
-		)
-		(pin "18"
-		)
-		(pin "7"
-		)
-		(pin "14"
-		)
-		(pin "1"
-		)
-		(pin "6"
-		)
-		(pin "12"
-		)
-		(pin "2"
-		)
-		(pin "5"
-		)
-		(pin "15"
-		)
-		(pin "10"
-		)
-		(pin "11"
-		)
-		(instances
-			(project "carrier"
-				(path "/f52509e6-8053-454c-b8e9-3e2670c5a5fe/7b90d14f-4142-447b-ad6a-0ca28adbd057"
-					(reference "U3")
-					(unit 1)
-				)
-			)
-		)
-	)
-	(symbol
-		(lib_id "Logic_LevelTranslator:TXB0108DQSR")
-		(at 135.89 100.33 0)
+		(lib_id "Logic_LevelTranslator:SN74LVC8T245")
+		(at 45.72 107.95 0)
 		(unit 1)
 		(exclude_from_sim no)
@@
 		(fields_autoplaced yes)
 		(property "Reference" "U1"
-			(at 138.0333 118.11 0)
-			(effects
-				(font
-					(size 1.27 1.27)
-				)
-				(justify left)
-			)
-		)
-		(property "Value" "TXB0108DQSR"
-			(at 138.0333 120.65 0)
-			(effects
-				(font
-					(size 1.27 1.27)
-				)
-				(justify left)
-			)
-		)
-		(property "Footprint" "Package_SON:USON-20_2x4mm_P0.4mm"
-			(at 135.89 119.38 0)
-			(effects
-				(font
-					(size 1.27 1.27)
-				)
-				(hide yes)
-			)
-		)
-		(property "Datasheet" "http://www.ti.com/lit/ds/symlink/txb0108.pdf"
-			(at 135.89 102.87 0)
-			(effects
-				(font
-					(size 1.27 1.27)
-				)
-				(hide yes)
-			)
-		)
-		(property "Description" "8-Bit Bidirectional Voltage-Level Translator, Auto Direction Sensing and ±15-kV ESD Protection, 1.2 - 3.6V APort, 1.65 - 5.5V BPort, USON-20"
-			(at 135.89 100.33 0)
-			(effects
-				(font
-					(size 1.27 1.27)
-				)
-				(hide yes)
-			)
+			(at 47.8633 135.89 0)
+			(effects
+				(font
+					(size 1.27 1.27)
+				)
+				(justify left)
+			)
+		)
+		(property "Value" "SN74LVC8T245"
+			(at 47.8633 138.43 0)
+			(effects
+				(font
+					(size 1.27 1.27)
+				)
+				(justify left)
+			)
+		)
+		(property "Footprint" ""
+			(at 66.04 132.08 0)
+			(effects
+				(font
+					(size 1.27 1.27)
+				)
+				(hide yes)
+			)
+		)
+		(property "Datasheet" "https://www.ti.com/lit/ds/symlink/sn74lvc8t245.pdf"
+			(at 45.72 143.51 0)
+			(effects
+				(font
+					(size 1.27 1.27)
+				)
+				(hide yes)
+			)
+		)
+		(property "Description" "8-Bit Dual-Supply Bus Transceiver With Configurable Voltage Translation and 3-State Outputs"
+			(at 45.72 107.95 0)
+			(effects
+				(font
+					(size 1.27 1.27)
+				)
+				(hide yes)
+			)
+		)
+		(pin "2"
+		)
+		(pin "23"
+		)
+		(pin "13"
+		)
+		(pin "1"
+		)
+		(pin "21"
+		)
+		(pin "22"
+		)
+		(pin "24"
+		)
+		(pin "19"
+		)
+		(pin "20"
+		)
+		(pin "3"
+		)
+		(pin "6"
+		)
+		(pin "5"
+		)
+		(pin "4"
+		)
+		(pin "10"
+		)
+		(pin "11"
+		)
+		(pin "12"
+		)
+		(pin "18"
+		)
+		(pin "7"
+		)
+		(pin "17"
+		)
+		(pin "15"
+		)
+		(pin "14"
+		)
+		(pin "8"
 		)
 		(pin "9"
 		)
-		(pin "8"
-		)
-		(pin "20"
-		)
-		(pin "17"
-		)
 		(pin "16"
-		)
-		(pin "19"
-		)
-		(pin "3"
-		)
-		(pin "4"
-		)
-		(pin "13"
-		)
-		(pin "18"
-		)
-		(pin "7"
-		)
-		(pin "14"
-		)
-		(pin "1"
-		)
-		(pin "6"
-		)
-		(pin "12"
-		)
-		(pin "2"
-		)
-		(pin "5"
-		)
-		(pin "15"
-		)
-		(pin "10"
-		)
-		(pin "11"
 		)
 		(instances
@@
 					(unit 1)
 				)
+			)
+		)
+	)
+	(symbol
+		(lib_id "Logic_LevelTranslator:SN74LVC8T245")
+		(at 87.63 107.95 0)
+		(unit 1)
+		(exclude_from_sim no)
+		(in_bom yes)
+		(on_board yes)
+		(dnp no)
+		(fields_autoplaced yes)
+		(property "Reference" "U2"
+			(at 89.7733 135.89 0)
+			(effects
+				(font
+					(size 1.27 1.27)
+				)
+				(justify left)
+			)
+		)
+		(property "Value" "SN74LVC8T245"
+			(at 89.7733 138.43 0)
+			(effects
+				(font
+					(size 1.27 1.27)
+				)
+				(justify left)
+			)
+		)
+		(property "Footprint" ""
+			(at 107.95 132.08 0)
+			(effects
+				(font
+					(size 1.27 1.27)
+				)
+				(hide yes)
+			)
+		)
+		(property "Datasheet" "https://www.ti.com/lit/ds/symlink/sn74lvc8t245.pdf"
+			(at 87.63 143.51 0)
+			(effects
+				(font
+					(size 1.27 1.27)
+				)
+				(hide yes)
+			)
+		)
+		(property "Description" "8-Bit Dual-Supply Bus Transceiver With Configurable Voltage Translation and 3-State Outputs"
+			(at 87.63 107.95 0)
+			(effects
+				(font
+					(size 1.27 1.27)
+				)
+				(hide yes)
+			)
+		)
+		(pin "2"
+		)
+		(pin "23"
+		)
+		(pin "13"
+		)
+		(pin "1"
+		)
+		(pin "21"
+		)
+		(pin "22"
+		)
+		(pin "24"
+		)
+		(pin "19"
+		)
+		(pin "20"
+		)
+		(pin "3"
+		)
+		(pin "6"
+		)
+		(pin "5"
+		)
+		(pin "4"
+		)
+		(pin "10"
+		)
+		(pin "11"
+		)
+		(pin "12"
+		)
+		(pin "18"
+		)
+		(pin "7"
+		)
+		(pin "17"
+		)
+		(pin "15"
+		)
+		(pin "14"
+		)
+		(pin "8"
+		)
+		(pin "9"
+		)
+		(pin "16"
+		)
+		(instances
+			(project "carrier"
+				(path "/f52509e6-8053-454c-b8e9-3e2670c5a5fe/7b90d14f-4142-447b-ad6a-0ca28adbd057"
+					(reference "U2")
+					(unit 1)
+				)

Commit message: fixing SPI label direction, and changing level shifting
Parts:
- removed U2: SN74LVC8T245, symbol Logic_LevelTranslator:SN74LVC8T245
Other:
- note added: "SPI 8-Bit Unidirectional Transceiver, one direction 8 pins - MOSI/CS/CLK output 2 pins - MISO input"
- note removed: "SPI 8-Bit Unidirectional Transceiver"
Changed lines of the file:
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@@
 	(generator_version "9.0")
 	(paper "A4")
-	(text "SPI 8-Bit Unidirectional Transceiver\n"
+	(text "SPI 8-Bit Unidirectional Transceiver, one direction\n8 pins - MOSI/CS/CLK output\n2 pins - MISO input\n"
 		(exclude_from_sim no)
-		(at 54.61 69.85 0)
+		(at 37.084 70.612 0)
 		(effects
 			(font
 				(size 1.27 1.27)
 			)
+			(justify left)
 		)
 	)
@@
 					(unit 1)
 				)
-			)
-		)
-	)
-	(symbol
-		(lib_id "Logic_LevelTranslator:SN74LVC8T245")
-		(at 87.63 107.95 0)
-		(unit 1)
-		(exclude_from_sim no)
-		(in_bom yes)
-		(on_board yes)
-		(dnp no)
-		(fields_autoplaced yes)
-		(property "Reference" "U2"
-			(at 89.7733 135.89 0)
-			(effects
-				(font
-					(size 1.27 1.27)
-				)
-				(justify left)
-			)
-		)
-		(property "Value" "SN74LVC8T245"
-			(at 89.7733 138.43 0)
-			(effects
-				(font
-					(size 1.27 1.27)
-				)
-				(justify left)
-			)
-		)
-		(property "Footprint" ""
-			(at 107.95 132.08 0)
-			(effects
-				(font
-					(size 1.27 1.27)
-				)
-				(hide yes)
-			)
-		)
-		(property "Datasheet" "https://www.ti.com/lit/ds/symlink/sn74lvc8t245.pdf"
-			(at 87.63 143.51 0)
-			(effects
-				(font
-					(size 1.27 1.27)
-				)
-				(hide yes)
-			)
-		)
-		(property "Description" "8-Bit Dual-Supply Bus Transceiver With Configurable Voltage Translation and 3-State Outputs"
-			(at 87.63 107.95 0)
-			(effects
-				(font
-					(size 1.27 1.27)
-				)
-				(hide yes)
-			)
-		)
-		(pin "2"
-		)
-		(pin "23"
-		)
-		(pin "13"
-		)
-		(pin "1"
-		)
-		(pin "21"
-		)
-		(pin "22"
-		)
-		(pin "24"
-		)
-		(pin "19"
-		)
-		(pin "20"
-		)
-		(pin "3"
-		)
-		(pin "6"
-		)
-		(pin "5"
-		)
-		(pin "4"
-		)
-		(pin "10"
-		)
-		(pin "11"
-		)
-		(pin "12"
-		)
-		(pin "18"
-		)
-		(pin "7"
-		)
-		(pin "17"
-		)
-		(pin "15"
-		)
-		(pin "14"
-		)
-		(pin "8"
-		)
-		(pin "9"
-		)
-		(pin "16"
-		)
-		(instances
-			(project "carrier"
-				(path "/f52509e6-8053-454c-b8e9-3e2670c5a5fe/7b90d14f-4142-447b-ad6a-0ca28adbd057"
-					(reference "U2")
-					(unit 1)
-				)

Commit message: starting to wire SPI shifting
Parts:
- added U2: SN74LVC2T45DCUR, Package_SO:VSSOP-8_2.3x2mm_P0.5mm, symbol Logic_LevelTranslator:SN74LVC2T45DCUR
Connections:
- net GND: now reaches U1.11 (GND), U1.12 (GND), U1.13 (GND)
- net GND: now also U2.4 (GND)
Other:
- moved on the sheet: U1
Changed lines of the file:
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@@
+		)
+	)
+	(wire
+		(pts
+			(xy 45.72 147.32) (xy 45.72 146.05)
+		)
+		(stroke
+			(width 0)
+			(type default)
+		)
+	)
+	(wire
+		(pts
+			(xy 93.98 116.84) (xy 93.98 115.57)
+		)
+		(stroke
+			(width 0)
+			(type default)
+		)
+	)
+	(symbol
+		(lib_id "power:GND")
+		(at 45.72 147.32 0)
+		(unit 1)
+		(exclude_from_sim no)
+		(in_bom yes)
+		(on_board yes)
+		(dnp no)
+		(fields_autoplaced yes)
+		(property "Reference" "#PWR014"
+			(at 45.72 153.67 0)
+			(effects
+				(font
+					(size 1.27 1.27)
+				)
+				(hide yes)
+			)
+		)
+		(property "Value" "GND"
+			(at 45.72 152.4 0)
+			(effects
+				(font
+					(size 1.27 1.27)
+				)
+			)
+		)
+		(property "Footprint" ""
+			(at 45.72 147.32 0)
+			(effects
+				(font
+					(size 1.27 1.27)
+				)
+				(hide yes)
+			)
+		)
+		(property "Datasheet" ""
+			(at 45.72 147.32 0)
+			(effects
+				(font
+					(size 1.27 1.27)
+				)
+				(hide yes)
+			)
+		)
+		(property "Description" "Power symbol creates a global label with name \"GND\" , ground"
+			(at 45.72 147.32 0)
+			(effects
+				(font
+					(size 1.27 1.27)
+				)
+				(hide yes)
+			)
+		)
+		(pin "1"
+		)
+		(instances
+			(project ""
+				(path "/f52509e6-8053-454c-b8e9-3e2670c5a5fe/7b90d14f-4142-447b-ad6a-0ca28adbd057"
+					(reference "#PWR014")
+					(unit 1)
+				)
+			)
 		)
 	)
 	(symbol
 		(lib_id "Logic_LevelTranslator:SN74LVC8T245")
-		(at 45.72 107.95 0)
+		(at 45.72 118.11 0)
 		(unit 1)
 		(exclude_from_sim no)
@@
 		(fields_autoplaced yes)
 		(property "Reference" "U1"
-			(at 47.8633 135.89 0)
+			(at 47.8633 146.05 0)
 			(effects
 				(font
@@
 		)
 		(property "Value" "SN74LVC8T245"
-			(at 47.8633 138.43 0)
+			(at 47.8633 148.59 0)
 			(effects
 				(font
@@
 		)
 		(property "Footprint" ""
-			(at 66.04 132.08 0)
+			(at 66.04 142.24 0)
 			(effects
 				(font
@@
 		)
 		(property "Datasheet" "https://www.ti.com/lit/ds/symlink/sn74lvc8t245.pdf"
-			(at 45.72 143.51 0)
+			(at 45.72 153.67 0)
 			(effects
 				(font
@@
 		)
 		(property "Description" "8-Bit Dual-Supply Bus Transceiver With Configurable Voltage Translation and 3-State Outputs"
-			(at 45.72 107.95 0)
+			(at 45.72 118.11 0)
 			(effects
 				(font
@@
 					(unit 1)
 				)
+			)
+		)
+	)
+	(symbol
+		(lib_id "Logic_LevelTranslator:SN74LVC2T45DCUR")
+		(at 93.98 102.87 0)
+		(unit 1)
+		(exclude_from_sim no)
+		(in_bom yes)
+		(on_board yes)
+		(dnp no)
+		(fields_autoplaced yes)
+		(property "Reference" "U2"
+			(at 96.1233 115.57 0)
+			(effects
+				(font
+					(size 1.27 1.27)
+				)
+				(justify left)
+			)
+		)
+		(property "Value" "SN74LVC2T45DCUR"
+			(at 96.1233 118.11 0)
+			(effects
+				(font
+					(size 1.27 1.27)
+				)
+				(justify left)
+			)
+		)
+		(property "Footprint" "Package_SO:VSSOP-8_2.3x2mm_P0.5mm"
+			(at 95.25 116.84 0)
+			(effects
+				(font
+					(size 1.27 1.27)
+				)
+				(hide yes)
+			)
+		)
+		(property "Datasheet" "http://www.ti.com/lit/ds/symlink/sn74lvc2t45.pdf"
+			(at 71.12 116.84 0)
+			(effects
+				(font
+					(size 1.27 1.27)
+				)
+				(hide yes)
+			)
+		)
+		(property "Description" "Dual-Bit Dual-Supply Bus Transceiver With Configurable Voltage Translation and 3-State Outputs, VSSOP-8"
+			(at 93.98 102.87 0)
+			(effects
+				(font
+					(size 1.27 1.27)
+				)
+				(hide yes)
+			)
+		)
+		(pin "2"
+		)
+		(pin "3"
+		)
+		(pin "5"
+		)
+		(pin "1"
+		)
+		(pin "4"
+		)
+		(pin "8"
+		)
+		(pin "7"
+		)
+		(pin "6"
+		)
+		(instances
+			(project ""
+				(path "/f52509e6-8053-454c-b8e9-3e2670c5a5fe/7b90d14f-4142-447b-ad6a-0ca28adbd057"
+					(reference "U2")
+					(unit 1)
+				)
+			)
+		)
+	)
+	(symbol
+		(lib_id "power:GND")
+		(at 93.98 116.84 0)
+		(unit 1)
+		(exclude_from_sim no)
+		(in_bom yes)
+		(on_board yes)
+		(dnp no)
+		(fields_autoplaced yes)
+		(property "Reference" "#PWR015"
+			(at 93.98 123.19 0)
+			(effects
+				(font
+					(size 1.27 1.27)
+				)
+				(hide yes)
+			)
+		)
+		(property "Value" "GND"
+			(at 93.98 121.92 0)
+			(effects
+				(font
+					(size 1.27 1.27)
+				)
+			)
+		)
+		(property "Footprint" ""
+			(at 93.98 116.84 0)
+			(effects
+				(font
+					(size 1.27 1.27)
+				)
+				(hide yes)
+			)
+		)
+		(property "Datasheet" ""
+			(at 93.98 116.84 0)
+			(effects
+				(font
+					(size 1.27 1.27)
+				)
+				(hide yes)
+			)
+		)
+		(property "Description" "Power symbol creates a global label with name \"GND\" , ground"
+			(at 93.98 116.84 0)
+			(effects
+				(font
+					(size 1.27 1.27)
+				)
+				(hide yes)
+			)
+		)
+		(pin "1"
+		)
+		(instances
+			(project "carrier"
+				(path "/f52509e6-8053-454c-b8e9-3e2670c5a5fe/7b90d14f-4142-447b-ad6a-0ca28adbd057"
+					(reference "#PWR015")
+					(unit 1)
+				)

Commit message: SPI inputs to level shift
Connections:
- net +1V8: now reaches U1.1 (V_{CCA})
- net +1V8: now also U2.1 (VCCA)
- net SPI-1_CS1_3V3: now reaches U1.14 (B8)
- net SPI-1_CS0_3V3: now reaches U1.15 (B7)
- net SPI-1_CLK_3V3: now reaches U1.16 (B6)
- net SPI-1_MOSI_3V3: now reaches U1.17 (B5)
- net SPI-0_CS1_3V3: now reaches U1.18 (B4)
- net SPI-0_CS0_3V3: now reaches U1.19 (B3)
- net SPI-0_CLK_3V3: now reaches U1.20 (B2)
- net SPI-0_MOSI_3V3: now reaches U1.21 (B1)
- net +3V3: now reaches U1.23 (V_{CCB}), U1.24 (V_{CCB})
- net +3V3: now also U2.8 (VCCB)
- net SPI-0_MISO_3V3: now reaches U2.2 (A1)
- net SPI-1_MISO_3V3: now reaches U2.3 (A2)
Other:
- moved on the sheet: U1, U2
