File: PCB_CARRIER/level-shifting.kicad_sch (KiCad schematic)
At the start: 11 parts, among them U1 SN74LVC8T245, U2 SN74LVC2T45DCUR

Commit message: fixed dir mode
Connections:
- net +3V3: no longer R2.1, R6.1
- net GND: now also R2.2, R6.2
- net at U1.2 (DIR): now also R2.1; no longer R2.2
- net at U2.5 (DIR): now also R6.1; no longer R6.2

Commit message: fixed SPI, this is breaking my head
Parts:
- removed C13, C15: 0.1uF, symbol Device:C
- removed U2: SN74LVC2T45DCUR, Package_SO:VSSOP-8_2.3x2mm_P0.5mm, symbol Logic_LevelTranslator:SN74LVC2T45DCUR
- added C12, C16: 1uF, symbol Device:C
- added C14, C17: 0.1uF, symbol Device:C
- added R7: 10K, symbol Device:R
- added U3: SN74LVC8T245, symbol Logic_LevelTranslator:SN74LVC8T245
Connections:
- net +1V8: now also C12.2, C14.2, U3.1 (V_{CCA})
- net +3V3: now also C16.1, C17.1, U3.23 (V_{CCB}), U3.24 (V_{CCB})
- net GND: now also C12.1, C14.1, C16.2, C17.2, R7.2, U3.11 (GND), U3.12 (GND), U3.13 (GND)
- net SPI-0_MISO_1V8: now also U3.21 (B1)
- net SPI-0_MISO_3V3: now also U3.3 (A1)
- net SPI-1_MISO_1V8: now also U3.20 (B2)
- net SPI-1_MISO_3V3: now also U3.4 (A2)
- net at R6.1: now also U3.2 (DIR)
- new net: R7.1, U3.22 (~{OE})
Other:
- moved on the sheet: C10, C3, C8, C9, R2, R5, U1

Commit message: level shifted UART
Connections:
- net +1V8: now also C16.1, C17.1, U3.23 (V_{CCB}), U3.24 (V_{CCB}); no longer C12.2, C14.2, U3.1 (V_{CCA})
- net +3V3: now also C12.2, C14.2, U3.1 (V_{CCA}); no longer C16.1, C17.1, U3.23 (V_{CCB}), U3.24 (V_{CCB})
- net UART-2_RX_1V8: now reaches U3.15 (B7)
- net UART-1_RX_1V8: now reaches U3.16 (B6)
- net UART-1_CTS_1V8: now reaches U3.17 (B5)
- net UART-0_RX_1V8: now reaches U3.18 (B4)
- net UART-0_CTS_1V8: now reaches U3.19 (B3)
- net UART-0_CTS_3V3: now reaches U3.5 (A3)
- net UART-0_RX_3V3: now reaches U3.6 (A4)
- net UART-1_CTS_3V3: now reaches U3.7 (A5)
- net UART-1_RX_3V3: now reaches U3.8 (A6)
- net UART-2_RX_3V3: now reaches U3.9 (A7)
- no-connect marks 0 -> 2

Commit message: moved SPI level shifting pins for better routing, working on UART
Parts:
- added C13, C18: 1uF, symbol Device:C
- added C15, C19: 0.1uF, symbol Device:C
- added R8, R9: 10K, symbol Device:R
- added U2: SN74LVC8T245, symbol Logic_LevelTranslator:SN74LVC8T245
Connections:
- net +1V8: now also C13.2, C15.2, U2.1 (V_{CCA})
- net +3V3: now also C18.1, C19.1, U2.23 (V_{CCB}), U2.24 (V_{CCB})
- net GND: now also C13.1, C15.1, C18.2, C19.2, R8.2, R9.2, U2.11 (GND), U2.12 (GND), U2.13 (GND)
- net UART-0_CTS_1V8: now also U3.18 (B4); no longer U3.19 (B3)
- net UART-0_CTS_3V3: now also U3.6 (A4); no longer U3.5 (A3)
- net UART-0_RX_1V8: now also U3.19 (B3); no longer U3.18 (B4)
- net UART-0_RX_3V3: now also U3.5 (A3); no longer U3.6 (A4)
- net UART-1_CTS_1V8: now also U3.16 (B6); no longer U3.17 (B5)
- net UART-1_CTS_3V3: now also U3.8 (A6); no longer U3.7 (A5)
- net UART-1_RX_1V8: now also U3.17 (B5); no longer U3.16 (B6)
- net UART-1_RX_3V3: now also U3.7 (A5); no longer U3.8 (A6)
- new net: R8.1, U2.2 (DIR)
- new net: R9.1, U2.22 (~{OE})
- no-connect marks 2 -> 3
Other:
- note removed: "Share bulks with MISO"

Commit message: level shifting UART
Connections:
- net UART-0_RTS_3V3: now also U2.20 (B2)
- net UART-0_TX_3V3: now also U2.21 (B1)
- net UART-1_RTS_3V3: now also U2.18 (B4)
- net UART-1_TX_3V3: now also U2.19 (B3)
- net UART-2_TX_3V3: now reaches U2.17 (B5)
- net UART-0_TX_1V8: now reaches U2.3 (A1)
- net UART-0_RTS_1V8: now reaches U2.4 (A2)
- net UART-1_TX_1V8: now reaches U2.5 (A3)
- net UART-1_RTS_1V8: now reaches U2.6 (A4)
- net UART-2_TX_1V8: now reaches U2.7 (A5)
- no-connect marks 3 -> 8
Other:
- moved on the sheet: C13, C15, C18, C19, R8, R9, U2

Commit message: only GPIO0 left to level shift, so I kinda wanna figure out a different way without adding a bidirectional shifter, but pwm and tach are in now
Connections:
- net FAN_PWM_3V3: now reaches U2.16 (B6)
- net FAN_PWM_1V8: now reaches U2.8 (A6)
- net FAN_TACH_3V3: now reaches U3.10 (A8)
- net FAN_TACH_1V8: now reaches U3.14 (B8)
- no-connect marks 8 -> 4
Changed lines of the file:
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@@
-	)
-	(no_connect
-		(at 113.03 119.38)
-	)
-	(no_connect
-		(at 184.15 109.22)
-	)
-	(no_connect
-		(at 204.47 109.22)
 	)
 	(no_connect
@@
 		(at 204.47 114.3)
 	)
-	(no_connect
-		(at 133.35 119.38)
-	)
 	(wire
 		(pts
@@
 	(wire
 		(pts
+			(xy 181.61 109.22) (xy 184.15 109.22)
+		)
+		(stroke
+			(width 0)
+			(type default)
+		)
+	)
+	(wire
+		(pts
 			(xy 110.49 109.22) (xy 113.03 109.22)
 		)
@@
 	(wire
 		(pts
+			(xy 207.01 109.22) (xy 204.47 109.22)
+		)
+		(stroke
+			(width 0)
+			(type default)
+		)
+	)
+	(wire
+		(pts
 			(xy 39.37 134.62) (xy 52.07 134.62)
 		)
@@
 	(wire
 		(pts
+			(xy 110.49 119.38) (xy 113.03 119.38)
+		)
+		(stroke
+			(width 0)
+			(type default)
+		)
+	)
+	(wire
+		(pts
 			(xy 135.89 69.85) (xy 138.43 69.85)
 		)
@@
 		(pts
 			(xy 110.49 93.98) (xy 113.03 93.98)
+		)
+		(stroke
+			(width 0)
+			(type default)
+		)
+	)
+	(wire
+		(pts
+			(xy 135.89 119.38) (xy 133.35 119.38)
 		)
 		(stroke
@@
 		)
 	)
+	(global_label "FAN_PWM_3V3"
+		(shape input)
+		(at 207.01 109.22 0)
+		(fields_autoplaced yes)
+		(effects
+			(font
+				(size 1.27 1.27)
+			)
+			(justify left)
+		)
+		(property "Intersheetrefs" "${INTERSHEET_REFS}"
+			(at 223.2136 109.22 0)
+			(effects
+				(font
+					(size 1.27 1.27)
+				)
+				(justify left)
+				(hide yes)
+			)
+		)
+	)
 	(global_label "UART-0_RTS_3V3"
 		(shape input)
@@
 		)
 	)
+	(global_label "FAN_TACH_1V8"
+		(shape input)
+		(at 135.89 119.38 0)
+		(fields_autoplaced yes)
+		(effects
+			(font
+				(size 1.27 1.27)
+			)
+			(justify left)
+		)
+		(property "Intersheetrefs" "${INTERSHEET_REFS}"
+			(at 152.5775 119.38 0)
+			(effects
+				(font
+					(size 1.27 1.27)
+				)
+				(justify left)
+				(hide yes)
+			)
+		)
+	)
 	(global_label "UART-1_TX_1V8"
 		(shape output)
@@
 		)
 	)
+	(global_label "FAN_PWM_1V8"
+		(shape output)
+		(at 181.61 109.22 180)
+		(fields_autoplaced yes)
+		(effects
+			(font
+				(size 1.27 1.27)
+			)
+			(justify right)
+		)
+		(property "Intersheetrefs" "${INTERSHEET_REFS}"
+			(at 165.4064 109.22 0)
+			(effects
+				(font
+					(size 1.27 1.27)
+				)
+				(justify right)
+				(hide yes)
+			)
+		)
+	)
 	(global_label "UART-0_RX_3V3"
 		(shape output)
@@
 			(effects
 				(font
+					(size 1.27 1.27)
+				)
+				(justify right)
+				(hide yes)
+			)
+		)
+	)
+	(global_label "FAN_TACH_3V3"
+		(shape output)
+		(at 110.49 119.38 180)
+		(fields_autoplaced yes)
+		(effects
+			(font
+				(size 1.27 1.27)
+			)
+			(justify right)
+		)
+		(property "Intersheetrefs" "${INTERSHEET_REFS}"
+			(at 93.8025 119.38 0)
+			(effects
+				(font

Commit message: finally finished level shiftinggit add .git add .git add .git add .git add .git add .git add .git add .!
Connections:
- net GPIO0_3V3: now reaches U2.15 (B7)
- net GPIO0_1V8: now reaches U2.9 (A7)
- no-connect marks 4 -> 2
Other:
- note added: "< GPIO0 is transmit only to save on IC's"
- note added: "Receive SPI/UART/TACH"
- note added: "TRANSMIT SPI"
- note added: "Transmit UART/PWM/GPIO0"
- note removed: "SPI 8-Bit Unidirectional Transceiver, one direction 8 pins - MOSI/CS/CLK output 2 pins - MISO input"
- moved on the sheet: C10, C12, C13, C14, C15, C16, C17, C18, C19, C3, C8, C9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
