File: PCB_CARRIER/level-shifting.kicad_sch (KiCad schematic)
At the start: 21 parts, among them U1 SN74LVC8T245, U2 SN74LVC8T245, U3 SN74LVC8T245

Commit message: footprints for passives
Parts:
- C10, C12, C13, C14, C15, C16, C17, C18, C19, C3, C8, C9: footprint (none) -> Capacitor_SMD:C_0402_1005Metric
- R2: footprint (none) -> Capacitor_SMD:C_0603_1608Metric
- R5, R6, R7, R8, R9: footprint (none) -> Resistor_SMD:R_0402_1005Metric
Changed lines of the file:
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@@
 			)
 		)
-		(property "Footprint" ""
+		(property "Footprint" "Capacitor_SMD:C_0402_1005Metric"
 			(at 226.06 71.4248 0)
 			(effects
@@
 			)
 		)
-		(property "Footprint" ""
+		(property "Footprint" "Resistor_SMD:R_0402_1005Metric"
 			(at 127.762 132.08 90)
 			(effects
@@
 			)
 		)
-		(property "Footprint" ""
+		(property "Footprint" "Capacitor_SMD:C_0402_1005Metric"
 			(at 66.04 71.4248 0)
 			(effects
@@
 			)
 		)
-		(property "Footprint" ""
+		(property "Footprint" "Capacitor_SMD:C_0402_1005Metric"
 			(at 226.06 66.3448 0)
 			(effects
@@
 			)
 		)
-		(property "Footprint" ""
+		(property "Footprint" "Capacitor_SMD:C_0402_1005Metric"
 			(at 208.28 71.4248 0)
 			(effects
@@
 			)
 		)
-		(property "Footprint" ""
+		(property "Footprint" "Capacitor_SMD:C_0402_1005Metric"
 			(at 66.04 66.3448 0)
 			(effects
@@
 			)
 		)
-		(property "Footprint" ""
+		(property "Footprint" "Capacitor_SMD:C_0402_1005Metric"
 			(at 83.82 66.3448 0)
 			(effects
@@
 			)
 		)
-		(property "Footprint" ""
+		(property "Footprint" "Capacitor_SMD:C_0603_1608Metric"
 			(at 49.022 132.08 90)
 			(effects
@@
 			)
 		)
-		(property "Footprint" ""
+		(property "Footprint" "Capacitor_SMD:C_0402_1005Metric"
 			(at 154.94 71.4248 0)
 			(effects
@@
 			)
 		)
-		(property "Footprint" ""
+		(property "Footprint" "Capacitor_SMD:C_0402_1005Metric"
 			(at 137.16 71.4248 0)
 			(effects
@@
 			)
 		)
-		(property "Footprint" ""
+		(property "Footprint" "Capacitor_SMD:C_0402_1005Metric"
 			(at 208.28 66.3448 0)
 			(effects
@@
 			)
 		)
-		(property "Footprint" ""
+		(property "Footprint" "Resistor_SMD:R_0402_1005Metric"
 			(at 191.262 132.08 90)
 			(effects
@@
 			)
 		)
-		(property "Footprint" ""
+		(property "Footprint" "Resistor_SMD:R_0402_1005Metric"
 			(at 120.142 132.08 90)
 			(effects
@@
 			)
 		)
-		(property "Footprint" ""
+		(property "Footprint" "Capacitor_SMD:C_0402_1005Metric"
 			(at 137.16 66.3448 0)
 			(effects
@@
 			)
 		)
-		(property "Footprint" ""
+		(property "Footprint" "Resistor_SMD:R_0402_1005Metric"
 			(at 198.882 132.08 90)
 			(effects
@@
 			)
 		)
-		(property "Footprint" ""
+		(property "Footprint" "Capacitor_SMD:C_0402_1005Metric"
 			(at 154.94 66.3448 0)
 			(effects
@@
 			)
 		)
-		(property "Footprint" ""
+		(property "Footprint" "Capacitor_SMD:C_0402_1005Metric"
 			(at 83.82 71.4248 0)
 			(effects
@@
 			)
 		)
-		(property "Footprint" ""
+		(property "Footprint" "Resistor_SMD:R_0402_1005Metric"
 			(at 56.642 132.08 90)
 			(effects

Commit message: level shifter footprints, holy these are expensive
Parts:
- U1, U2, U3: footprint (none) -> Package_SO:TSSOP-24_4.4x5mm_P0.4mm
Changed lines of the file:
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@@
 			)
 		)
-		(property "Footprint" ""
+		(property "Footprint" "Package_SO:TSSOP-24_4.4x5mm_P0.4mm"
 			(at 233.68 128.27 0)
 			(effects
@@
 			)
 		)
-		(property "Footprint" ""
+		(property "Footprint" "Package_SO:TSSOP-24_4.4x5mm_P0.4mm"
 			(at 91.44 128.27 0)
 			(effects
@@
 			)
 		)
-		(property "Footprint" ""
+		(property "Footprint" "Package_SO:TSSOP-24_4.4x5mm_P0.4mm"
 			(at 162.56 128.27 0)
 			(effects

Commit message: organizing more components
Parts:
- R2: footprint Capacitor_SMD:C_0603_1608Metric -> Resistor_SMD:R_0402_1005Metric
Changed lines of the file:
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@@
 			)
 		)
-		(property "Footprint" "Capacitor_SMD:C_0603_1608Metric"
+		(property "Footprint" "Resistor_SMD:R_0402_1005Metric"
 			(at 49.022 132.08 90)
 			(effects

Commit message: connected unused pins 8 on a level shifter as per datasheet, thanks Strong-Mud199 on reddit :D
Connections:
- net GND: now also U2.10 (A8), U2.14 (B8)
- no-connect marks 2 -> 0
Changed lines of the file:
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@@
+	)
+	(junction
+		(at 193.04 137.16)
+		(diameter 0)
+		(color 0 0 0 0)
 	)
 	(junction
@@
 		(color 0 0 0 0)
 	)
-	(no_connect
-		(at 203.2 121.92)
-	)
-	(no_connect
-		(at 223.52 121.92)
-	)
 	(wire
 		(pts
@@
 	(wire
 		(pts
+			(xy 190.5 137.16) (xy 193.04 137.16)
+		)
+		(stroke
+			(width 0)
+			(type default)
+		)
+	)
+	(wire
+		(pts
 			(xy 129.54 111.76) (xy 132.08 111.76)
 		)
@@
 	(wire
 		(pts
+			(xy 231.14 121.92) (xy 231.14 137.16)
+		)
+		(stroke
+			(width 0)
+			(type default)
+		)
+	)
+	(wire
+		(pts
 			(xy 137.16 72.39) (xy 139.7 72.39)
 		)
@@
 	(wire
 		(pts
+			(xy 203.2 121.92) (xy 190.5 121.92)
+		)
+		(stroke
+			(width 0)
+			(type default)
+		)
+	)
+	(wire
+		(pts
 			(xy 129.54 137.16) (xy 142.24 137.16)
 		)
@@
 	(wire
 		(pts
+			(xy 190.5 121.92) (xy 190.5 137.16)
+		)
+		(stroke
+			(width 0)
+			(type default)
+		)
+	)
+	(wire
+		(pts
 			(xy 55.88 67.31) (xy 58.42 67.31)
 		)
@@
 	(wire
 		(pts
+			(xy 231.14 137.16) (xy 213.36 137.16)
+		)
+		(stroke
+			(width 0)
+			(type default)
+		)
+	)
+	(wire
+		(pts
 			(xy 200.66 96.52) (xy 203.2 96.52)
 		)
@@
 		)
 		(stroke
+			(width 0)
+			(type default)
+		)
+	)
+	(wire
+		(pts
+			(xy 231.14 121.92) (xy 223.52 121.92)
+		)
+		(stroke

Commit message: changed the board stackup, doing LOTS of research on how EMI/Signal integrity works
Changed lines of the file:
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@@
 	(wire
 		(pts
-			(xy 190.5 137.16) (xy 193.04 137.16)
+			(xy 189.23 137.16) (xy 193.04 137.16)
 		)
 		(stroke
@@
 	(wire
 		(pts
-			(xy 203.2 121.92) (xy 190.5 121.92)
+			(xy 203.2 121.92) (xy 189.23 121.92)
 		)
 		(stroke
@@
 	(wire
 		(pts
-			(xy 190.5 121.92) (xy 190.5 137.16)
-		)
-		(stroke
+			(xy 189.23 121.92) (xy 189.23 137.16)
+		)
+		(stroke

Commit message: moving level shifting pins to be easier to route
Connections:
- net FAN_PWM_1V8: now also U2.9 (A7); no longer U2.8 (A6)
- net FAN_PWM_3V3: now also U2.15 (B7); no longer U2.16 (B6)
- net FAN_TACH_1V8: now also U3.21 (B1); no longer U3.14 (B8)
- net FAN_TACH_3V3: now also U3.3 (A1); no longer U3.10 (A8)
- net GPIO0_1V8: now also U2.5 (A3); no longer U2.9 (A7)
- net GPIO0_3V3: now also U2.19 (B3); no longer U2.15 (B7)
- net SPI-0_CLK_1V8: now also U1.5 (A3); no longer U1.4 (A2)
- net SPI-0_CLK_3V3: now also U1.19 (B3); no longer U1.20 (B2)
- net SPI-0_CS0_1V8: now also U1.7 (A5); no longer U1.5 (A3)
- net SPI-0_CS0_3V3: now also U1.17 (B5); no longer U1.19 (B3)
- net SPI-0_CS1_1V8: now also U1.8 (A6); no longer U1.6 (A4)
- net SPI-0_CS1_3V3: now also U1.16 (B6); no longer U1.18 (B4)
- net SPI-0_MISO_1V8: now also U3.15 (B7); no longer U3.21 (B1)
- net SPI-0_MISO_3V3: now also U3.9 (A7); no longer U3.3 (A1)
- net SPI-0_MOSI_1V8: now also U1.4 (A2); no longer U1.3 (A1)
- net SPI-0_MOSI_3V3: now also U1.20 (B2); no longer U1.21 (B1)
- net SPI-1_CLK_1V8: now also U1.10 (A8); no longer U1.8 (A6)
- net SPI-1_CLK_3V3: now also U1.14 (B8); no longer U1.16 (B6)
- net SPI-1_CS0_1V8: now also U1.6 (A4); no longer U1.9 (A7)
- net SPI-1_CS0_3V3: now also U1.18 (B4); no longer U1.15 (B7)
- net SPI-1_CS1_1V8: now also U1.3 (A1); no longer U1.10 (A8)
- net SPI-1_CS1_3V3: now also U1.21 (B1); no longer U1.14 (B8)
- net SPI-1_MISO_1V8: now also U3.19 (B3); no longer U3.20 (B2)
- net SPI-1_MISO_3V3: now also U3.5 (A3); no longer U3.4 (A2)
- net SPI-1_MOSI_1V8: now also U1.9 (A7); no longer U1.7 (A5)
- net SPI-1_MOSI_3V3: now also U1.15 (B7); no longer U1.17 (B5)
- net UART-0_CTS_1V8: now also U3.14 (B8); no longer U3.18 (B4)
- net UART-0_CTS_3V3: now also U3.10 (A8); no longer U3.6 (A4)
- net UART-0_RTS_1V8: now also U2.3 (A1); no longer U2.4 (A2)
- net UART-0_RTS_3V3: now also U2.21 (B1); no longer U2.20 (B2)
- net UART-0_RX_1V8: now also U3.20 (B2); no longer U3.19 (B3)
- net UART-0_RX_3V3: now also U3.4 (A2); no longer U3.5 (A3)
- net UART-0_TX_1V8: now also U2.6 (A4); no longer U2.3 (A1)
- net UART-0_TX_3V3: now also U2.18 (B4); no longer U2.21 (B1)
- net UART-1_CTS_1V8: now also U3.18 (B4); no longer U3.16 (B6)
- net UART-1_CTS_3V3: now also U3.6 (A4); no longer U3.8 (A6)
- net UART-1_RTS_1V8: now also U2.7 (A5); no longer U2.6 (A4)
- net UART-1_RTS_3V3: now also U2.17 (B5); no longer U2.18 (B4)
- net UART-1_TX_1V8: now also U2.8 (A6); no longer U2.5 (A3)
- net UART-1_TX_3V3: now also U2.16 (B6); no longer U2.19 (B3)
- net UART-2_RX_1V8: now also U3.16 (B6); no longer U3.15 (B7)
- net UART-2_RX_3V3: now also U3.8 (A6); no longer U3.9 (A7)
- net UART-2_TX_1V8: now also U2.4 (A2); no longer U2.7 (A5)
- net UART-2_TX_3V3: now also U2.20 (B2); no longer U2.17 (B5)

Commit message: changing level shifting pinout, to have an organized pinout and not pinin for easy routing to tight via's
Connections:
- net FAN_PWM_1V8: now also U2.8 (A6); no longer U2.9 (A7)
- net FAN_PWM_3V3: now also U2.16 (B6); no longer U2.15 (B7)
- net FAN_TACH_1V8: now also U3.19 (B3); no longer U3.21 (B1)
- net FAN_TACH_3V3: now also U3.5 (A3); no longer U3.3 (A1)
- net GPIO0_1V8: now also U2.3 (A1); no longer U2.5 (A3)
- net GPIO0_3V3: now also U2.21 (B1); no longer U2.19 (B3)
- net SPI-0_CLK_1V8: now also U1.4 (A2); no longer U1.5 (A3)
- net SPI-0_CLK_3V3: now also U1.20 (B2); no longer U1.19 (B3)
- net SPI-0_CS0_1V8: now also U1.5 (A3); no longer U1.7 (A5)
- net SPI-0_CS0_3V3: now also U1.19 (B3); no longer U1.17 (B5)
- net SPI-0_CS1_1V8: now also U1.6 (A4); no longer U1.8 (A6)
- net SPI-0_CS1_3V3: now also U1.18 (B4); no longer U1.16 (B6)
- net SPI-0_MISO_1V8: now also U3.14 (B8); no longer U3.15 (B7)
- net SPI-0_MISO_3V3: now also U3.10 (A8); no longer U3.9 (A7)
- net SPI-0_MOSI_1V8: now also U1.3 (A1); no longer U1.4 (A2)
- net SPI-0_MOSI_3V3: now also U1.21 (B1); no longer U1.20 (B2)
- net SPI-1_CLK_1V8: now also U1.7 (A5); no longer U1.10 (A8)
- net SPI-1_CLK_3V3: now also U1.17 (B5); no longer U1.14 (B8)
- net SPI-1_CS0_1V8: now also U1.10 (A8); no longer U1.6 (A4)
- net SPI-1_CS0_3V3: now also U1.14 (B8); no longer U1.18 (B4)
- net SPI-1_CS1_1V8: now also U1.9 (A7); no longer U1.3 (A1)
- net SPI-1_CS1_3V3: now also U1.15 (B7); no longer U1.21 (B1)
- net SPI-1_MISO_1V8: now also U3.17 (B5); no longer U3.19 (B3)
- net SPI-1_MISO_3V3: now also U3.7 (A5); no longer U3.5 (A3)
- net SPI-1_MOSI_1V8: now also U1.8 (A6); no longer U1.9 (A7)
- net SPI-1_MOSI_3V3: now also U1.16 (B6); no longer U1.15 (B7)
- net UART-0_CTS_1V8: now also U3.16 (B6); no longer U3.14 (B8)
- net UART-0_CTS_3V3: now also U3.8 (A6); no longer U3.10 (A8)
- net UART-0_RTS_1V8: now also U2.5 (A3); no longer U2.3 (A1)
- net UART-0_RTS_3V3: now also U2.19 (B3); no longer U2.21 (B1)
- net UART-0_RX_1V8: now also U3.15 (B7); no longer U3.20 (B2)
- net UART-0_RX_3V3: now also U3.9 (A7); no longer U3.4 (A2)
- net UART-0_TX_1V8: now also U2.4 (A2); no longer U2.6 (A4)
- net UART-0_TX_3V3: now also U2.20 (B2); no longer U2.18 (B4)
- net UART-1_CTS_1V8: now also U3.20 (B2); no longer U3.18 (B4)
- net UART-1_CTS_3V3: now also U3.4 (A2); no longer U3.6 (A4)
- net UART-1_RX_1V8: now also U3.18 (B4); no longer U3.17 (B5)
- net UART-1_RX_3V3: now also U3.6 (A4); no longer U3.7 (A5)
- net UART-1_TX_1V8: now also U2.6 (A4); no longer U2.8 (A6)
- net UART-1_TX_3V3: now also U2.18 (B4); no longer U2.16 (B6)
- net UART-2_RX_1V8: now also U3.21 (B1); no longer U3.16 (B6)
- net UART-2_RX_3V3: now also U3.3 (A1); no longer U3.8 (A6)
- net UART-2_TX_1V8: now also U2.9 (A7); no longer U2.4 (A2)
- net UART-2_TX_3V3: now also U2.15 (B7); no longer U2.20 (B2)

Commit message: adding dampening resistors to SPI - schematic
Connections:
- net SPI-0_CLK_1V8 renamed dSPI-0_CLK_1V8
- net SPI-0_CS0_1V8 renamed dSPI-0_CS0_1V8
- net SPI-0_CS1_1V8 renamed dSPI-0_CS1_1V8
- net SPI-0_MISO_3V3 renamed dSPI-0_MISO_3V3
- net SPI-0_MOSI_1V8 renamed dSPI-0_MOSI_1V8
- net SPI-1_CLK_1V8 renamed dSPI-1_CLK_1V8
- net SPI-1_CS0_1V8 renamed dSPI-1_CS0_1V8
- net SPI-1_CS1_1V8 renamed dSPI-1_CS1_1V8
- net SPI-1_MISO_3V3 renamed dSPI-1_MISO_3V3
- net SPI-1_MOSI_1V8 renamed dSPI-1_MOSI_1V8
Changed lines of the file:
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@@
 		)
 	)
-	(global_label "SPI-1_CS1_1V8"
+	(global_label "dSPI-1_CS1_1V8"
 		(shape output)
 		(at 58.42 116.84 180)
@@
 		)
 		(property "Intersheetrefs" "${INTERSHEET_REFS}"
-			(at 40.3417 116.84 0)
-			(effects
-				(font
-					(size 1.27 1.27)
-				)
-				(justify right)
-				(hide yes)
-			)
-		)
-	)
-	(global_label "SPI-0_CS0_1V8"
+			(at 39.1927 116.84 0)
+			(effects
+				(font
+					(size 1.27 1.27)
+				)
+				(justify right)
+				(hide yes)
+			)
+		)
+	)
+	(global_label "dSPI-0_CS0_1V8"
 		(shape output)
 		(at 58.42 96.52 180)
@@
 		)
 		(property "Intersheetrefs" "${INTERSHEET_REFS}"
-			(at 40.3417 96.52 0)
+			(at 39.1927 96.52 0)
 			(effects
 				(font
@@
 		)
 	)
-	(global_label "SPI-1_MISO_3V3"
+	(global_label "dSPI-1_MISO_3V3"
 		(shape output)
 		(at 129.54 106.68 180)
@@
 		)
 		(property "Intersheetrefs" "${INTERSHEET_REFS}"
-			(at 110.5545 106.68 0)
+			(at 109.4055 106.68 0)
 			(effects
 				(font
@@
 		)
 	)
-	(global_label "SPI-1_CLK_1V8"
+	(global_label "dSPI-1_CLK_1V8"
 		(shape output)
 		(at 58.42 106.68 180)
@@
 		)
 		(property "Intersheetrefs" "${INTERSHEET_REFS}"
-			(at 40.4626 106.68 0)
+			(at 39.3136 106.68 0)
 			(effects
 				(font
@@
 		)
 	)
-	(global_label "SPI-1_MOSI_1V8"
+	(global_label "dSPI-1_MOSI_1V8"
 		(shape output)
 		(at 58.42 111.76 180)
@@
 		)
 		(property "Intersheetrefs" "${INTERSHEET_REFS}"
-			(at 39.4345 111.76 0)
+			(at 38.2855 111.76 0)
 			(effects
 				(font
@@
 		)
 	)
-	(global_label "SPI-0_MOSI_1V8"
+	(global_label "dSPI-0_MOSI_1V8"
 		(shape output)
 		(at 58.42 86.36 180)
@@
 		)
 		(property "Intersheetrefs" "${INTERSHEET_REFS}"
-			(at 39.4345 86.36 0)
+			(at 38.2855 86.36 0)
 			(effects
 				(font
@@
 		)
 	)
-	(global_label "SPI-0_CS1_1V8"
+	(global_label "dSPI-0_CS1_1V8"
 		(shape output)
 		(at 58.42 101.6 180)
@@
 		)
 		(property "Intersheetrefs" "${INTERSHEET_REFS}"
-			(at 40.3417 101.6 0)
+			(at 39.1927 101.6 0)
 			(effects
 				(font
@@
 		)
 	)
-	(global_label "SPI-0_MISO_3V3"
+	(global_label "dSPI-0_MISO_3V3"
 		(shape output)
 		(at 129.54 121.92 180)
@@
 		)
 		(property "Intersheetrefs" "${INTERSHEET_REFS}"
-			(at 110.5545 121.92 0)
-			(effects
-				(font
-					(size 1.27 1.27)
-				)
-				(justify right)
-				(hide yes)
-			)
-		)
-	)
-	(global_label "SPI-0_CLK_1V8"
+			(at 109.4055 121.92 0)
+			(effects
+				(font
+					(size 1.27 1.27)
+				)
+				(justify right)
+				(hide yes)
+			)
+		)
+	)
+	(global_label "dSPI-0_CLK_1V8"
 		(shape output)
 		(at 58.42 91.44 180)
@@
 		)
 		(property "Intersheetrefs" "${INTERSHEET_REFS}"
-			(at 40.4626 91.44 0)
+			(at 39.3136 91.44 0)
 			(effects
 				(font
@@
 		)
 	)
-	(global_label "SPI-1_CS0_1V8"
+	(global_label "dSPI-1_CS0_1V8"
 		(shape output)
 		(at 58.42 121.92 180)
@@
 		)
 		(property "Intersheetrefs" "${INTERSHEET_REFS}"
-			(at 40.3417 121.92 0)
-			(effects
-				(font
+			(at 39.1927 121.92 0)
+			(effects
+				(font
