File: PCB_CARRIER/carrier.kicad_sch (KiCad schematic)
At the start: 0 parts

Commit message: updating journal
Other:
- added sheet Carrier SO-DIMM (SO-DIMM.kicad_sch)
- title: Raspberry Pi Compute Module 4 Carrier Template -> CM4/CM5 Carrier Board
Changed lines of the file:
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@@
 	(paper "A4")
 	(title_block
-		(title "Raspberry Pi Compute Module 4 Carrier Template")
-		(date "2020-10-31")
-		(rev "v01")
-		(comment 2 "creativecommons.org/licenses/by-sa/4.0/")
-		(comment 3 "License: CC BY 4.0")
-		(comment 4 "Author: Shawn Hymel")
+		(title "CM4/CM5 Carrier Board")
 	)
 	(sheet
-		(at 101.6 101.6)
+		(at 24.13 121.92)
+		(size 38.1 38.1)
+		(exclude_from_sim no)
+		(in_bom yes)
+		(on_board yes)
+		(dnp no)
+		(fields_autoplaced yes)
+		(stroke
+			(width 0.1524)
+			(type solid)
+		)
+		(fill
+			(color 0 0 0 0.0000)
+		)
+		(property "Sheetname" "Carrier SO-DIMM"
+			(at 24.13 121.2084 0)
+			(effects
+				(font
+					(size 1.27 1.27)
+				)
+				(justify left bottom)
+			)
+		)
+		(property "Sheetfile" "SO-DIMM.kicad_sch"
+			(at 24.13 160.6046 0)
+			(effects
+				(font
+					(size 1.27 1.27)
+				)
+				(justify left top)
+			)
+		)
+		(instances
+			(project "carrier"
+				(path "/f52509e6-8053-454c-b8e9-3e2670c5a5fe"
+					(page "4")
+				)
+			)
+		)
+	)
+	(sheet
+		(at 24.13 73.66)
 		(size 38.1 38.1)
 		(exclude_from_sim no)
@@
 		)
 		(property "Sheetname" "CM4 High Speed"
-			(at 101.6 100.9645 0)
+			(at 24.13 73.0245 0)
 			(effects
 				(font
@@
 		)
 		(property "Sheetfile" "cm4-high-speed.kicad_sch"
-			(at 101.6 140.2085 0)
+			(at 24.13 112.2685 0)
 			(effects
 				(font
@@
 		)
 		(instances
-			(project "rpi-cm4-carrier-template"
+			(project "carrier"
 				(path "/f52509e6-8053-454c-b8e9-3e2670c5a5fe"
 					(page "3")
@@
 	)
 	(sheet
-		(at 101.6 50.8)
+		(at 24.13 25.4)
 		(size 38.1 38.1)
 		(exclude_from_sim no)
@@
 		)
 		(property "Sheetname" "CM4 GPIO"
-			(at 101.6 50.1645 0)
+			(at 24.13 24.7645 0)
 			(effects
 				(font
@@
 		)
 		(property "Sheetfile" "cm4-gpio.kicad_sch"
-			(at 101.6 89.4085 0)
+			(at 24.13 64.0085 0)
 			(effects
 				(font
@@
 		)
 		(instances
-			(project "rpi-cm4-carrier-template"
+			(project "carrier"
 				(path "/f52509e6-8053-454c-b8e9-3e2670c5a5fe"
 					(page "3")

Commit message: working on level shifting
Other:
- added sheet Level Shifting (level-shifting.kicad_sch)
Changed lines of the file:
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@@
+	)
+	(sheet
+		(at 71.12 25.4)
+		(size 38.1 38.1)
+		(exclude_from_sim no)
+		(in_bom yes)
+		(on_board yes)
+		(dnp no)
+		(fields_autoplaced yes)
+		(stroke
+			(width 0.1524)
+			(type solid)
+		)
+		(fill
+			(color 0 0 0 0.0000)
+		)
+		(property "Sheetname" "Level Shifting"
+			(at 71.12 24.6884 0)
+			(effects
+				(font
+					(size 1.27 1.27)
+				)
+				(justify left bottom)
+			)
+		)
+		(property "Sheetfile" "level-shifting.kicad_sch"
+			(at 71.12 64.0846 0)
+			(effects
+				(font
+					(size 1.27 1.27)
+				)
+				(justify left top)
+			)
+		)
+		(instances
+			(project "carrier"
+				(path "/f52509e6-8053-454c-b8e9-3e2670c5a5fe"
+					(page "5")
+				)
+			)
+		)
 	)
 	(sheet

Commit message: starting on damping resistors
Other:
- added sheet Damping Resistors (damping-resistors.kicad_sch)
Changed lines of the file:
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@@
+	)
+	(sheet
+		(at 71.12 73.66)
+		(size 38.1 38.1)
+		(exclude_from_sim no)
+		(in_bom yes)
+		(on_board yes)
+		(dnp no)
+		(fields_autoplaced yes)
+		(stroke
+			(width 0.1524)
+			(type solid)
+		)
+		(fill
+			(color 0 0 0 0.0000)
+		)
+		(property "Sheetname" "Damping Resistors"
+			(at 71.12 72.9484 0)
+			(effects
+				(font
+					(size 1.27 1.27)
+				)
+				(justify left bottom)
+			)
+		)
+		(property "Sheetfile" "damping-resistors.kicad_sch"
+			(at 71.12 112.3446 0)
+			(effects
+				(font
+					(size 1.27 1.27)
+				)
+				(justify left top)
+			)
+		)
+		(instances
+			(project "carrier"
+				(path "/f52509e6-8053-454c-b8e9-3e2670c5a5fe"
+					(page "6")
+				)
+			)
+		)
 	)
 	(sheet

Commit message: working on testing points
Other:
- added sheet Testing Points (testing-points.kicad_sch)
Changed lines of the file:
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@@
+	)
+	(sheet
+		(at 71.12 121.92)
+		(size 38.1 38.1)
+		(exclude_from_sim no)
+		(in_bom yes)
+		(on_board yes)
+		(dnp no)
+		(fields_autoplaced yes)
+		(stroke
+			(width 0.1524)
+			(type solid)
+		)
+		(fill
+			(color 0 0 0 0.0000)
+		)
+		(property "Sheetname" "Testing Points"
+			(at 71.12 121.2084 0)
+			(effects
+				(font
+					(size 1.27 1.27)
+				)
+				(justify left bottom)
+			)
+		)
+		(property "Sheetfile" "testing-points.kicad_sch"
+			(at 71.12 160.6046 0)
+			(effects
+				(font
+					(size 1.27 1.27)
+				)
+				(justify left top)
+			)
+		)
+		(instances
+			(project "carrier"
+				(path "/f52509e6-8053-454c-b8e9-3e2670c5a5fe"
+					(page "7")
+				)
+			)
+		)
 	)
 	(sheet

Commit message: removing and adding some test points to the schematic
Other:
- removed sheet Testing Points
- added sheet Test Points (test-points.kicad_sch)
Changed lines of the file:
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@@
 			(color 0 0 0 0.0000)
 		)
-		(property "Sheetname" "Testing Points"
+		(property "Sheetname" "Test Points"
 			(at 71.12 121.2084 0)
 			(effects
@@
 			)
 		)
-		(property "Sheetfile" "testing-points.kicad_sch"
+		(property "Sheetfile" "test-points.kicad_sch"
 			(at 71.12 160.6046 0)
 			(effects

Commit message: finished adding test points
Other:
- removed sheet Test Points
Changed lines of the file:
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@@
-	)
-	(sheet
-		(at 71.12 121.92)
-		(size 38.1 38.1)
-		(exclude_from_sim no)
-		(in_bom yes)
-		(on_board yes)
-		(dnp no)
-		(fields_autoplaced yes)
-		(stroke
-			(width 0.1524)
-			(type solid)
-		)
-		(fill
-			(color 0 0 0 0.0000)
-		)
-		(property "Sheetname" "Test Points"
-			(at 71.12 121.2084 0)
-			(effects
-				(font
-					(size 1.27 1.27)
-				)
-				(justify left bottom)
-			)
-		)
-		(property "Sheetfile" "test-points.kicad_sch"
-			(at 71.12 160.6046 0)
-			(effects
-				(font
-					(size 1.27 1.27)
-				)
-				(justify left top)
-			)
-		)
-		(instances
-			(project "carrier"
-				(path "/f52509e6-8053-454c-b8e9-3e2670c5a5fe"
-					(page "7")
-				)
-			)
-		)
 	)
 	(sheet
