File: PCB_CARRIER/test-points.kicad_sch (KiCad schematic)
At the start: 2 parts

Commit message: finished adding test points
Parts:
- removed TP1: RTC Test, symbol Connector:TestPoint
- removed TP2: Sleep Status Output, symbol Connector:TestPoint
