File: PCB_CARRIER/damping-resistors.kicad_sch (KiCad schematic)
At the start: 0 parts

Commit message: fixed some label names for routing
Changed lines of the file:
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@@
 	(paper "A4")
 	(global_label "USB_P"
-		(shape input)
+		(shape bidirectional)
 		(at 82.55 80.01 180)
 		(fields_autoplaced yes)
@@
 		)
 		(property "Intersheetrefs" "${INTERSHEET_REFS}"
-			(at 73.4221 80.01 0)
+			(at 72.4061 80.01 0)
 			(effects
 				(font
@@
 	)
 	(global_label "USB3-1-DM"
-		(shape input)
+		(shape bidirectional)
 		(at 82.55 68.58 180)
 		(fields_autoplaced yes)
@@
 		)
 		(property "Intersheetrefs" "${INTERSHEET_REFS}"
-			(at 67.3745 68.58 0)
+			(at 66.3585 68.58 0)
 			(effects
 				(font
@@
 	)
 	(global_label "USB3-1-DP"
-		(shape input)
+		(shape bidirectional)
 		(at 82.55 72.39 180)
 		(fields_autoplaced yes)
@@
 		)
 		(property "Intersheetrefs" "${INTERSHEET_REFS}"
-			(at 67.5559 72.39 0)
+			(at 66.5399 72.39 0)
 			(effects
 				(font
@@
 	)
 	(global_label "USB3-0-DP"
-		(shape input)
+		(shape bidirectional)
 		(at 82.55 64.77 180)
 		(fields_autoplaced yes)
@@
 		)
 		(property "Intersheetrefs" "${INTERSHEET_REFS}"
-			(at 67.5559 64.77 0)
+			(at 66.5399 64.77 0)
 			(effects
 				(font
@@
 	)
 	(global_label "USB3-0-DM"
-		(shape input)
+		(shape bidirectional)
 		(at 82.55 60.96 180)
 		(fields_autoplaced yes)
@@
 		)
 		(property "Intersheetrefs" "${INTERSHEET_REFS}"
-			(at 67.3745 60.96 0)
+			(at 66.3585 60.96 0)
 			(effects
 				(font
@@
 		)
 	)
-	(global_label "USB_N"
-		(shape input)
+	(global_label "USB_M"
+		(shape bidirectional)
 		(at 82.55 76.2 180)
 		(fields_autoplaced yes)
@@
 		)
 		(property "Intersheetrefs" "${INTERSHEET_REFS}"
-			(at 73.3616 76.2 0)
+			(at 72.2247 76.2 0)
 			(effects
 				(font

Commit message: terminations on USB M/P
Parts:
- added R22, R23, R24, R25, R26, R27: 22, symbol Device:R
Connections:
- net USB3-0-DM: now also R22.1, R22.2
- net USB3-0-DP: now also R23.1, R23.2
- net USB3-1-DM: now also R24.1, R24.2
- net USB3-1-DP: now also R25.1, R25.2
- net USB_M: now also R26.1, R26.2
- net USB_P: now also R27.1, R27.2

Commit message: dampened CSI0
Parts:
- added R28, R29, R30, R31, R32, R33, R34, R35, R36, R37, R38, R39, R40, R41, R42, R43: 22, symbol Device:R
Connections:
- new net CSI-0_CLK_N: R34.1, R34.2
- new net CSI-0_CLK_P: R35.1, R35.2
- new net CSI-0_D0_N: R36.1, R36.2
- new net CSI-0_D0_P: R37.1, R37.2
- new net CSI-0_D1_N: R38.1, R38.2
- new net CSI-0_D1_P: R39.1, R39.2
- new net CSI-0_D2_N: R40.1, R40.2
- new net CSI-0_D2_P: R41.1, R41.2
- new net CSI-0_D3_N: R42.1, R42.2
- new net CSI-0_D3_P: R43.1, R43.2
- new net HDMI-0_TX0_N: R28.1, R28.2
- new net HDMI-0_TX0_P: R29.1, R29.2
- new net HDMI-0_TX1_N: R30.1, R30.2
- new net HDMI-0_TX1_P: R31.1, R31.2
- new net HDMI-0_TX2_N: R32.1, R32.2
- new net HDMI-0_TX2_P: R33.1, R33.2

Commit message: damping on CSI 1
Parts:
- added R44, R45, R46, R47, R48, R49, R50, R51, R52, R53: 22, symbol Device:R
Connections:
- new net CSI-1_CLK_N: R44.1, R44.2
- new net CSI-1_CLK_P: R45.1, R45.2
- new net CSI-1_D0_N: R46.1, R46.2
- new net CSI-1_D0_P: R47.1, R47.2
- new net CSI-1_D1_N: R48.1, R48.2
- new net CSI-1_D1_P: R49.1, R49.2
- new net CSI-1_D2_N: R50.1, R50.2
- new net CSI-1_D2_P: R51.1, R51.2
- new net CSI-1_D3_N: R52.1, R52.2
- new net CSI-1_D3_P: R53.1, R53.2
Other:
- moved on the sheet: R22, R23, R24, R25, R26, R27, R28, R29, R30, R31, R32, R33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

Commit message: footprints for passives
Parts:
- R22, R23, R24, R25, R26, R27, R28, R29, R30, R31, R32, R33, R34, R35, R36, R37, R38, R39, R40, R41, R42, R43, R44, R45, R46, R47, R48, R49, R50, R51, R52, R53: footprint (none) -> Resistor_SMD:R_0402_1005Metric
Changed lines of the file:
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@@
 			)
 		)
-		(property "Footprint" ""
+		(property "Footprint" "Resistor_SMD:R_0402_1005Metric"
 			(at 63.5 89.408 90)
 			(effects
@@
 			)
 		)
-		(property "Footprint" ""
+		(property "Footprint" "Resistor_SMD:R_0402_1005Metric"
 			(at 123.19 84.328 90)
 			(effects
@@
 			)
 		)
-		(property "Footprint" ""
+		(property "Footprint" "Resistor_SMD:R_0402_1005Metric"
 			(at 232.41 119.888 90)
 			(effects
@@
 			)
 		)
-		(property "Footprint" ""
+		(property "Footprint" "Resistor_SMD:R_0402_1005Metric"
 			(at 232.41 74.168 90)
 			(effects
@@
 			)
 		)
-		(property "Footprint" ""
+		(property "Footprint" "Resistor_SMD:R_0402_1005Metric"
 			(at 63.5 84.328 90)
 			(effects
@@
 			)
 		)
-		(property "Footprint" ""
+		(property "Footprint" "Resistor_SMD:R_0402_1005Metric"
 			(at 123.19 89.408 90)
 			(effects
@@
 			)
 		)
-		(property "Footprint" ""
+		(property "Footprint" "Resistor_SMD:R_0402_1005Metric"
 			(at 179.07 114.808 90)
 			(effects
@@
 			)
 		)
-		(property "Footprint" ""
+		(property "Footprint" "Resistor_SMD:R_0402_1005Metric"
 			(at 179.07 74.168 90)
 			(effects
@@
 			)
 		)
-		(property "Footprint" ""
+		(property "Footprint" "Resistor_SMD:R_0402_1005Metric"
 			(at 232.41 109.728 90)
 			(effects
@@
 			)
 		)
-		(property "Footprint" ""
+		(property "Footprint" "Resistor_SMD:R_0402_1005Metric"
 			(at 232.41 79.248 90)
 			(effects
@@
 			)
 		)
-		(property "Footprint" ""
+		(property "Footprint" "Resistor_SMD:R_0402_1005Metric"
 			(at 232.41 89.408 90)
 			(effects
@@
 			)
 		)
-		(property "Footprint" ""
+		(property "Footprint" "Resistor_SMD:R_0402_1005Metric"
 			(at 123.19 74.168 90)
 			(effects
@@
 			)
 		)
-		(property "Footprint" ""
+		(property "Footprint" "Resistor_SMD:R_0402_1005Metric"
 			(at 179.07 94.488 90)
 			(effects
@@
 			)
 		)
-		(property "Footprint" ""
+		(property "Footprint" "Resistor_SMD:R_0402_1005Metric"
 			(at 232.41 114.808 90)
 			(effects
@@
 			)
 		)
-		(property "Footprint" ""
+		(property "Footprint" "Resistor_SMD:R_0402_1005Metric"
 			(at 179.07 119.888 90)
 			(effects
@@
 			)
 		)
-		(property "Footprint" ""
+		(property "Footprint" "Resistor_SMD:R_0402_1005Metric"
 			(at 232.41 104.648 90)
 			(effects
@@
 			)
 		)
-		(property "Footprint" ""
+		(property "Footprint" "Resistor_SMD:R_0402_1005Metric"
 			(at 179.07 104.648 90)
 			(effects
@@
 			)
 		)
-		(property "Footprint" ""
+		(property "Footprint" "Resistor_SMD:R_0402_1005Metric"
 			(at 232.41 84.328 90)
 			(effects
@@
 			)
 		)
-		(property "Footprint" ""
+		(property "Footprint" "Resistor_SMD:R_0402_1005Metric"
 			(at 179.07 99.568 90)
 			(effects
@@
 			)
 		)
-		(property "Footprint" ""
+		(property "Footprint" "Resistor_SMD:R_0402_1005Metric"
 			(at 232.41 94.488 90)
 			(effects
@@
 			)
 		)
-		(property "Footprint" ""
+		(property "Footprint" "Resistor_SMD:R_0402_1005Metric"
 			(at 63.5 99.568 90)
 			(effects
@@
 			)
 		)
-		(property "Footprint" ""
+		(property "Footprint" "Resistor_SMD:R_0402_1005Metric"
 			(at 63.5 79.248 90)
 			(effects
@@
 			)
 		)
-		(property "Footprint" ""
+		(property "Footprint" "Resistor_SMD:R_0402_1005Metric"
 			(at 232.41 99.568 90)
 			(effects
@@
 			)
 		)
-		(property "Footprint" ""
+		(property "Footprint" "Resistor_SMD:R_0402_1005Metric"
 			(at 123.19 79.248 90)
 			(effects
@@
 			)
 		)
-		(property "Footprint" ""
+		(property "Footprint" "Resistor_SMD:R_0402_1005Metric"
 			(at 123.19 94.488 90)
 			(effects
@@
 			)
 		)
-		(property "Footprint" ""
+		(property "Footprint" "Resistor_SMD:R_0402_1005Metric"
 			(at 179.07 89.408 90)
 			(effects
@@
 			)
 		)
-		(property "Footprint" ""
+		(property "Footprint" "Resistor_SMD:R_0402_1005Metric"
 			(at 179.07 79.248 90)
 			(effects
@@
 			)
 		)
-		(property "Footprint" ""
+		(property "Footprint" "Resistor_SMD:R_0402_1005Metric"
 			(at 179.07 109.728 90)
 			(effects
@@
 			)
 		)
-		(property "Footprint" ""
+		(property "Footprint" "Resistor_SMD:R_0402_1005Metric"
 			(at 179.07 84.328 90)
 			(effects
@@
 			)
 		)
-		(property "Footprint" ""
+		(property "Footprint" "Resistor_SMD:R_0402_1005Metric"
 			(at 63.5 74.168 90)
 			(effects
@@
 			)
 		)
-		(property "Footprint" ""
+		(property "Footprint" "Resistor_SMD:R_0402_1005Metric"
 			(at 63.5 94.488 90)
 			(effects
@@
 			)
 		)
-		(property "Footprint" ""
+		(property "Footprint" "Resistor_SMD:R_0402_1005Metric"
 			(at 123.19 99.568 90)
 			(effects

Commit message: fixed dampening resistors, decent commit to revert too
Connections:
- net CSI-0_CLK_N: no longer R34.1
- net CSI-0_CLK_P: no longer R35.1
- net CSI-0_D0_N: no longer R36.1
- net CSI-0_D0_P: no longer R37.1
- net CSI-0_D1_N: no longer R38.1
- net CSI-0_D1_P: no longer R39.1
- net CSI-0_D2_N: no longer R40.1
- net CSI-0_D2_P: no longer R41.1
- net CSI-0_D3_N: no longer R42.1
- net CSI-0_D3_P: no longer R43.1
- net CSI-1_CLK_N: no longer R44.1
- net CSI-1_CLK_P: no longer R45.1
- net CSI-1_D0_N: no longer R46.1
- net CSI-1_D0_P: no longer R47.1
- net CSI-1_D1_N: no longer R48.1
- net CSI-1_D1_P: no longer R49.1
- net CSI-1_D2_N: no longer R50.1
- net CSI-1_D2_P: no longer R51.1
- net CSI-1_D3_N: no longer R52.1
- net CSI-1_D3_P: no longer R53.1
- net HDMI-0_TX0_N: no longer R28.2
- net HDMI-0_TX0_P: no longer R29.2
- net HDMI-0_TX1_N: no longer R30.2
- net HDMI-0_TX1_P: no longer R31.2
- net HDMI-0_TX2_N: no longer R32.2
- net HDMI-0_TX2_P: no longer R33.2
- net USB3-0-DM: no longer R22.2
- net USB3-0-DP: no longer R23.2
- net USB3-1-DM: no longer R24.2
- net USB3-1-DP: no longer R25.2
- net USB_M: no longer R26.2
- net USB_P: no longer R27.2
- new net dCSI-0_CLK_N: R34.1
- new net dCSI-0_CLK_P: R35.1
- new net dCSI-0_D0_N: R36.1
- new net dCSI-0_D0_P: R37.1
- new net dCSI-0_D1_N: R38.1
- new net dCSI-0_D1_P: R39.1
- new net dCSI-0_D2_N: R40.1
- new net dCSI-0_D2_P: R41.1
- new net dCSI-0_D3_N: R42.1
- new net dCSI-0_D3_P: R43.1
- new net dCSI-1_CLK_N: R44.1
- new net dCSI-1_CLK_P: R45.1
- new net dCSI-1_D0_N: R46.1
- new net dCSI-1_D0_P: R47.1
- new net dCSI-1_D1_N: R48.1
- new net dCSI-1_D1_P: R49.1
- new net dCSI-1_D2_N: R50.1
- new net dCSI-1_D2_P: R51.1
- new net dCSI-1_D3_N: R52.1
- new net dCSI-1_D3_P: R53.1
- new net dHDMI-0_TX0_N: R28.2
- new net dHDMI-0_TX0_P: R29.2
- new net dHDMI-0_TX1_N: R30.2
- new net dHDMI-0_TX1_P: R31.2
- new net dHDMI-0_TX2_N: R32.2
- new net dHDMI-0_TX2_P: R33.2
- new net dUSB3-0-DM: R22.2
- new net dUSB3-0-DP: R23.2
- new net dUSB3-1-DM: R24.2
- new net dUSB3-1-DP: R25.2
- new net dUSB_M: R26.2
- new net dUSB_P: R27.2
Other:
- moved on the sheet: R22, R23, R24, R25, R26, R27, R28, R29, R30, R31, R32, R33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

Commit message: removing and adding some test points to the schematic
Parts:
- R22, R23, R24, R25, R26, R27, R28, R29, R30, R31, R32, R33, R34, R35, R36, R37, R38, R39, R40, R41, R42, R43, R44, R45, R46, R47, R48, R49, R50, R51, R52, R53: value 22 -> 0

Commit message: renaming all labels to use N instead of M
Connections:
- net USB3-0-DM renamed USB3-0-DN
- net USB3-1-DM renamed USB3-1-DN
- net USB_M renamed USB_N
Changed lines of the file:
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@@
 		)
 	)
-	(global_label "USB3-1-DM"
+	(global_label "USB3-1-DN"
 		(shape bidirectional)
 		(at 54.61 82.55 180)
@@
 		)
 		(property "Intersheetrefs" "${INTERSHEET_REFS}"
-			(at 38.4185 82.55 0)
+			(at 38.5394 82.55 0)
 			(effects
 				(font
@@
 		)
 	)
-	(global_label "USB3-0-DM"
+	(global_label "USB3-0-DN"
 		(shape bidirectional)
 		(at 54.61 72.39 180)
@@
 		)
 		(property "Intersheetrefs" "${INTERSHEET_REFS}"
-			(at 38.4185 72.39 0)
+			(at 38.5394 72.39 0)
 			(effects
 				(font
@@
 		)
 	)
-	(global_label "USB_M"
+	(global_label "USB_N"
 		(shape bidirectional)
 		(at 54.61 92.71 180)
@@
 		)
 		(property "Intersheetrefs" "${INTERSHEET_REFS}"
-			(at 44.2847 92.71 0)
-			(effects
-				(font
+			(at 44.4056 92.71 0)
+			(effects
+				(font
