File: PCB_CARRIER/damping-resistors.kicad_sch (KiCad schematic)
At the start: 32 parts

Commit message: added USB 2 netclass
Parts:
- removed R22, R23, R24, R25: 0, Resistor_SMD:R_0402_1005Metric, symbol Device:R
Other:
- moved on the sheet: R26, R27

Commit message: more damping resistors on HDMI CLK, and organizing some resistors
Parts:
- added R22, R23: 0, Resistor_SMD:R_0402_1005Metric, symbol Device:R
Connections:
- new net HDMI-0_CLK_N: R22.1
- new net HDMI-0_CLK_P: R23.1
- new net dHDMI-0_CLK_N: R22.2
- new net dHDMI-0_CLK_P: R23.2
