File: PCB_CARRIER/damping-resistors.kicad_sch (KiCad schematic)
At the start: 30 parts

Commit message: adding return via's to every single pair
Connections:
- net dUSB_M renamed dUSB_N
Changed lines of the file:
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@@
 		)
 	)
-	(global_label "dUSB_M"
+	(global_label "dUSB_N"
 		(shape bidirectional)
 		(at 66.04 72.39 0)
@@
 		)
 		(property "Intersheetrefs" "${INTERSHEET_REFS}"
-			(at 77.5143 72.39 0)
+			(at 77.3934 72.39 0)
 			(effects
 				(font

Commit message: adding dampening resistors to SPI - schematic
Parts:
- added R3, R4, R54, R55, R56, R57, R58, R59, R60, R61: 0, Resistor_SMD:R_0402_1005Metric, symbol Device:R
Connections:
- new net SPI-0_CLK_1V8: R3.1
- new net SPI-0_CS0_1V8: R4.1
- new net SPI-0_CS1_1V8: R54.1
- new net SPI-0_MISO_3V3: R55.1
- new net SPI-0_MOSI_1V8: R56.1
- new net SPI-1_CLK_1V8: R57.1
- new net SPI-1_CS0_1V8: R58.1
- new net SPI-1_CS1_1V8: R59.1
- new net SPI-1_MISO_3V3: R60.1
- new net SPI-1_MOSI_1V8: R61.1
- new net dSPI-0_CLK_1V8: R3.2
- new net dSPI-0_CS0_1V8: R4.2
- new net dSPI-0_CS1_1V8: R54.2
- new net dSPI-0_MISO_3V3: R55.2
- new net dSPI-0_MOSI_1V8: R56.2
- new net dSPI-1_CLK_1V8: R57.2
- new net dSPI-1_CS0_1V8: R58.2
- new net dSPI-1_CS1_1V8: R59.2
- new net dSPI-1_MISO_3V3: R60.2
- new net dSPI-1_MOSI_1V8: R61.2

Commit message: fixing dampening resistors to use input instead of output!
Connections:
- net SPI-0_CLK_1V8 renamed SPI-0_CLK_3V3
- net SPI-0_CS0_1V8 renamed SPI-0_CS0_3V3
- net SPI-0_CS1_1V8 renamed SPI-0_CS1_3V3
- net SPI-0_MOSI_1V8 renamed SPI-0_MOSI_3V3
- net SPI-1_CLK_1V8 renamed SPI-1_CLK_3V3
- net SPI-1_CS0_1V8 renamed SPI-1_CS0_3V3
- net SPI-1_CS1_1V8 renamed SPI-1_CS1_3V3
- net SPI-1_MOSI_1V8 renamed SPI-1_MOSI_3V3
- net dSPI-0_CLK_1V8 renamed dSPI-0_CLK_3V3
- net dSPI-0_CS0_1V8 renamed dSPI-0_CS0_3V3
- net dSPI-0_CS1_1V8 renamed dSPI-0_CS1_3V3
- net dSPI-0_MOSI_1V8 renamed dSPI-0_MOSI_3V3
- net dSPI-1_CLK_1V8 renamed dSPI-1_CLK_3V3
- net dSPI-1_CS0_1V8 renamed dSPI-1_CS0_3V3
- net dSPI-1_CS1_1V8 renamed dSPI-1_CS1_3V3
- net dSPI-1_MOSI_1V8 renamed dSPI-1_MOSI_3V3
