File: PCB_CARRIER/carrier.kicad_pcb (KiCad board)
At the start: 6 copper layers, 69.6 x 46 mm, 87 parts, among them J1 SODIMM-260_Split, J2 Micro_SD_Card_Det2, Q1 BSS138, Q2 BSS138, Q3 BSS138, Q4 BC817-40, SW1 SW_DIP_x04, U1 SN74LVC8T245, U2 SN74LVC8T245, U3 SN74LVC8T245, U4 RT9742GGJ5

Commit message: holy routing
Parts:
- moved R46 0.07 mm to (127.8, 86.6)
- moved R47 0.07 mm to (126.8, 86.6)
Routing:
- net GND: track 54.9 -> 66.6 mm, vias 52 -> 66
- net USB3-1-DP: track 8.44 -> 11.2 mm, vias 1 -> 2
- net USB3-1-DN: track 8.83 -> 11.3 mm, vias 1 -> 2
- net dCSI-1_CLK_N: track 0.00 -> 1.67 mm, vias 0 -> 1
- net dCSI-1_CLK_P: track 0.00 -> 1.67 mm, vias 0 -> 1
- net dCSI-1_D1_P: track 0.00 -> 1.09 mm, vias 0 -> 1
- net dCSI-1_D1_N: track 0.00 -> 1.09 mm, vias 0 -> 1
- net dCSI-1_D0_P: track 0.00 -> 1.08 mm, vias 0 -> 1
- net dCSI-1_D0_N: track 0.00 -> 1.08 mm, vias 0 -> 1

Commit message: yes I'm still routing CSI
Parts:
- moved R52 5.06 mm to (113.8, 85.8), turned to -45 degrees
- moved R53 4.33 mm to (114.5, 85.1), turned to -45 degrees
- moved R50 0.75 mm to (122.2, 88.1)
- moved R51 0.75 mm to (121.5, 88.8)
Routing:
- net USB3-1-RX_N: track 4.59 -> 48.6 mm
- net USB3-1-RX_P: track 4.59 -> 47.7 mm
- net USB3-1-TX_N: track 4.73 -> 46.2 mm
- net USB3-1-TX_P: track 4.73 -> 45.2 mm
- net dCSI-1_D0_N: track 1.08 -> 36.5 mm
- net dCSI-1_D0_P: track 1.08 -> 35.5 mm
- net dCSI-1_D2_N: track 0.00 -> 32.8 mm, vias 0 -> 2
- net dCSI-1_D2_P: track 0.00 -> 32.3 mm, vias 0 -> 2
- net dCSI-1_D1_N: track 1.09 -> 33.2 mm
- net dCSI-1_D1_P: track 1.09 -> 32.3 mm
- net dCSI-1_CLK_N: track 1.67 -> 28.9 mm
- net dCSI-1_CLK_P: track 1.67 -> 28.1 mm
- net dCSI-1_D3_P: track 0.00 -> 22.1 mm
- net dCSI-1_D3_N: track 0.00 -> 21.0 mm
- net CSI-1_D3_N: track 10.4 -> 16.5 mm
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
Commit message: finished routing top layer CSI
Routing:
- net dCSI-0_D2_N: track 0.00 -> 49.2 mm
- net dCSI-0_D2_P: track 0.00 -> 48.2 mm
- net dCSI-0_D3_N: track 0.00 -> 45.8 mm
- net dCSI-0_D3_P: track 0.00 -> 44.9 mm
- net USB3-1-RX_P: track 47.7 -> 47.0 mm
- net USB3-1-RX_N: track 48.6 -> 47.9 mm

Commit message: finished routing bottom CSI, just have to skew match now
Routing:
- net dCSI-0_D0_N: track 0.00 -> 56.6 mm, vias 0 -> 1
- net dCSI-0_D0_P: track 0.00 -> 55.8 mm, vias 0 -> 1
- net dCSI-0_D1_N: track 0.00 -> 50.4 mm, vias 0 -> 1
- net dCSI-0_D1_P: track 0.00 -> 49.2 mm, vias 0 -> 1
- net dCSI-0_CLK_N: track 0.00 -> 48.7 mm, vias 0 -> 1
- net dCSI-0_CLK_P: track 0.00 -> 47.7 mm, vias 0 -> 1
- net GND: vias 65 -> 69

Commit message: tuned skew before dampening resistors
Parts:
- moved R40 0.22 mm to (135.5, 88.1)
- moved R41 0.22 mm to (134.5, 88.1)
- moved R26 0.08 mm to (142.5, 88.1)
- moved R27 0.08 mm to (141.6, 88.1)
Routing:
- net USB_N: track 2.32 -> 0.00 mm
- net USB_P: track 2.01 -> 0.00 mm
- net CSI-1_CLK_N: track 4.50 -> 5.47 mm
- net USB3-1-RX_P: track 47.0 -> 47.8 mm
- net USB3-1-TX_P: track 45.2 -> 46.1 mm

Commit message: tuned the skew of every CSI line, done CSI and some DP/DMgit add .!
Routing:
- net dCSI-0_D1_P: track 49.2 -> 50.3 mm
- net dCSI-1_D3_N: track 20.6 -> 21.7 mm
- net dCSI-0_CLK_P: track 47.7 -> 48.7 mm
- net dCSI-1_D0_P: track 35.5 -> 36.4 mm
- net dCSI-1_CLK_P: track 28.1 -> 29.1 mm
- net dCSI-0_D2_P: track 48.3 -> 49.2 mm
- net dCSI-0_D3_P: track 44.9 -> 45.7 mm
- net dCSI-0_D0_P: track 55.8 -> 56.6 mm
- net CSI-1_D3_P: track 15.5 -> 16.3 mm
- net dCSI-1_D1_P: track 32.3 -> 32.9 mm

Commit message: moving some stuff so I can connect grounds, HDMI routing a bit sketchy
Routing:
- net GND: track 67.9 -> 75.8 mm, vias 69 -> 68
- net SPI-0_CLK_1V8: track 5.59 -> 0.00 mm, vias 1 -> 0
- net HDMI-0_SCL: track 9.68 -> 10.9 mm, vias 2 -> 1
- net USB3-1-TX_N: track 46.2 -> 45.5 mm
- net USB3-1-TX_P: track 46.1 -> 45.4 mm

Commit message: adding return via's to every single pair
Parts:
- moved R50 0.22 mm to (122.3, 88.3)
- moved R51 0.22 mm to (121.6, 89.0)
Connections:
- R26 pad 2: dUSB_M -> dUSB_N
Routing:
- net HDMI-0_SDA: track 5.82 -> 14.6 mm
- net GND: track 75.8 -> 84.5 mm, vias 68 -> 77
- net USB_N: track 0.00 -> 2.28 mm
- net USB_P: track 0.00 -> 1.98 mm
- net HDMI-0_CEC: track 4.14 -> 5.06 mm, vias 1 -> 2
- net HDMI-0_HPD: track 5.17 -> 5.94 mm, vias 1 -> 2
- net dCSI-1_D2_N: track 32.5 -> 33.1 mm
- net dCSI-1_D2_P: track 32.4 -> 33.1 mm
