File: PCB_CARRIER/carrier.kicad_pcb (KiCad board)
At the start: 6 copper layers, 69.6 x 46 mm, 87 parts, among them J1 SODIMM-260_Split, J2 Micro_SD_Card_Det2, Q2 BSS138, Q3 BSS138, Q4 BC817-40, Q5 BSS138, SW1 SW_DIP_x04, U1 SN74LVC8T245, U2 SN74LVC8T245, U3 SN74LVC8T245, U4 RT9742GGJ5

Commit message: routing the SD card!
Parts:
- C20, J2, R14, R17, R18, R19, R20, R21, U4: moved to F.Cu
- moved R17 9.86 mm to (150.8, 75.0), turned to 0 degrees
- moved R18 7.56 mm to (150.8, 73.8), turned to 0 degrees
- moved R14 5.59 mm to (148.3, 74.8), turned to 180 degrees
- moved R21 5.55 mm to (150.8, 67.2), turned to 0 degrees
- moved C20 4.83 mm to (150.9, 71.5), turned to -90 degrees
- moved U4 1.93 mm to (148.3, 72.2), turned to -90 degrees
- moved R20 1.15 mm to (150.8, 69.4), turned to 0 degrees
- moved R19 0.12 mm to (150.8, 68.3), turned to 0 degrees
- turned J2 to 90 degrees
Routing:
- net GND: track 122.3 -> 126.6 mm, vias 115 -> 121
- net SD_PWR: track 0.00 -> 3.90 mm
- net SD_PWR_ON: track 0.00 -> 1.70 mm
- net SD_DAT1: track 0.00 -> 1.64 mm
- net SD_DAT3: track 0.00 -> 1.63 mm
- net SD_DAT0: track 0.00 -> 1.63 mm
- net SD_DAT2: track 0.00 -> 1.62 mm
- net SD_CMD: track 0.00 -> 1.62 mm

Commit message: re-routing USB to have less crosstalk
Parts:
- moved C16 0.54 mm to (141.5, 73.4)
- moved C17 0.54 mm to (140.5, 73.4)
- moved C12 0.54 mm to (141.5, 66.5)
- moved C14 0.54 mm to (140.5, 66.5)
- moved R6 0.54 mm to (141.2, 67.9)
- moved R7 0.54 mm to (141.2, 71.9)
- moved U3 0.54 mm to (137.4, 69.9)
- moved U1 0.41 mm to (119.8, 69.2)
- moved C3 0.41 mm to (116.7, 72.6)
- moved C8 0.41 mm to (115.7, 72.6)
- moved R5 0.41 mm to (116.0, 67.2)
- moved C10 0.41 mm to (116.7, 65.8)
- moved C9 0.41 mm to (115.7, 65.8)
- moved R2 0.41 mm to (116.0, 71.2)
- moved C13 0.24 mm to (125.1, 73.2)
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Routing:
- net USB3-0-TX_P: track 19.5 -> 22.1 mm
- net USB3-0-RX_P: track 17.0 -> 19.1 mm
- net USB3-0-TX_N: track 19.4 -> 18.3 mm

Commit message: starting to route my level shifters!
Parts:
- moved R12 7.34 mm to (158.1, 79.1)
- moved R13 7.34 mm to (156.1, 83.3), turned to 0 degrees
- moved Q3 7.34 mm to (157.6, 81.7)
- moved R25 6.83 mm to (163.0, 83.4), turned to 0 degrees
- moved Q5 6.82 mm to (164.6, 81.7)
- moved R24 6.81 mm to (165.2, 79.1)
- moved C16 0.91 mm to (141.4, 72.5)
- moved C17 0.91 mm to (140.4, 72.5)
- moved C12 0.91 mm to (141.4, 65.6)
- moved C14 0.91 mm to (140.4, 65.6)
- moved R6 0.91 mm to (141.1, 67.0)
- moved R7 0.91 mm to (141.1, 71.0)
- moved U3 0.91 mm to (137.3, 69.0)
- moved C13 0.89 mm to (125.7, 72.5)
- moved C15 0.89 mm to (126.7, 72.5)
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Routing:
- net GND: track 126.6 -> 138.8 mm, vias 121 -> 132
- net SPI-0_MISO_3V3: track 0.00 -> 7.20 mm
- net FAN_TACH_3V3: track 0.00 -> 7.10 mm
- net SPI-1_MISO_3V3: track 0.00 -> 6.60 mm
Other:
- outline, holes or cut-outs redrawn

Commit message: some level shifting routing, gonna head out but work on GBe in the morning
Routing:
- net UART-0_RTS_3V3: track 0.00 -> 7.26 mm
- net UART-2_TX_3V3: track 0.00 -> 6.76 mm
- net GND: track 138.8 -> 144.7 mm, vias 132 -> 142

Commit message: routing low speeds!
Routing:
- net UART-1_TX_3V3: track 0.00 -> 13.6 mm, vias 0 -> 2
- net UART-1_RTS_3V3: track 0.00 -> 10.8 mm, vias 0 -> 2
- net GPIO0_3V3: track 0.00 -> 9.92 mm, vias 0 -> 2
- net UART-2_RX_3V3: track 0.00 -> 8.68 mm, vias 0 -> 2
- net UART-1_RX_3V3: track 0.00 -> 7.56 mm, vias 0 -> 2
- net GND: track 144.7 -> 151.1 mm, vias 142 -> 153

Commit message: trying a new way of routing low speeds!
Routing:
- net UART-1_TX_3V3: track 13.6 -> 1.73 mm, vias 2 -> 1
- net UART-0_TX_3V3: track 0.00 -> 11.6 mm
- net UART-1_RTS_3V3: track 10.8 -> 1.85 mm, vias 2 -> 1
- net UART-2_RX_3V3: track 8.68 -> 2.53 mm, vias 2 -> 1
- net SPI-0_MISO_3V3: track 7.20 -> 1.56 mm, vias 0 -> 1
- net UART-1_RX_3V3: track 7.56 -> 2.45 mm, vias 2 -> 1
- net UART-1_CTS_3V3: track 0.00 -> 2.82 mm, vias 0 -> 1
- net UART-0_CTS_3V3: track 0.00 -> 2.66 mm, vias 0 -> 1
- net UART-0_RX_3V3: track 0.00 -> 1.77 mm, vias 0 -> 1
- net SPI-1_CS1_3V3: track 0.00 -> 1.18 mm, vias 0 -> 1
- net FAN_PWM_3V3: track 0.00 -> 1.16 mm, vias 0 -> 1
- net SPI-1_MISO_3V3: track 6.60 -> 7.27 mm, vias 0 -> 1
- net FAN_TACH_3V3: track 7.10 -> 7.61 mm, vias 0 -> 1
- net GPIO0_3V3: track 9.92 -> 9.69 mm, vias 2 -> 0
- net UART-2_TX_3V3: track 6.76 -> 6.84 mm, vias 0 -> 2
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
Commit message: more routing level shifting, almost done!
Routing:
- net SPI-0_CLK_3V3: track 0.00 -> 24.3 mm, vias 0 -> 2
- net SPI-0_MOSI_3V3: track 0.00 -> 24.2 mm, vias 0 -> 2
- net SPI-1_CS1_3V3: track 1.18 -> 15.3 mm, vias 1 -> 0
- net UART-1_TX_3V3: track 1.73 -> 14.8 mm, vias 1 -> 3
- net UART-0_RX_3V3: track 1.77 -> 10.3 mm, vias 1 -> 2
- net UART-1_RTS_3V3: track 1.85 -> 10.4 mm, vias 1 -> 2
- net UART-2_RX_3V3: track 2.53 -> 9.18 mm, vias 1 -> 2
- net SPI-0_MISO_3V3: track 1.56 -> 7.46 mm, vias 1 -> 2
- net UART-1_RX_3V3: track 2.45 -> 6.91 mm, vias 1 -> 2
- net SPI-1_CLK_3V3: track 0.00 -> 2.40 mm, vias 0 -> 1
- net SPI-0_CS1_3V3: track 0.00 -> 2.19 mm, vias 0 -> 1
- net SPI-0_CS0_3V3: track 0.00 -> 2.12 mm, vias 0 -> 1
- net SPI-1_MOSI_3V3: track 0.00 -> 1.71 mm, vias 0 -> 1
- net SPI-1_CS0_3V3: track 0.00 -> 1.63 mm, vias 0 -> 1
- net I2C-0_SDA: track 0.00 -> 1.40 mm, vias 0 -> 1
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Other:
- outline, holes or cut-outs redrawn

Commit message: finished wiring pin-in for level shifters! I want to make sure I space out SPI/I2C a bit bc they're kinda higher speed!
Routing:
- net SPI-1_MOSI_3V3: track 1.71 -> 22.3 mm, vias 1 -> 2
- net SPI-1_CLK_3V3: track 2.40 -> 22.3 mm, vias 1 -> 2
- net SPI-0_CS1_3V3: track 2.19 -> 20.6 mm, vias 1 -> 2
- net SPI-0_CS0_3V3: track 2.12 -> 20.4 mm, vias 1 -> 2
- net UART-1_CTS_3V3: track 2.82 -> 17.7 mm, vias 1 -> 2
- net SPI-1_CS0_3V3: track 1.63 -> 15.8 mm, vias 1 -> 2
- net FAN_PWM_3V3: track 1.16 -> 13.6 mm, vias 1 -> 2
- net UART-0_CTS_3V3: track 2.66 -> 11.3 mm, vias 1 -> 2
