File: PCB_CARRIER/carrier.kicad_pcb (KiCad board)
At the start: 6 copper layers, 69.6 x 46 mm, 97 parts, among them J1 SODIMM-260_Split, J2 Micro_SD_Card_Det2, Q2 BSS138, Q3 BSS138, Q4 BC817-40, Q5 BSS138, SW1 SW_DIP_x04, U1 SN74LVC8T245, U2 SN74LVC8T245, U3 SN74LVC8T245, U4 RT9742GGJ5

Commit message: routed all the level shifters!
Routing:
- net UART-2_RX_1V8: track 4.53 -> 49.2 mm, vias 2 -> 3
- net FAN_TACH_1V8: track 2.32 -> 42.5 mm, vias 1 -> 3
- net UART-1_CTS_1V8: track 5.55 -> 40.0 mm, vias 2 -> 3
- net UART-1_RX_1V8: track 6.62 -> 38.4 mm
- net UART-2_TX_1V8: track 30.5 -> 47.5 mm
- net FAN_PWM_1V8: track 30.5 -> 47.3 mm
- net POWER_BMC: track 0.00 -> 4.84 mm, vias 0 -> 1
- net VBAT: track 0.00 -> 4.66 mm, vias 0 -> 1
- net SHUT_REQ_BMC: track 0.00 -> 4.41 mm, vias 0 -> 1
- net RESET_BMC: track 0.00 -> 3.35 mm, vias 0 -> 1
- net GND: track 157.4 -> 160.2 mm, vias 168 -> 169
- net CSI-0_SDA: track 3.90 -> 2.70 mm
- net CSI-0_SCL: track 3.79 -> 3.09 mm

Commit message: routing the SD card and some other peripherals
Parts:
- moved R16 1.91 mm to (152.4, 56.8), turned to 90 degrees
Routing:
- net MOD_PWR_REQ: track 0.00 -> 47.0 mm, vias 0 -> 2
- net SD_DAT1: track 1.64 -> 45.1 mm
- net SD_DAT0: track 1.63 -> 42.2 mm
- net SD_DAT2: track 1.62 -> 36.3 mm, vias 0 -> 2
- net SD_DAT3: track 1.63 -> 33.9 mm
- net ACTIVITY_LED: track 0.00 -> 30.2 mm, vias 0 -> 2
- net Net-(D2-K): track 0.00 -> 11.5 mm
- net GND: track 160.2 -> 164.8 mm, vias 169 -> 171
- net RESET_BMC: track 3.35 -> 4.85 mm
- net SHUT_REQ_BMC: track 4.41 -> 5.89 mm
- net POWER_BMC: track 4.84 -> 6.30 mm
- net Net-(D2-A): track 0.00 -> 1.36 mm
- net Net-(D1-A): track 0.00 -> 1.36 mm
- net SYS_RESET: track 0.00 -> 1.30 mm
- net I2C-0_SCL: track 0.00 -> 1.28 mm, vias 0 -> 1
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
Commit message: routing out power/gnd, not the cleanest so I'm going to research
Routing:
- net SD_PWR_ON: track 1.70 -> 45.5 mm, vias 0 -> 2
- net LED_PWR: track 0.00 -> 31.5 mm, vias 0 -> 2
- net +5V: track 13.2 -> 22.9 mm, vias 0 -> 10
- net GND: track 164.8 -> 166.5 mm
- added copper zone on B.Cu, net +5V
- added copper zone on F.Cu, net +5V

Commit message: journaling about routing low speeds, nothing exciting
Routing:
- net +5V: track 22.9 -> 106.8 mm
- net SHUT_REQ_BMC: track 5.89 -> 25.9 mm, vias 1 -> 2
- net POWER_BMC: track 6.30 -> 24.1 mm, vias 1 -> 2
- net RESET_BMC: track 4.85 -> 20.8 mm, vias 1 -> 2

Commit message: adding power to the journal
Routing:
- net +5V: track 106.8 -> 93.7 mm
Changed lines of the file:
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@@
-	)
-	(segment
-		(start 124.812501 56.500025)
-		(end 124.812501 55.997625)
-		(width 0.1524)
-		(layer "F.Cu")
-		(net 33)
 	)
 	(segment
@@
 	)
 	(segment
-		(start 121.905 55.24)
-		(end 122.81 55.24)
-		(width 0.1524)
-		(layer "F.Cu")
-		(net 33)
-	)
-	(segment
 		(start 114.35 59.35)
 		(end 116.1 57.6)
 		(width 0.75)
-		(layer "F.Cu")
-		(net 33)
-	)
-	(segment
-		(start 126.012501 56.297499)
-		(end 126.74 55.57)
-		(width 0.1524)
 		(layer "F.Cu")
 		(net 33)
@@
 		(end 168.1 96.65)
 		(width 0.75)
-		(layer "F.Cu")
-		(net 33)
-	)
-	(segment
-		(start 126.74 55.57)
-		(end 127.01 55.57)
-		(width 0.1524)
-		(layer "F.Cu")
-		(net 33)
-	)
-	(segment
-		(start 124.384876 55.57)
-		(end 124.1 55.57)
-		(width 0.1524)
 		(layer "F.Cu")
 		(net 33)
@@
 	)
 	(segment
-		(start 125.612501 56.500025)
-		(end 125.612501 55.997499)
-		(width 0.1524)
-		(layer "F.Cu")
-		(net 33)
-	)
-	(segment
-		(start 127.97 55.56)
-		(end 127.98 55.57)
-		(width 0.1524)
-		(layer "F.Cu")
-		(net 33)
-	)
-	(segment
-		(start 125.612501 55.997499)
-		(end 126.04 55.57)
-		(width 0.1524)
-		(layer "F.Cu")
-		(net 33)
-	)
-	(segment
 		(start 144.4 79.25)
 		(end 144.4 70.55)
 		(width 0.75)
-		(layer "F.Cu")
-		(net 33)
-	)
-	(segment
-		(start 123.13 55.56)
-		(end 127.97 55.56)
-		(width 0.1524)
 		(layer "F.Cu")
 		(net 33)
@@
 	)
 	(segment
-		(start 125.212501 56.500025)
-		(end 125.212501 55.712501)
-		(width 0.1524)
-		(layer "F.Cu")
-		(net 33)
-	)
-	(segment
 		(start 142.75 68.9)
 		(end 115.5 68.9)
 		(width 0.75)
-		(layer "F.Cu")
-		(net 33)
-	)
-	(segment
-		(start 126.412501 56.500025)
-		(end 127.342526 55.57)
-		(width 0.1524)
-		(layer "F.Cu")
-		(net 33)
-	)
-	(segment
-		(start 124.812501 55.997625)
-		(end 124.384876 55.57)
-		(width 0.1524)
-		(layer "F.Cu")
-		(net 33)
-	)
-	(segment
-		(start 125.212501 55.712501)
-		(end 125.07 55.57)
-		(width 0.1524)
-		(layer "F.Cu")
-		(net 33)
-	)
-	(segment
-		(start 122.81 55.24)
-		(end 123.13 55.56)
-		(width 0.1524)
 		(layer "F.Cu")
 		(net 33)
@@
 		(layer "F.Cu")
 		(net 33)
-	)
-	(segment
-		(start 126.012501 56.500025)
-		(end 126.012501 56.297499)
-		(width 0.1524)
-		(layer "F.Cu")
-		(net 33)
-	)
-	(segment
-		(start 127.342526 55.57)
-		(end 127.98 55.57)
-		(width 0.1524)
-		(layer "F.Cu")
-		(net 33)

Commit message: only 36 connections leftgit add .!
Parts:
- moved TP2 14.2 mm to (144.6, 42.7)
Routing:
- net +3V3: track 6.62 -> 109.0 mm
- net +1V8: track 6.26 -> 95.1 mm, vias 0 -> 4
- net SYS_RESET: track 1.30 -> 33.4 mm, vias 0 -> 2
- net PWR_Button: track 0.00 -> 26.5 mm, vias 0 -> 2
- net PMIC_EN: track 1.27 -> 27.0 mm, vias 0 -> 2
- net nRPIBOOT: track 0.00 -> 25.2 mm, vias 0 -> 2
- net dUSB_N: track 3.79 -> 22.2 mm, vias 1 -> 2
- net dUSB_P: track 4.18 -> 22.5 mm, vias 1 -> 2
- net +5V: track 93.7 -> 106.4 mm, vias 10 -> 12
- net SLEEP/WAKE: track 4.79 -> 8.49 mm
- net MOD_PWR_REQ: track 47.0 -> 47.6 mm
- net LED_PWR: track 31.5 -> 32.1 mm
- net SPI-1_CS1_3V3: track 12.0 -> 12.5 mm, vias 0 -> 2
- net GND: vias 171 -> 173

Commit message: only 21 more nets leftgit add .
Parts:
- moved TP1 17.0 mm to (128.6, 49.4)
Routing:
- net CSI-0_SCL: track 3.09 -> 66.8 mm, vias 1 -> 4
- net CSI-0_SDA: track 2.70 -> 65.4 mm, vias 1 -> 4
- net VBAT: track 4.66 -> 64.2 mm, vias 1 -> 4
- net CSI-1_PWDN: track 3.08 -> 56.6 mm, vias 1 -> 4
- net CSI-0_PWDN: track 5.29 -> 53.6 mm, vias 1 -> 2
- net +3V3: track 109.0 -> 133.3 mm, vias 0 -> 2
- net GND: track 166.5 -> 183.9 mm, vias 173 -> 177
- net I2C-0_SCL: track 1.28 -> 7.67 mm, vias 1 -> 2
- net I2C-0_SDA: track 1.40 -> 7.60 mm, vias 1 -> 2
- net UART-2_RX_1V8: track 49.2 -> 44.5 mm
- net UART-1_CTS_3V3: track 17.7 -> 19.5 mm
- net SPI-1_MOSI_1V8: track 48.7 -> 49.4 mm
- net SPI-0_MOSI_3V3: track 24.6 -> 25.3 mm
- net SPI-0_CLK_3V3: track 29.4 -> 30.0 mm

Commit message: 11 nets left, no long ones anymoregit add .!
Parts:
- moved TP2 50.3 mm to (146.9, 93.0)
- moved TP1 47.8 mm to (156.4, 88.2)
Routing:
- net SLEEP/WAKE: track 8.49 -> 74.1 mm, vias 2 -> 4
- net PMIC_EN: track 26.7 -> 89.2 mm, vias 2 -> 3
- net I2C-0_SCL: track 7.67 -> 65.2 mm
- net MOD_SLEEP: track 0.00 -> 55.6 mm, vias 0 -> 2
- net I2C-0_SDA: track 7.60 -> 60.9 mm, vias 2 -> 4
- net SYS_RESET: track 33.4 -> 85.5 mm, vias 2 -> 3
- net SD_CLK: track 0.00 -> 39.7 mm, vias 0 -> 2
- net SD_CMD: track 1.62 -> 32.8 mm, vias 0 -> 2
- net VBAT: track 64.2 -> 65.9 mm
- net UART-1_CTS_3V3: track 19.5 -> 21.1 mm
- net UART-0_CTS_3V3: track 11.4 -> 12.5 mm
- net GND: track 183.9 -> 184.5 mm
